File: pre-amp-discret-v3/pre-amp-discret.sch (KiCad schematic (older format))
At the start: 56 parts, among them J1 Conn_01x01, J2 Conn_01x01, J3 Conn_01x01, J4 Conn_01x01, J5 Conn_01x01, J6 Conn_01x01, J7 Conn_01x01, Q1 BC860C, Q10 BC860C, Q11 BC850C, Q12 BC860C, Q2 BC850C, Q3 BC860C, Q4 BC850C, Q5 BC860C, Q6 BC850C, Q7 BC860C, Q8 BC850C, Q9 BC860C

Commit message: WIP
Parts:
- removed C6: 100uF, Capacitor_THT:CP_Radial_D8.0mm_P3.50mm, symbol Device:CP
- added C6: 100uF, Capacitor_SMD:C_1210_3225Metric_Pad1.33x2.70mm_HandSolder, symbol Device:C
- C1, C3: footprint Capacitor_THT:CP_Radial_D8.0mm_P3.50mm -> Capacitor_SMD:CP_Elec_8x10
- C10, C11, C8, C9: footprint Capacitor_THT:CP_Radial_D5.0mm_P2.00mm -> Capacitor_SMD:CP_Elec_4x4.5
- C13, C14, C4, C5: footprint Capacitor_THT:C_Rect_L7.2mm_W2.5mm_P5.00mm_FKS2_FKP2_MKS2_MKP2 -> Capacitor_SMD:C_0805_2012Metric_Pad1.18x1.45mm_HandSolder
Connections:
- net GND: now also C6.2
- net at R8.2: now also C6.1
Changed lines of the file:
@@
-$EndComp
-$Comp
-L Device:CP C6
-U 1 1 5F7FEF9F
-P 3650 4050
-F 0 "C6" H 3768 4096 50  0000 L CNN
-F 1 "100uF" H 3768 4005 50  0000 L CNN
-F 2 "Capacitor_THT:CP_Radial_D8.0mm_P3.50mm" H 3688 3900 50  0001 C CNN
-F 3 "~" H 3650 4050 50  0001 C CNN
-	1    3650 4050
-	1    0    0    -1
 $EndComp
 $Comp
@@
 F 0 "C3" H 1368 5496 50  0000 L CNN
 F 1 "100uF" H 1368 5405 50  0000 L CNN
-F 2 "Capacitor_THT:CP_Radial_D8.0mm_P3.50mm" H 1288 5300 50  0001 C CNN
+F 2 "Capacitor_SMD:CP_Elec_8x10" H 1288 5300 50  0001 C CNN
 F 3 "~" H 1250 5450 50  0001 C CNN
 	1    1250 5450
@@
 F 0 "C1" H 1368 1496 50  0000 L CNN
 F 1 "100uF" H 1368 1405 50  0000 L CNN
-F 2 "Capacitor_THT:CP_Radial_D8.0mm_P3.50mm" H 1288 1300 50  0001 C CNN
+F 2 "Capacitor_SMD:CP_Elec_8x10" H 1288 1300 50  0001 C CNN
 F 3 "~" H 1250 1450 50  0001 C CNN
 	1    1250 1450
@@
 F 0 "C8" H 8868 2346 50  0000 L CNN
 F 1 "4.7uF" H 8868 2255 50  0000 L CNN
-F 2 "Capacitor_THT:CP_Radial_D5.0mm_P2.00mm" H 8788 2150 50  0001 C CNN
+F 2 "Capacitor_SMD:CP_Elec_4x4.5" H 8788 2150 50  0001 C CNN
 F 3 "~" H 8750 2300 50  0001 C CNN
 	1    8750 2300
@@
 F 0 "C9" H 9718 2546 50  0000 L CNN
 F 1 "4.7uF" H 9718 2455 50  0000 L CNN
-F 2 "Capacitor_THT:CP_Radial_D5.0mm_P2.00mm" H 9638 2350 50  0001 C CNN
+F 2 "Capacitor_SMD:CP_Elec_4x4.5" H 9638 2350 50  0001 C CNN
 F 3 "~" H 9600 2500 50  0001 C CNN
 	1    9600 2500
@@
 F 0 "C10" H 8632 5154 50  0000 R CNN
 F 1 "4.7uF" H 8632 5245 50  0000 R CNN
-F 2 "Capacitor_THT:CP_Radial_D5.0mm_P2.00mm" H 8788 5050 50  0001 C CNN
+F 2 "Capacitor_SMD:CP_Elec_4x4.5" H 8788 5050 50  0001 C CNN
 F 3 "~" H 8750 5200 50  0001 C CNN
 	1    8750 5200
@@
 F 0 "C11" H 9482 5354 50  0000 R CNN
 F 1 "4.7uF" H 9482 5445 50  0000 R CNN
-F 2 "Capacitor_THT:CP_Radial_D5.0mm_P2.00mm" H 9638 5250 50  0001 C CNN
+F 2 "Capacitor_SMD:CP_Elec_4x4.5" H 9638 5250 50  0001 C CNN
 F 3 "~" H 9600 5400 50  0001 C CNN
 	1    9600 5400
@@
 F 0 "C13" H 6485 1404 50  0000 R CNN
 F 1 "100nF" H 6485 1495 50  0000 R CNN
-F 2 "Capacitor_THT:C_Rect_L7.2mm_W2.5mm_P5.00mm_FKS2_FKP2_MKS2_MKP2" H 6638 1300 50  0001 C CNN
+F 2 "Capacitor_SMD:C_0805_2012Metric_Pad1.18x1.45mm_HandSolder" H 6638 1300 50  0001 C CNN
 F 3 "~" H 6600 1450 50  0001 C CNN
 	1    6600 1450
@@
 F 0 "C4" H 1635 1404 50  0000 R CNN
 F 1 "100nF" H 1635 1495 50  0000 R CNN
-F 2 "Capacitor_THT:C_Rect_L7.2mm_W2.5mm_P5.00mm_FKS2_FKP2_MKS2_MKP2" H 1788 1300 50  0001 C CNN
+F 2 "Capacitor_SMD:C_0805_2012Metric_Pad1.18x1.45mm_HandSolder" H 1788 1300 50  0001 C CNN
 F 3 "~" H 1750 1450 50  0001 C CNN
 	1    1750 1450
@@
 F 0 "C14" H 6485 5404 50  0000 R CNN
 F 1 "100nF" H 6485 5495 50  0000 R CNN
-F 2 "Capacitor_THT:C_Rect_L7.2mm_W2.5mm_P5.00mm_FKS2_FKP2_MKS2_MKP2" H 6638 5300 50  0001 C CNN
+F 2 "Capacitor_SMD:C_0805_2012Metric_Pad1.18x1.45mm_HandSolder" H 6638 5300 50  0001 C CNN
 F 3 "~" H 6600 5450 50  0001 C CNN
 	1    6600 5450
@@
 F 0 "C5" H 1635 5404 50  0000 R CNN
 F 1 "100nF" H 1635 5495 50  0000 R CNN
-F 2 "Capacitor_THT:C_Rect_L7.2mm_W2.5mm_P5.00mm_FKS2_FKP2_MKS2_MKP2" H 1788 5300 50  0001 C CNN
+F 2 "Capacitor_SMD:C_0805_2012Metric_Pad1.18x1.45mm_HandSolder" H 1788 5300 50  0001 C CNN
 F 3 "~" H 1750 5450 50  0001 C CNN
 	1    1750 5450
 	-1   0    0    1
 $EndComp
+$Comp
+L Device:C C6
+U 1 1 5F970BD8
+P 3650 4050
+F 0 "C6" H 3765 4096 50  0000 L CNN
+F 1 "100uF" H 3765 4005 50  0000 L CNN
+F 2 "Capacitor_SMD:C_1210_3225Metric_Pad1.33x2.70mm_HandSolder" H 3688 3900 50  0001 C CNN
+F 3 "~" H 3650 4050 50  0001 C CNN
+	1    3650 4050
+	1    0    0    -1
+$EndComp
 $EndSCHEMATC
