File: lv-lownoise-psu-v3/lv-lownoise-psu.kicad_pcb (KiCad board)
At the start: 2 copper layers, 50.8 x 48.9 mm, 33 parts, among them J1 AC, J2 GND, J3 AC, J4 +15V, J5 GND, J6 -15V, Q1 BD139, Q2 BD140, U1 LT1761-BYP, U2 LT1964-BYP

Commit message: WIP
Parts:
- removed C10: 100n, Capacitor_SMD:C_0805_2012Metric_Pad1.18x1.45mm_HandSolder
- removed C8: 10u, Capacitor_Tantalum_SMD:CP_EIA-3528-12_Kemet-T_Pad1.50x2.35mm_HandSolder
- removed U1: LT1761-BYP, Package_TO_SOT_SMD:TSOT-23-5
- removed U2: LT1964-BYP, Package_TO_SOT_SMD:TSOT-23-5
- added U3: LT3045xMSE, Package_SO:MSOP-12-1EP_3x4mm_P0.65mm_EP1.65x2.85mm, F.Cu at (101.7, 26.7)
- added U4: LT3094xMSE, Package_SO:MSOP-12-1EP_3x4mm_P0.65mm_EP1.65x2.85mm, F.Cu at (109.0, 26.7)
- C1: footprint Capacitor_SMD:CP_Elec_8x10 -> Capacitor_SMD:CP_Elec_8x6.9
- C3, C4: value 1u -> 4.7u; footprint Capacitor_SMD:C_0805_2012Metric_Pad1.18x1.45mm_HandSolder -> Capacitor_SMD:C_1206_3216Metric_Pad1.33x1.80mm_HandSolder
- C5, C6: value 10n -> 0.47u
- C7: footprint Capacitor_Tantalum_SMD:CP_EIA-3528-12_Kemet-T_Pad1.50x2.35mm_HandSolder -> Capacitor_SMD:C_1210_3225Metric_Pad1.33x2.70mm_HandSolder
- C9: value 100n -> 10u; footprint Capacitor_SMD:C_0805_2012Metric_Pad1.18x1.45mm_HandSolder -> Capacitor_SMD:C_1210_3225Metric_Pad1.33x2.70mm_HandSolder
- R1, R2: value 15k -> 150k
- RV1, RV2: value 250k -> 200k
- moved RV2 57.5 mm to (106.2, 27.1), turned to 0 degrees
- moved R2 50.4 mm to (111.6, 29.6), turned to 0 degrees
- moved C6 48.2 mm to (106.5, 31.8), turned to 0 degrees
- moved C4 43.0 mm to (101.1, 32.0), turned to 0 degrees
- moved C5 28.8 mm to (100.5, 30.9), turned to 0 degrees
- moved C7 23.7 mm to (112.2, 26.0), turned to 0 degrees
Connections:
- C7 pad 1: Net-(C7-Pad1) -> GND
- C7 pad 2: GND -> Net-(C7-Pad2)
- C9 pad 1: Net-(C7-Pad1) -> Net-(C9-Pad1)
- J4 pad 1: Net-(C7-Pad1) -> Net-(C9-Pad1)
- J6 pad 1: Net-(C10-Pad2) -> Net-(C7-Pad2)
- R1 pad 1: Net-(R1-Pad1) -> Net-(C5-Pad1)
- R2 pad 2: Net-(R2-Pad2) -> Net-(C6-Pad2)
- RV1 pad 1: Net-(C7-Pad1) -> Net-(C5-Pad1)
- RV1 pad 2: Net-(R1-Pad1) -> GND
- RV1 pad 3: Net-(R1-Pad1) -> GND
- RV2 pad 1: Net-(R2-Pad2) -> GND
- RV2 pad 2: Net-(R2-Pad2) -> GND
- RV2 pad 3: Net-(C10-Pad2) -> Net-(C6-Pad2)
Routing:
- net Net-(C7-Pad2): track 0.00 -> 18.0 mm, vias 0 -> 2
- net Net-(C10-Pad2): track 18.0 -> 0.00 mm, vias 2 -> 0

Commit message: WIP
Parts:
- C2: footprint Capacitor_SMD:CP_Elec_8x10 -> Capacitor_SMD:CP_Elec_8x6.9
- moved RV2 53.4 mm to (114.2, 79.9), turned to 270 degrees
- moved C6 46.7 mm to (109.5, 78.5), turned to 90 degrees
- moved R2 46.0 mm to (108.5, 75.5)
- moved U4 45.4 mm to (108.3, 72.1)
- moved C7 43.5 mm to (113.2, 69.5), turned to 270 degrees
- moved C4 37.0 mm to (103.8, 68.9), turned to 270 degrees
- moved C5 31.2 mm to (109.4, 60.9), turned to 270 degrees
- moved U3 28.7 mm to (108.5, 54.6)
- moved Q2 10.1 mm to (100.2, 70.4), turned to 270 degrees
- moved Q1 6.89 mm to (100.4, 53.0), turned to 270 degrees
- moved R6 5.69 mm to (101.4, 60.9), turned to 0 degrees
- moved R7 4.72 mm to (101.2, 78.5), turned to 180 degrees
- moved C3 3.86 mm to (104.0, 51.4), turned to 90 degrees
- moved R1 3.41 mm to (108.4, 58.0), turned to 180 degrees
- moved R5 2.32 mm to (103.9, 56.6)
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Routing:
- net Net-(C1-Pad1): track 26.9 -> 0.63 mm, vias 1 -> 0
- net Net-(C2-Pad2): track 26.5 -> 1.36 mm, vias 3 -> 1
- net Net-(C7-Pad1): track 18.5 -> 0.00 mm, vias 2 -> 0
- net Net-(C7-Pad2): track 18.0 -> 0.00 mm, vias 2 -> 0
- net Net-(R1-Pad1): track 10.5 -> 0.00 mm, vias 1 -> 0
- net Net-(R2-Pad2): track 10.2 -> 0.00 mm, vias 1 -> 0
- net Net-(Q1-Pad3): track 7.63 -> 0.00 mm
- net Net-(Q2-Pad3): track 6.97 -> 0.00 mm
- net GND: track 6.23 -> 0.00 mm, vias 0 -> 3
- net Net-(C3-Pad1): track 5.97 -> 0.00 mm
- net Net-(C4-Pad2): track 5.36 -> 0.00 mm
- net Net-(C6-Pad2): track 2.25 -> 0.00 mm
- net Net-(C5-Pad1): track 2.21 -> 0.00 mm

Commit message: WIP
Parts:
- moved C5 8.41 mm to (116.0, 55.6), turned to 0 degrees
- moved C6 7.74 mm to (115.7, 73.9), turned to 180 degrees
- moved R1 4.77 mm to (113.0, 56.6), turned to 270 degrees
- moved R2 4.05 mm to (112.5, 74.9), turned to 90 degrees
- moved J6 3.56 mm to (122.8, 71.1)
- moved RV2 3.26 mm to (116.5, 77.5), turned to 90 degrees
- moved RV1 3.19 mm to (116.8, 59.3)
- moved J5 2.19 mm to (122.7, 61.9)
- moved J4 0.27 mm to (122.7, 53.6)
Connections:
- RV2 pad 1: GND -> Net-(C6-Pad2)
- RV2 pad 3: Net-(C6-Pad2) -> GND
Routing:
- net Net-(C3-Pad1): track 0.00 -> 16.1 mm, vias 0 -> 2
- net Net-(C9-Pad1): track 0.00 -> 13.4 mm, vias 0 -> 1
- net Net-(C1-Pad1): track 0.63 -> 13.6 mm, vias 0 -> 1
- net Net-(C7-Pad2): track 0.00 -> 9.62 mm, vias 0 -> 1
- net Net-(C5-Pad1): track 0.00 -> 9.40 mm, vias 0 -> 1
- net Net-(Q1-Pad3): track 0.00 -> 6.59 mm
- net GND: track 0.00 -> 5.40 mm, vias 3 -> 0
- net Net-(C6-Pad2): track 0.00 -> 5.10 mm, vias 0 -> 1

Commit message: Update lv-lownoise-psu.kicad_pcb
Parts:
- moved R8 1.59 mm to (103.6, 73.9)
Routing:
- net Net-(C2-Pad2): track 1.36 -> 21.2 mm, vias 1 -> 3
- net Net-(C4-Pad2): track 0.00 -> 12.1 mm
- net Net-(C1-Pad1): track 13.6 -> 21.3 mm
- net Net-(Q2-Pad3): track 0.00 -> 6.70 mm
- net Net-(C6-Pad2): track 5.10 -> 9.63 mm
- net Net-(C7-Pad2): track 9.62 -> 13.6 mm
- net GND: track 5.40 -> 8.28 mm, vias 0 -> 2
Other:
- board text added: "Low noise dual power supply V3 Michael Schenk, 2020.11.01"
- board text removed: "Low noise dual power supply V2 Michael Schenk, 2020.10.26"

Commit message: Optimize layout
Parts:
- Q1: value BD139 -> BD679
- Q2: value BD140 -> BD680
