File: pre-amp-discret-v4/pre-amp-discret.kicad_pcb (KiCad board)
At the start: 2 copper layers, 81.9 x 52.1 mm, 56 parts, among them J1 Conn_01x01, J2 Conn_01x01, J3 Conn_01x01, J4 Conn_01x01, J5 Conn_01x01, J6 Conn_01x01, J7 Conn_01x01, Q1 BC860C, Q10 BC860C, Q11 BC850C, Q12 BC860C, Q2 BC850C, Q3 BC860C, Q4 BC850C, Q5 BC860C, Q6 BC850C, Q7 BC860C, Q8 BC850C, Q9 BC860C

Commit message: start with version 4
Parts:
- J1, J2, J3, J4, J5, J6, J7: footprint Connector_Pin:Pin_D1.3mm_L11.0mm -> Connector_Pin:Pin_D1.0mm_L10.0mm

Commit message: WIP
Parts:
- added C15: 470uF, Capacitor_THT:CP_Radial_D10.0mm_P5.00mm, F.Cu at (113.8, 86.6)
- added C16: 470uF, Capacitor_THT:CP_Radial_D10.0mm_P5.00mm, F.Cu at (125.6, 86.6)
- C1, C3: value 100uF -> 470uF; footprint Capacitor_SMD:CP_Elec_8x10 -> Capacitor_THT:CP_Radial_D10.0mm_P5.00mm
- C10, C8: value 4.7uF -> 100uF; footprint Capacitor_SMD:CP_Elec_4x4.5 -> Capacitor_THT:CP_Radial_D8.0mm_P3.50mm
- C11, C9: value 4.7uF -> 10uF; footprint Capacitor_SMD:CP_Elec_4x4.5 -> Capacitor_THT:CP_Radial_D5.0mm_P2.00mm
- C13, C14, C4, C5: footprint Capacitor_SMD:C_0805_2012Metric_Pad1.18x1.45mm_HandSolder -> Capacitor_THT:C_Rect_L7.2mm_W2.5mm_P5.00mm_FKS2_FKP2_MKS2_MKP2
- C6: footprint Capacitor_SMD:C_1210_3225Metric_Pad1.33x2.70mm_HandSolder -> Capacitor_THT:CP_Radial_D8.0mm_P3.50mm
- moved C6 36.1 mm to (146.9, 85.9), turned to 0 degrees
- moved C8 10.3 mm to (188.0, 102.6), turned to 270 degrees
- moved C10 9.94 mm to (188.6, 137.8)
- moved R14 4.56 mm to (179.3, 106.1)
- moved Q11 3.37 mm to (174.9, 106.1)
- moved C9 2.94 mm to (175.9, 102.0)
- moved R15 2.24 mm to (171.7, 109.7)
- moved C11 0.59 mm to (173.0, 135.0)
Routing:
- net Net-(C10-Pad2): track 29.5 -> 0.00 mm, vias 1 -> 0
- net Net-(C8-Pad1): track 26.8 -> 0.00 mm, vias 1 -> 0
- net +15V: track 48.8 -> 37.1 mm, vias 6 -> 5
- net -15V: track 46.7 -> 39.1 mm, vias 7 -> 6
- net Net-(C9-Pad1): track 4.57 -> 0.00 mm
- net Net-(C11-Pad2): track 4.47 -> 0.02 mm
