File: pre-amp-discret-symetric-v1a/pre-amp-discret.kicad_pcb (KiCad board)
At the start: 2 copper layers, 81.9 x 52.1 mm, 72 parts, among them J1 Conn_01x01, J2 Conn_01x01, J3 Conn_01x01, J4 Conn_01x01, J5 Conn_01x01, J6 Conn_01x01, J7 Conn_01x01, Q1 BCM857DS,115, Q10 BC860C, Q11 BC850C, Q12 BC860C, Q13 BCM847DS,115, Q14 BCM857DS,115, Q15 BC850C, Q2 BCM847DS,115, Q3 BC860C, Q4 BCM847DS,115, Q7 BCM857DS,115, Q9 BC860C

Commit message: Copy of v1 bugfix
Parts:
- added Q16: BC860C, Package_TO_SOT_SMD:SOT-23, F.Cu at (148.7, 109.0)
- added Q17: BC850C, Package_TO_SOT_SMD:SOT-23, F.Cu at (148.7, 113.2)
- added Q18: BC860C, Package_TO_SOT_SMD:SOT-23, F.Cu at (165.0, 112.1)
- added Q5: BC860C, Package_TO_SOT_SMD:SOT-23, F.Cu at (148.7, 130.9)
- added Q6: BC850C, Package_TO_SOT_SMD:SOT-23, F.Cu at (166.2, 131.8)
- added Q8: BC850C, Package_TO_SOT_SMD:SOT-23, F.Cu at (170.7, 131.8)
- Q1, Q14, Q7: value BCM857DS,115 -> BC860C; footprint Package_SO:SC-74-6_1.5x2.9mm_P0.95mm -> Package_TO_SOT_SMD:SOT-23
- Q13, Q2, Q4: value BCM847DS,115 -> BC850C; footprint Package_SO:SC-74-6_1.5x2.9mm_P0.95mm -> Package_TO_SOT_SMD:SOT-23
- moved Q4 22.7 mm to (146.7, 135.4)
- moved R4 10.3 mm to (154.4, 101.3)
- moved R11 9.55 mm to (169.9, 101.3)
- moved R26 9.52 mm to (166.0, 101.3)
- moved C15 8.49 mm to (135.0, 100.3), turned to 270 degrees
- moved R20 8.20 mm to (144.7, 101.3)
- moved D5 8.02 mm to (173.0, 101.9)
- moved R10 6.68 mm to (165.2, 142.4)
- moved R27 5.23 mm to (169.7, 142.4)
- moved R6 5.09 mm to (147.6, 142.4)
- moved C1 4.76 mm to (180.6, 100.3)
- moved D1 4.34 mm to (157.4, 101.9)
- moved R2 3.84 mm to (143.7, 126.1)
- moved D6 3.82 mm to (174.6, 110.8), turned to 180 degrees
- moved R23 3.79 mm to (147.8, 101.3)
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Connections:
- C7 pad 1: Net-(C7-Pad1) -> Net-(C17-Pad1)
- C7 pad 2: Net-(C17-Pad1) -> Net-(C7-Pad2)
- Q1 pad 1: Net-(Q1-Pad1) -> Net-(C2-Pad1)
- Q1 pad 2: Net-(C12-Pad2) -> Net-(Q1-Pad2)
- Q1 pad 3: Net-(C7-Pad1) -> Net-(C7-Pad2)
- Q13 pad 1: Net-(Q13-Pad1) -> Net-(C2-Pad1)
- Q13 pad 2: Net-(C12-Pad2) -> Net-(Q13-Pad2)
- Q14 pad 2: Net-(Q13-Pad6) -> Net-(Q14-Pad2)
- Q14 pad 3: Net-(Q13-Pad6) -> Net-(C17-Pad2)
- Q2 pad 2: Net-(Q1-Pad6) -> Net-(Q2-Pad2)
- Q2 pad 3: Net-(Q1-Pad6) -> Net-(C7-Pad2)
- Q4 pad 1: Net-(Q4-Pad1) -> Net-(Q2-Pad1)
- Q4 pad 3: GND -> Net-(Q2-Pad1)
- Q7 pad 1: Net-(Q7-Pad1) -> Net-(Q18-Pad2)
- Q7 pad 2: Net-(C17-Pad2) -> Net-(Q7-Pad2)
- R10 pad 1: Net-(Q4-Pad2) -> Net-(Q6-Pad2)
- R11 pad 2: Net-(Q7-Pad4) -> Net-(Q7-Pad2)
- R2 pad 2: Net-(Q1-Pad4) -> Net-(Q1-Pad2)
- R20 pad 2: Net-(Q14-Pad1) -> Net-(Q14-Pad2)
- R21 pad 1: Net-(Q13-Pad4) -> Net-(Q13-Pad2)
- R23 pad 2: Net-(Q14-Pad4) -> Net-(Q16-Pad2)
- R24 pad 1: Net-(Q13-Pad1) -> Net-(Q17-Pad2)
- R26 pad 2: Net-(Q7-Pad1) -> Net-(Q18-Pad2)
- R27 pad 1: Net-(Q4-Pad1) -> Net-(Q8-Pad2)
- R3 pad 1: Net-(Q2-Pad1) -> Net-(Q2-Pad2)
- R5 pad 2: Net-(Q1-Pad1) -> Net-(Q5-Pad2)
- R6 pad 1: Net-(Q2-Pad4) -> Net-(Q4-Pad2)
Routing:
- net Net-(C7-Pad2): track 0.00 -> 32.4 mm, vias 0 -> 3
- net Net-(C7-Pad1): track 31.2 -> 0.00 mm, vias 3 -> 0
- net +15V: track 99.1 -> 69.9 mm, vias 7 -> 9
- net Net-(Q6-Pad2): track 0.00 -> 14.2 mm, vias 0 -> 2
- net Net-(Q18-Pad2): track 0.00 -> 14.0 mm, vias 0 -> 2
- net -15V: track 83.2 -> 69.9 mm, vias 7 -> 8
- net Net-(Q1-Pad6): track 9.13 -> 0.00 mm, vias 2 -> 0
- net Net-(Q7-Pad2): track 0.00 -> 8.94 mm, vias 0 -> 2
- net Net-(Q13-Pad6): track 8.81 -> 0.00 mm, vias 2 -> 0
- net Net-(Q8-Pad2): track 0.00 -> 8.67 mm, vias 0 -> 2
- net Net-(Q14-Pad1): track 2.04 -> 10.6 mm
- net Net-(Q3-Pad2): track 1.88 -> 10.0 mm, vias 0 -> 2
- net Net-(Q3-Pad3): track 13.9 -> 21.4 mm, vias 3 -> 5
- net Net-(Q2-Pad2): track 0.00 -> 6.99 mm, vias 0 -> 2
- net Net-(Q2-Pad1): track 2.35 -> 8.73 mm
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Other:
- board text added: "Pre-Amp Symetrical Discret V1 Michael Schenk 2020.11.05"
- board text removed: "Pre-Amp Symetrical Discret V2 Michael Schenk 2020.12.13"

Commit message: WIP
Parts:
- added R15: 250k, Resistor_SMD:R_0805_2012Metric_Pad1.20x1.40mm_HandSolder, F.Cu at (158.1, 122.1)
- C17, C7: value 270pF -> 1nF
- R22, R4: value 220R -> 150R
- moved R4 11.2 mm to (155.9, 112.4)
- moved R22 11.1 mm to (157.7, 131.5)
- moved D5 10.4 mm to (176.0, 111.9)
- moved R11 7.32 mm to (171.7, 108.4)
- moved R26 7.26 mm to (167.6, 108.3)
- moved R27 6.79 mm to (169.7, 135.6)
- moved R10 6.74 mm to (165.2, 135.6)
- moved D6 6.23 mm to (176.0, 116.9), turned to 90 degrees
- moved R28 6.10 mm to (180.4, 121.2), turned to 90 degrees
- moved C6 5.46 mm to (162.9, 125.9)
- moved D1 5.20 mm to (159.5, 106.6)
- moved D4 5.16 mm to (153.9, 137.1)
- moved R8 4.67 mm to (165.8, 124.9)
- moved Q15 4.50 mm to (156.7, 127.7)
- moved R9 4.12 mm to (168.1, 124.9)
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Routing:
- net +15V: track 69.9 -> 101.9 mm, vias 9 -> 8
- net -15V: track 69.9 -> 96.4 mm
- net Net-(Q15-Pad3): track 20.3 -> 10.6 mm, vias 4 -> 3
- net Net-(C17-Pad2): track 29.3 -> 38.5 mm, vias 2 -> 3
- net Net-(Q3-Pad2): track 10.0 -> 1.71 mm, vias 2 -> 0
- net Net-(C7-Pad2): track 32.4 -> 40.2 mm, vias 3 -> 4
- net Net-(Q3-Pad3): track 21.4 -> 13.7 mm, vias 5 -> 4
- net Net-(Q15-Pad2): track 9.24 -> 1.82 mm, vias 2 -> 0
- net Net-(Q7-Pad2): track 8.94 -> 1.81 mm, vias 2 -> 0
- net Net-(Q18-Pad2): track 14.0 -> 6.94 mm, vias 2 -> 0
- net Net-(Q8-Pad2): track 8.67 -> 1.89 mm, vias 2 -> 0
- net Net-(Q6-Pad2): track 14.2 -> 7.45 mm, vias 2 -> 0
- net Net-(D6-Pad1): track 12.3 -> 6.62 mm, vias 3 -> 0
- net Net-(D5-Pad1): track 7.24 -> 1.73 mm, vias 2 -> 0
- net Net-(C12-Pad1): track 23.8 -> 19.6 mm, vias 5 -> 4
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Other:
- board text added: "Pre-Amp Symetrical Discret V1a Michael Schenk 2020.12.22"
- board text removed: "Pre-Amp Symetrical Discret V1 Michael Schenk 2020.11.05"

Commit message: WIP
Parts:
- moved R20 6.81 mm to (144.5, 108.1)
- moved R23 6.80 mm to (147.9, 108.1)
- moved R6 5.48 mm to (148.1, 136.9)
- moved R3 5.44 mm to (141.8, 136.9)
- moved Q4 3.05 mm to (148.7, 133.1)
- moved Q14 2.77 mm to (143.7, 111.8)
- moved Q16 2.71 mm to (148.7, 111.8)
- moved Q2 2.17 mm to (142.8, 133.2)
- moved Q13 2.16 mm to (142.7, 115.3)
- moved Q17 2.09 mm to (148.7, 115.3)
- moved Q5 1.45 mm to (148.7, 129.4)
- moved Q1 1.42 mm to (142.8, 129.4)
- moved R21 1.37 mm to (143.7, 119.0)
- moved R24 1.33 mm to (147.8, 119.0)
- moved R2 0.39 mm to (143.7, 125.7)
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Routing:
- net Net-(C7-Pad2): track 40.2 -> 18.2 mm, vias 4 -> 2
- net Net-(C2-Pad1): track 28.1 -> 9.08 mm, vias 2 -> 0
- net -15V: track 96.4 -> 109.6 mm
- net +15V: track 101.9 -> 113.7 mm
- net Net-(C12-Pad2): track 39.4 -> 30.1 mm, vias 3 -> 1
- net Net-(Q2-Pad1): track 8.73 -> 0.00 mm
- net Net-(Q3-Pad3): track 13.7 -> 6.68 mm, vias 4 -> 2
- net Net-(Q2-Pad2): track 6.99 -> 0.00 mm, vias 2 -> 0
- net Net-(Q4-Pad2): track 4.99 -> 0.00 mm, vias 2 -> 0
- net Net-(Q1-Pad2): track 4.70 -> 0.00 mm, vias 2 -> 0
- net Net-(Q16-Pad2): track 5.78 -> 1.74 mm, vias 2 -> 0
- net Net-(Q14-Pad2): track 5.82 -> 1.89 mm, vias 2 -> 0
- net Net-(Q15-Pad3): track 10.6 -> 6.74 mm, vias 3 -> 2
- net Net-(Q5-Pad2): track 2.78 -> 0.00 mm
- net Net-(C17-Pad2): track 38.5 -> 37.4 mm
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
Commit message: WIP
Parts:
- added C18: 220uF, Capacitor_THT:CP_Radial_D8.0mm_P3.50mm, F.Cu at (164.9, 100.3)
- added C19: 220uF, Capacitor_THT:CP_Radial_D8.0mm_P3.50mm, F.Cu at (162.6, 139.8)
- moved C15 13.0 mm to (147.9, 101.7), turned to 180 degrees
- moved C16 8.75 mm to (143.0, 143.3), turned to 0 degrees
- moved C13 1.60 mm to (152.2, 105.3)
Routing:
- net Net-(C7-Pad2): track 18.2 -> 39.2 mm, vias 2 -> 4
- net Net-(Q15-Pad3): track 6.74 -> 26.1 mm, vias 2 -> 5
- net Net-(Q3-Pad3): track 6.68 -> 25.9 mm, vias 2 -> 5
- net Net-(C2-Pad1): track 9.08 -> 24.4 mm, vias 0 -> 2
- net +15V: track 113.7 -> 100.2 mm
- net -15V: track 109.6 -> 98.4 mm
- net Net-(Q2-Pad1): track 0.00 -> 8.96 mm, vias 0 -> 2
- net Net-(C12-Pad2): track 30.1 -> 35.8 mm, vias 1 -> 3
- net Net-(Q2-Pad2): track 0.00 -> 3.71 mm
- net Net-(Q1-Pad2): track 0.00 -> 3.66 mm
- net Net-(Q4-Pad2): track 0.00 -> 2.47 mm
- net Net-(Q5-Pad2): track 0.00 -> 1.69 mm

Commit message: Finish 1
Parts:
- moved C8 8.96 mm to (188.8, 113.1), turned to 180 degrees
- moved C10 7.16 mm to (188.8, 130.8)
- moved Q12 6.79 mm to (184.3, 137.8), turned to 90 degrees
- moved C9 6.50 mm to (191.7, 107.8), turned to 0 degrees
- moved R16 6.12 mm to (187.3, 138.6), turned to 90 degrees
- moved R19 5.39 mm to (184.4, 140.6)
- moved C11 4.43 mm to (192.3, 137.9), turned to 180 degrees
- moved R14 2.96 mm to (188.8, 106.6)
- moved R18 2.94 mm to (187.8, 103.7)
- moved Q11 2.70 mm to (185.9, 106.5)
- moved C3 2.41 mm to (178.2, 139.9)
Routing:
- net Net-(C8-Pad1): track 13.6 -> 18.0 mm
- net -15V: track 98.4 -> 101.7 mm
- net +15V: track 100.2 -> 97.3 mm
- net Net-(C10-Pad2): track 20.1 -> 19.1 mm
- net Net-(C9-Pad1): track 5.11 -> 5.77 mm
- net Net-(C11-Pad2): track 6.60 -> 6.09 mm, vias 1 -> 0
