File: lv-lownoise-psu-v3c/lv-lownoise-psu.sch (KiCad schematic (older format))
At the start: 50 parts, among them J1 AC, J10 GND, J11 GND, J12 -5V, J2 GND, J3 AC, J4 +15V, J5 GND, J6 -15V, J7 LED, J8 GND, J9 +5V, Q1 BD679, Q2 BD680, U1 L78L05_SOT89, U2 L79L05_SOT89, U3 LT3045xMSE, U4 LT3094xMSE

Commit message: Finalize 3c design and layout
Parts:
- removed C7, C9: 10u, Capacitor_SMD:C_1210_3225Metric_Pad1.33x2.70mm_HandSolder, symbol Device:C
- removed D1: DF06M, Diode_THT:Diode_Bridge_DIP-4_W7.62mm_P5.08mm, symbol Diode_Bridge:DF06M
- removed U1: L78L05_SOT89, Package_TO_SOT_SMD:SOT-89-3, symbol Regulator_Linear:L78L05_SOT89
- removed U2: L79L05_SOT89, Package_TO_SOT_SMD:SOT-89-3, symbol Regulator_Linear:L79L05_SOT89
- added C15, C16, C7, C9: 4.7uF, Capacitor_Tantalum_SMD:CP_EIA-2012-12_Kemet-R_Pad1.30x1.05mm_HandSolder, symbol Device:CP
- added C17, C18: 47uF, Capacitor_Tantalum_SMD:CP_EIA-7343-31_Kemet-D_Pad2.25x2.55mm_HandSolder, symbol Device:CP
- added D1, D2, D3, D4: BYG20D, Diode_SMD:D_SMA_Handsoldering, symbol Device:D
- added U1: LM7805_TO220, Package_TO_SOT_THT:TO-220-3_Vertical, symbol Regulator_Linear:LM7805_TO220
- added U2: LM7905_TO220, Package_TO_SOT_THT:TO-220-3_Vertical, symbol Regulator_Linear:LM7905_TO220
- C3, C4: value 4.7u -> 10nF; footprint Capacitor_SMD:C_1206_3216Metric_Pad1.33x1.80mm_HandSolder -> Capacitor_SMD:C_0805_2012Metric_Pad1.18x1.45mm_HandSolder
- C5, C6: value 0.47u -> 10nF
Connections:
- net GND: now also C15.2, C16.1, C17.2, C18.1, C7.2, C9.1, U1.2 (GND), U2.1 (GND); no longer C3.2, C4.1, C5.2, C6.1
- net at R1.1, RV1.1, U3.8 (SET): now also C15.1; no longer C5.1
- net at Q1.1 (E), R9.2, U3.1 (IN)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: now also C7.1; no longer C3.1
- net at J1.1 (Pin_1): now also C3.1, C5.1, D1.1 (K), D3.2 (A)
- net at J3.1 (Pin_1): now also C4.2, C6.2, D2.1 (K), D4.2 (A)
- net at C1.1, Q1.2 (C), R4.2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: now also C5.2, C6.1, D3.1 (K), D4.1 (K)
- net at J4.1 (Pin_1), U3.10 (OUTS), U3.11 (OUT)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: now also C17.1
- net at J6.1 (Pin_1), U4.10 (OUTS), U4.11 (OUT)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: now also C18.2
- net at C2.2, Q2.2 (C), R10.1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: now also C3.2, C4.1, D1.2 (A), D2.2 (A)
- net at Q2.1 (E), R11.1, U4.1 (IN)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: now also C9.2; no longer C4.2
- net at R2.2, RV2.1, U4.8 (SET): now also C16.2; no longer C6.2
- net at C11.1, C13.1, J9.1 (Pin_1)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: now also U1.3 (VO)
- net at C8.1, R4.1, R9.1: now also U1.1 (VI)
- net at C12.2, C14.2, J12.1 (Pin_1): now also U2.3 (VO)
- net at C10.2, R10.2, R11.2: now also U2.2 (VI)
Other:
- moved on the sheet: C1, C10, C11, C12, C13, C14, C2, C8, J10, J11, J12, J4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
