File: pre-amp-ECC88-v1/pre-amp-ecc88.kicad_pcb (KiCad board)
At the start: 2 copper layers, 1 part, among them T1 ECC88

Commit message: WIP
Parts:
- added C1: 3.3uF, Capacitor_THT:C_Rect_L7.2mm_W7.2mm_P5.00mm_FKS2_FKP2_MKS2_MKP2, F.Cu at (61.0, 120.0)
- added C2: 100nF, Capacitor_THT:C_Rect_L16.5mm_W5.0mm_P15.00mm_MKT, F.Cu at (113.7, 139.1)
- added C3: 100uF, Capacitor_THT:CP_Radial_D18.0mm_P7.50mm, F.Cu at (99.1, 143.5)
- added C4: 2.2uF, Capacitor_THT:C_Rect_L31.5mm_W9.0mm_P27.50mm_MKS4, F.Cu at (146.9, 119.4)
- added C5: 3.3uF, Capacitor_THT:C_Rect_L7.2mm_W7.2mm_P5.00mm_FKS2_FKP2_MKS2_MKP2, F.Cu at (60.3, 94.0)
- added C6: 100nF, Capacitor_THT:C_Rect_L16.5mm_W5.0mm_P15.00mm_MKT, F.Cu at (128.9, 94.6)
- added C7: 100uF, Capacitor_THT:CP_Radial_D18.0mm_P7.50mm, F.Cu at (115.6, 98.4)
- added C8: 2.2uF, Capacitor_THT:C_Rect_L31.5mm_W9.0mm_P27.50mm_MKS4, F.Cu at (152.4, 74.3)
- added H1: MountingHole, MountingHole:MountingHole_3.2mm_M3, F.Cu at (96.5, 183.5)
- added H2: MountingHole, MountingHole:MountingHole_3.2mm_M3, F.Cu at (121.9, 188.0)
- added H3: MountingHole, MountingHole:MountingHole_3.2mm_M3, F.Cu at (161.9, 182.2)
- added H4: MountingHole, MountingHole:MountingHole_3.2mm_M3, F.Cu at (144.8, 184.8)
- added J1: Conn_01x01, Connector_Pin:Pin_D1.0mm_L10.0mm, F.Cu at (44.5, 93.3)
- added J10: Conn_01x01, Connector_Pin:Pin_D1.3mm_L11.0mm, F.Cu at (81.3, 64.8)
- added J11: Conn_01x01, Connector_Pin:Pin_D1.0mm_L10.0mm, F.Cu at (163.2, 74.3)
- added J12: Conn_01x01, Connector_Pin:Pin_D1.0mm_L10.0mm, F.Cu at (163.2, 81.9)
- added J2: Conn_01x01, Connector_Pin:Pin_D1.0mm_L10.0mm, F.Cu at (44.5, 102.2)
- added J3: Conn_01x01, Connector_Pin:Pin_D1.0mm_L10.0mm, F.Cu at (49.5, 120.0)
- added J4: Conn_01x01, Connector_Pin:Pin_D1.0mm_L10.0mm, F.Cu at (49.5, 129.5)
- added J5: Conn_01x01, Connector_Pin:Pin_D1.3mm_L11.0mm, F.Cu at (108.6, 65.4)
- added J6: Conn_01x01, Connector_Pin:Pin_D1.3mm_L11.0mm, F.Cu at (101.0, 65.4)
- added J7: Conn_01x01, Connector_Pin:Pin_D1.0mm_L10.0mm, F.Cu at (154.3, 119.4)
- added J8: Conn_01x01, Connector_Pin:Pin_D1.0mm_L10.0mm, F.Cu at (154.3, 128.3)
- added J9: Conn_01x01, Connector_Pin:Pin_D1.3mm_L11.0mm, F.Cu at (88.3, 65.4)
- added R1: 1Meg, Resistor_SMD:R_MELF_MMB-0207, F.Cu at (61.0, 129.4)
- added R10: 1Meg, Resistor_SMD:R_MELF_MMB-0207, F.Cu at (60.3, 102.9)
- added R11: 47k, Resistor_SMD:R_MELF_MMB-0207, F.Cu at (70.4, 93.3)
- added R12: 1.21k, Resistor_SMD:R_MiniMELF_MMA-0204, F.Cu at (84.0, 100.3)
- added R13: 56k, Resistor_SMD:R_MELF_MMB-0207, F.Cu at (118.7, 88.2)
- added R14: 39k, Resistor_SMD:R_MELF_MMB-0207, F.Cu at (112.4, 88.2)
- added R15: 100k, Resistor_SMD:R_MELF_MMB-0207, F.Cu at (74.3, 83.9)
- added R16: 56k, Resistor_SMD:R_MELF_MMB-0207, F.Cu at (117.5, 73.1)
- added R17: 39k, Resistor_SMD:R_MELF_MMB-0207, F.Cu at (111.8, 73.1)
- added R18: 1Meg, Resistor_SMD:R_MELF_MMB-0207, F.Cu at (153.0, 85.1)
- added R2: 47k, Resistor_SMD:R_MELF_MMB-0207, F.Cu at (75.7, 119.4)
- added R3: 1.21k, Resistor_SMD:R_MiniMELF_MMA-0204, F.Cu at (82.5, 135.9)
- added R4: 56k, Resistor_SMD:R_MELF_MMB-0207, F.Cu at (121.3, 131.4)
- added R5: 39k, Resistor_SMD:R_MELF_MMB-0207, F.Cu at (110.5, 130.7)
- added R6: 100k, Resistor_SMD:R_MELF_MMB-0207, F.Cu at (78.1, 111.2)
- added R7: 56k, Resistor_SMD:R_MELF_MMB-0207, F.Cu at (113.0, 116.8)
- added R8: 39k, Resistor_SMD:R_MELF_MMB-0207, F.Cu at (108.6, 116.8)
- added R9: 1Meg, Resistor_SMD:R_MELF_MMB-0207, F.Cu at (146.7, 129.0)
- added T2: ECC88, w_vacuum:socket_gzc9-b, F.Cu at (96.5, 88.3)
- moved T1 56.5 mm to (93.3, 122.6), turned to 180 degrees
Connections:
- T1 pad 1: (no net) -> Net-(R4-Pad2)
- T1 pad 2: (no net) -> Net-(R2-Pad1)
- T1 pad 3: (no net) -> Net-(R3-Pad1)
- T1 pad 4: (no net) -> GND
- T1 pad 5: (no net) -> VDDF
- T1 pad 6: (no net) -> VDDA
- T1 pad 7: (no net) -> Net-(R4-Pad2)
- T1 pad 8: (no net) -> Net-(C4-Pad2)
- T1 pad 9: (no net) -> GND
Routing:
- added copper zone on F.Cu, net GND
Other:
- board outline added: 189.2 x 105.4 mm

Commit message: WIP
Parts:
- added C10: 2200uF, Capacitor_THT:CP_Radial_D16.0mm_P7.50mm, F.Cu at (73.7, 151.1)
- added C11: 100nF, Capacitor_THT:C_Rect_L7.2mm_W2.5mm_P5.00mm_FKS2_FKP2_MKS2_MKP2, F.Cu at (84.5, 111.8)
- added C12: 2200uF, Capacitor_THT:CP_Radial_D16.0mm_P7.50mm, F.Cu at (73.7, 111.8)
- added C9: 100nF, Capacitor_THT:C_Rect_L7.2mm_W2.5mm_P5.00mm_FKS2_FKP2_MKS2_MKP2, F.Cu at (84.5, 151.1)
- moved H2 83.6 mm to (43.8, 158.1)
- moved C6 42.1 mm to (90.4, 111.8), turned to 0 degrees
- moved C2 26.1 mm to (90.2, 150.5), turned to 0 degrees
- moved H3 26.0 mm to (162.6, 156.2)
- moved R6 20.5 mm to (70.5, 130.3)
- moved R14 19.4 mm to (99.1, 102.3)
- moved R13 19.0 mm to (106.0, 102.3)
- moved R4 18.4 mm to (106.0, 141.7)
- moved R2 17.7 mm to (64.0, 132.7)
- moved T1 16.1 mm to (84.4, 136.0)
- moved C3 15.9 mm to (114.9, 144.1), turned to 0 degrees
- moved R5 15.8 mm to (99.1, 141.7)
- moved T2 14.7 mm to (84.4, 96.6)
- moved C1 14.5 mm to (54.0, 132.7)
- moved R12 14.4 mm to (69.6, 100.3), turned to 180 degrees
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Routing:
- net Net-(R2-Pad1): track 0.00 -> 8.51 mm
- net Net-(C1-Pad1): track 0.00 -> 7.62 mm
- net Net-(C1-Pad2): track 0.00 -> 5.16 mm
- net Net-(R3-Pad1): track 0.00 -> 3.81 mm

Commit message: Update pre-amp-ecc88.kicad_pcb
Parts:
- moved R17 22.2 mm to (99.1, 91.3)
- moved R16 21.5 mm to (106.0, 91.3)
- moved C8 19.2 mm to (139.9, 88.9)
- moved C4 3.61 mm to (139.9, 128.9)
Changed lines of the file:
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@@
   )
   (module Resistor_SMD:R_MELF_MMB-0207 (layer F.Cu)
-    (at 111.76 73.115 270)
+    (at 99.06 91.35 270)
     (descr "Resistor, MELF, MMB-0207, http://www.vishay.com/docs/28713/melfprof.pdf")
     (tags "MELF Resistor")
@@
   )
   (module Resistor_SMD:R_MELF_MMB-0207 (layer F.Cu)
-    (at 117.475 73.115 270)
+    (at 106.045 91.35 270)
     (descr "Resistor, MELF, MMB-0207, http://www.vishay.com/docs/28713/melfprof.pdf")
     (tags "MELF Resistor")
@@
   )
   (module Capacitor_THT:C_Rect_L31.5mm_W9.0mm_P27.50mm_MKS4 (layer F.Cu)
-    (at 152.4 74.295 180)
+    (at 139.895 88.9 180)
     (descr "C, Rect series, Radial, pin pitch=27.50mm, , length*width=31.5*9mm^2, Capacitor, http://www.wima.com/EN/WIMA_MKS_4.pdf")
     (tags "C Rect series Radial pin pitch 27.50mm  length 31.5mm width 9mm Capacitor")
@@
   )
   (module Capacitor_THT:C_Rect_L31.5mm_W9.0mm_P27.50mm_MKS4 (layer F.Cu)
-    (at 143.51 128.905 180)
+    (at 139.895 128.905 180)
     (descr "C, Rect series, Radial, pin pitch=27.50mm, , length*width=31.5*9mm^2, Capacitor, http://www.wima.com/EN/WIMA_MKS_4.pdf")
     (tags "C Rect series Radial pin pitch 27.50mm  length 31.5mm width 9mm Capacitor")

Commit message: Update pre-amp-ecc88.kicad_pcb
Parts:
- moved H1 119.6 mm to (43.8, 76.2)
- moved H4 108.9 mm to (152.4, 76.2)
- moved J12 20.6 mm to (151.8, 99.1)
- moved J8 20.2 mm to (151.8, 120.0)
- moved J11 18.5 mm to (151.8, 88.9)
- moved J5 14.8 mm to (118.7, 76.2)
- moved J10 14.1 mm to (73.0, 76.2)
- moved J6 13.6 mm to (109.2, 76.2)
- moved J9 10.8 mm to (87.6, 76.2)
- moved H3 10.3 mm to (152.4, 158.1)
- moved R18 9.86 mm to (145.4, 91.3)
- moved J7 3.81 mm to (151.8, 128.9)
- moved R9 2.54 mm to (145.4, 131.4)
- moved R12 0.64 mm to (69.6, 99.7)
Routing:
- net VDDA: track 0.00 -> 137.5 mm
- net VDDF: track 0.00 -> 107.5 mm
- net Net-(C8-Pad2): track 0.00 -> 20.4 mm
- net Net-(C4-Pad2): track 0.00 -> 20.1 mm
- net Net-(R4-Pad2): track 0.00 -> 12.2 mm
- net Net-(R13-Pad2): track 0.00 -> 12.2 mm
- net Net-(C8-Pad1): track 0.00 -> 11.9 mm
- net Net-(C4-Pad1): track 0.00 -> 11.9 mm
- net Net-(R11-Pad1): track 0.00 -> 8.51 mm
- net Net-(C5-Pad1): track 0.00 -> 7.70 mm
- net Net-(C5-Pad2): track 0.00 -> 4.45 mm
- net Net-(R12-Pad1): track 0.00 -> 3.81 mm
Other:
- board size 189.2 x 105.4 mm -> 118.7 x 92.1 mm
Changed lines of the file:
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@@
     (thickness 1.6)
     (drawings 4)
-    (tracks 7)
+    (tracks 59)
     (zones 0)
     (modules 48)
@@
   )
   (module Resistor_SMD:R_MELF_MMB-0207 (layer F.Cu)
-    (at 153.035 85.09 270)
+    (at 145.415 91.35 270)
     (descr "Resistor, MELF, MMB-0207, http://www.vishay.com/docs/28713/melfprof.pdf")
     (tags "MELF Resistor")
@@
   )
   (module Resistor_SMD:R_MiniMELF_MMA-0204 (layer F.Cu)
-    (at 69.62 100.33 180)
+    (at 69.62 99.695 180)
     (descr "Resistor, MiniMELF, MMA-0204, http://www.vishay.com/docs/28713/melfprof.pdf")
     (tags "MiniMELF Resistor")
@@
   )
   (module Connector_Pin:Pin_D1.0mm_L10.0mm (layer F.Cu)
-    (at 163.195 81.915)
+    (at 151.765 99.06)
     (descr "solder Pin_ diameter 1.0mm, hole diameter 1.0mm (press fit), length 10.0mm")
     (tags "solder Pin_ press fit")
@@
   )
   (module Connector_Pin:Pin_D1.0mm_L10.0mm (layer F.Cu)
-    (at 163.195 74.295)
+    (at 151.765 88.9)
     (descr "solder Pin_ diameter 1.0mm, hole diameter 1.0mm (press fit), length 10.0mm")
     (tags "solder Pin_ press fit")
@@
   )
   (module Connector_Pin:Pin_D1.3mm_L11.0mm (layer F.Cu)
-    (at 81.28 64.77)
+    (at 73.025 76.2)
     (descr "solder Pin_ diameter 1.3mm, hole diameter 1.3mm, length 11.0mm")
     (tags "solder Pin_ pressfit")
@@
   )
   (module Connector_Pin:Pin_D1.3mm_L11.0mm (layer F.Cu)
-    (at 88.265 65.405)
+    (at 87.63 76.2)
     (descr "solder Pin_ diameter 1.3mm, hole diameter 1.3mm, length 11.0mm")
     (tags "solder Pin_ pressfit")
@@
   )
   (module Resistor_SMD:R_MELF_MMB-0207 (layer F.Cu)
-    (at 147.955 131.355 270)
+    (at 145.415 131.355 270)
     (descr "Resistor, MELF, MMB-0207, http://www.vishay.com/docs/28713/melfprof.pdf")
     (tags "MELF Resistor")
@@
   )
   (module Connector_Pin:Pin_D1.0mm_L10.0mm (layer F.Cu)
-    (at 156.21 139.7)
+    (at 151.765 120.015)
     (descr "solder Pin_ diameter 1.0mm, hole diameter 1.0mm (press fit), length 10.0mm")
     (tags "solder Pin_ press fit")
@@
   )
   (module Connector_Pin:Pin_D1.0mm_L10.0mm (layer F.Cu)
-    (at 155.575 128.905)
+    (at 151.765 128.905)
     (descr "solder Pin_ diameter 1.0mm, hole diameter 1.0mm (press fit), length 10.0mm")
     (tags "solder Pin_ press fit")
@@
   )
   (module Connector_Pin:Pin_D1.3mm_L11.0mm (layer F.Cu)
-    (at 100.965 65.405)
+    (at 109.22 76.2)
     (descr "solder Pin_ diameter 1.3mm, hole diameter 1.3mm, length 11.0mm")
     (tags "solder Pin_ pressfit")
@@
   )
   (module Connector_Pin:Pin_D1.3mm_L11.0mm (layer F.Cu)
-    (at 108.585 65.405)
+    (at 118.745 76.2)
     (descr "solder Pin_ diameter 1.3mm, hole diameter 1.3mm, length 11.0mm")
     (tags "solder Pin_ pressfit")
@@
   )
   (module MountingHole:MountingHole_3.2mm_M3 (layer F.Cu)
-    (at 144.78 184.785)
+    (at 152.4 76.2)
     (descr "Mounting Hole 3.2mm, no annular, M3")
     (tags "mounting hole 3.2mm no annular m3")
@@
   )
   (module MountingHole:MountingHole_3.2mm_M3 (layer F.Cu)
-    (at 162.56 156.21)
+    (at 152.4 158.115)
     (descr "Mounting Hole 3.2mm, no annular, M3")
     (tags "mounting hole 3.2mm no annular m3")
@@
   )
   (module MountingHole:MountingHole_3.2mm_M3 (layer F.Cu)
-    (at 96.52 183.515)
+    (at 43.815 76.2)
     (descr "Mounting Hole 3.2mm, no annular, M3")
     (tags "mounting hole 3.2mm no annular m3")
@@
     )
   )
-  (gr_line (start 227.965 57.785) (end 227.965 163.195) (layer Edge.Cuts) (width 0.1))
-  (gr_line (start 38.735 57.785) (end 227.965 57.785) (layer Edge.Cuts) (width 0.1))
-  (gr_line (start 38.735 163.195) (end 38.735 57.785) (layer Edge.Cuts) (width 0.1))
-  (gr_line (start 227.965 163.195) (end 38.735 163.195) (layer Edge.Cuts) (width 0.1))
+  (gr_line (start 157.48 71.12) (end 157.48 163.195) (layer Edge.Cuts) (width 0.1))
+  (gr_line (start 38.735 71.12) (end 157.48 71.12) (layer Edge.Cuts) (width 0.1))
+  (gr_line (start 38.735 163.195) (end 38.735 71.12) (layer Edge.Cuts) (width 0.1))
+  (gr_line (start 157.48 163.195) (end 38.735 163.195) (layer Edge.Cuts) (width 0.1))
   (segment (start 43.815 132.715) (end 48.975 132.715) (width 0.5) (layer B.Cu) (net 1))
   (segment (start 53.975 132.715) (end 57.785 132.715) (width 0.5) (layer F.Cu) (net 2))
   (segment (start 57.785 132.715) (end 61.595 132.715) (width 0.5) (layer F.Cu) (net 2))
+  (segment (start 118.745 140.335) (end 114.935 144.145) (width 1) (layer B.Cu) (net 4))
+  (segment (start 115.57 104.775) (end 118.745 101.6) (width 1) (layer B.Cu) (net 4))
+  (segment (start 118.745 101.6) (end 118.745 140.335) (width 1) (layer B.Cu) (net 4))
+  (segment (start 114.935 104.775) (end 115.57 104.775) (width 1) (layer B.Cu) (net 4))
+  (segment (start 118.745 101.6) (end 118.745 76.2) (width 1) (layer B.Cu) (net 4))
+  (segment (start 90.41 104.79148) (end 90.31732 104.6988) (width 1) (layer B.Cu) (net 4))
+  (segment (start 90.41 111.76) (end 90.41 104.79148) (width 1) (layer B.Cu) (net 4))
+  (segment (start 90.17 144.21612) (end 90.31732 144.0688) (width 1) (layer B.Cu) (net 4))
+  (segment (start 90.17 150.495) (end 90.17 144.21612) (width 1) (layer B.Cu) (net 4))
+  (segment (start 114.935 144.145) (end 106.045 144.145) (width 1) (layer F.Cu) (net 4))
+  (segment (start 106.045 144.145) (end 99.06 144.145) (width 1) (layer F.Cu) (net 4))
+  (segment (start 90.39352 144.145) (end 90.31732 144.0688) (width 1) (layer F.Cu) (net 4))
+  (segment (start 99.06 144.145) (end 90.39352 144.145) (width 1) (layer F.Cu) (net 4))
+  (segment (start 114.935 104.775) (end 106.045 104.775) (width 1) (layer F.Cu) (net 4))
+  (segment (start 106.045 104.775) (end 99.06 104.775) (width 1) (layer F.Cu) (net 4))
+  (segment (start 90.39352 104.775) (end 90.31732 104.6988) (width 1) (layer F.Cu) (net 4))
+  (segment (start 99.06 104.775) (end 90.39352 104.775) (width 1) (layer F.Cu) (net 4))
+  (segment (start 97.93732 128.905) (end 99.06 128.905) (width 0.5) (layer F.Cu) (net 5))
+  (segment (start 93.94952 132.8928) (end 97.93732 128.905) (width 0.5) (layer F.Cu) (net 5))
+  (segment (start 99.06 128.905) (end 106.045 128.905) (width 0.5) (layer F.Cu) (net 5))
+  (segment (start 106.045 128.905) (end 112.395 128.905) (width 0.5) (layer F.Cu) (net 5))
+  (segment (start 139.895 128.905) (end 145.415 128.905) (width 0.5) (layer F.Cu) (net 6))
+  (segment (start 145.415 128.905) (end 151.765 128.905) (width 0.5) (layer F.Cu) (net 6))
+  (segment (start 87.63 103.41864) (end 84.43976 106.60888) (width 1) (layer B.Cu) (net 7))
+  (segment (start 87.63 142.78864) (end 84.43976 145.97888) (width 1) (layer B.Cu) (net 7))
+  (segment (start 87.63 103.41864) (end 87.63 142.78864) (width 1) (layer B.Cu) (net 7))
+  (segment (start 84.455 106.62412) (end 84.43976 106.60888) (width 1) (layer B.Cu) (net 7))
+  (segment (start 84.455 111.76) (end 84.455 106.62412) (width 1) (layer B.Cu) (net 7))
+  (segment (start 73.66 111.76) (end 84.455 111.76) (width 1) (layer B.Cu) (net 7))
+  (segment (start 84.455 145.99412) (end 84.43976 145.97888) (width 1) (layer B.Cu) (net 7))
+  (segment (start 84.455 151.13) (end 84.455 145.99412) (width 1) (layer B.Cu) (net 7))
+  (segment (start 73.66 151.13) (end 84.455 151.13) (width 1) (layer B.Cu) (net 7))
+  (segment (start 87.63 103.41864) (end 87.63 76.2) (width 1) (layer B.Cu) (net 7))
   (segment (start 66.495 132.715) (end 70.485 132.715) (width 0.5) (layer F.Cu) (net 8))
   (segment (start 74.7522 132.715) (end 74.93 132.8928) (width 0.5) (layer F.Cu) (net 8))
   (segment (start 70.485 132.715) (end 74.7522 132.715) (width 0.5) (layer F.Cu) (net 8))
   (segment (start 71.12 139.065) (end 74.93 139.065) (width 0.5) (layer F.Cu) (net 9))
+  (segment (start 106.045 139.245) (end 99.06 139.245) (width 0.5) (layer F.Cu) (net 10))
+  (segment (start 94.12952 139.245) (end 93.94952 139.065) (width 0.5) (layer F.Cu) (net 10))
+  (segment (start 99.06 139.245) (end 94.12952 139.245) (width 0.5) (layer F.Cu) (net 10))
+  (segment (start 44.45 93.345) (end 48.895 93.345) (width 0.5) (layer B.Cu) (net 11))
+  (segment (start 53.895 93.345) (end 57.785 93.345) (width 0.5) (layer F.Cu) (net 12))
+  (segment (start 57.785 93.345) (end 61.595 93.345) (width 0.5) (layer F.Cu) (net 12))
+  (segment (start 98.57232 88.9) (end 99.06 88.9) (width 0.5) (layer F.Cu) (net 13))
+  (segment (start 93.94952 93.5228) (end 98.57232 88.9) (width 0.5) (layer F.Cu) (net 13))
+  (segment (start 99.06 88.9) (end 106.045 88.9) (width 0.5) (layer F.Cu) (net 13))
+  (segment (start 106.045 88.9) (end 112.395 88.9) (width 0.5) (layer F.Cu) (net 13))
+  (segment (start 139.895 88.9) (end 145.415 88.9) (width 0.5) (layer F.Cu) (net 14))
+  (segment (start 145.415 88.9) (end 151.765 88.9) (width 0.5) (layer F.Cu) (net 14))
+  (segment (start 66.495 93.345) (end 70.485 93.345) (width 0.5) (layer F.Cu) (net 15))
+  (segment (start 74.7522 93.345) (end 74.93 93.5228) (width 0.5) (layer F.Cu) (net 15))
+  (segment (start 70.485 93.345) (end 74.7522 93.345) (width 0.5) (layer F.Cu) (net 15))
+  (segment (start 71.12 99.695) (end 74.93 99.695) (width 0.5) (layer F.Cu) (net 16))
+  (segment (start 106.045 99.875) (end 99.06 99.875) (width 0.5) (layer F.Cu) (net 17))
+  (segment (start 94.12952 99.875) (end 93.94952 99.695) (width 0.5) (layer F.Cu) (net 17))
+  (segment (start 99.06 99.875) (end 94.12952 99.875) (width 0.5) (layer F.Cu) (net 17))
   (zone (net 3) (net_name GND) (layer F.Cu) (hatch edge 0.508)
     (connect_pads (clearance 0.508))
@@
     (polygon
       (pts
-        (xy 226.695 161.925) (xy 40.005 161.925) (xy 40.005 59.055) (xy 226.695 59.055)
+        (xy 156.21 161.925) (xy 40.005 161.925) (xy 40.005 72.39) (xy 156.21 72.39)
       )
     )
