File: pre-amp-ECC88-v1/pre-amp-ecc88.kicad_pcb (KiCad board)
At the start: 2 copper layers, 118.7 x 92.1 mm, 48 parts, among them J1 Conn_01x01, J10 Conn_01x01, J11 Conn_01x01, J12 Conn_01x01, J2 Conn_01x01, J3 Conn_01x01, J4 Conn_01x01, J5 Conn_01x01, J6 Conn_01x01, J7 Conn_01x01, J8 Conn_01x01, J9 Conn_01x01, T1 ECC88, T2 ECC88

Commit message: WIP
Parts:
- moved J10 5.08 mm to (78.1, 76.2)
- moved J2 0.90 mm to (43.8, 102.9)
- moved J1 0.64 mm to (43.8, 93.3)
- moved J12 0.64 mm to (151.8, 98.4)
- moved J8 0.64 mm to (151.8, 119.4)
Routing:
- net Net-(C8-Pad1): track 11.9 -> 86.9 mm, vias 0 -> 5
- net Net-(C4-Pad1): track 11.9 -> 85.9 mm, vias 0 -> 5
- net Net-(R4-Pad2): track 12.2 -> 35.7 mm, vias 0 -> 1
- net Net-(R13-Pad2): track 12.2 -> 35.7 mm, vias 0 -> 1
- net Net-(C5-Pad2): track 4.45 -> 5.08 mm
Other:
- board text added: "+200VDC"
- board text added: "+6.3VDC"
- board text added: "ECC88 Tube Pre-Amp V1 Michael Schenk 2021.01.19"
- board text added: "GND"
- board text added: "IN"
- board text added: "OUT"
- board text added: "michaelschenk72@gmail.com"
Changed lines of the file:
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@@
   (general
     (thickness 1.6)
-    (drawings 4)
-    (tracks 59)
+    (drawings 18)
+    (tracks 96)
     (zones 0)
     (modules 48)
@@
     (via_min_size 0.4)
     (via_min_drill 0.3)
+    (user_via 1 0.5)
     (uvia_size 0.3)
     (uvia_drill 0.1)
@@
   )
   (module Connector_Pin:Pin_D1.0mm_L10.0mm (layer F.Cu)
-    (at 151.765 99.06)
+    (at 151.765 98.425)
     (descr "solder Pin_ diameter 1.0mm, hole diameter 1.0mm (press fit), length 10.0mm")
     (tags "solder Pin_ press fit")
@@
   )
   (module Connector_Pin:Pin_D1.3mm_L11.0mm (layer F.Cu)
-    (at 73.025 76.2)
+    (at 78.105 76.2)
     (descr "solder Pin_ diameter 1.3mm, hole diameter 1.3mm, length 11.0mm")
     (tags "solder Pin_ pressfit")
@@
   )
   (module Connector_Pin:Pin_D1.0mm_L10.0mm (layer F.Cu)
-    (at 44.45 102.235)
+    (at 43.815 102.87)
     (descr "solder Pin_ diameter 1.0mm, hole diameter 1.0mm (press fit), length 10.0mm")
     (tags "solder Pin_ press fit")
@@
   )
   (module Connector_Pin:Pin_D1.0mm_L10.0mm (layer F.Cu)
-    (at 44.45 93.345)
+    (at 43.815 93.345)
     (descr "solder Pin_ diameter 1.0mm, hole diameter 1.0mm (press fit), length 10.0mm")
     (tags "solder Pin_ press fit")
@@
   )
   (module Connector_Pin:Pin_D1.0mm_L10.0mm (layer F.Cu)
-    (at 151.765 120.015)
+    (at 151.765 119.38)
     (descr "solder Pin_ diameter 1.0mm, hole diameter 1.0mm (press fit), length 10.0mm")
     (tags "solder Pin_ press fit")
@@
     )
   )
+  (gr_text GND (at 78.105 73.025 180) (layer F.SilkS)
+    (effects (font (size 1 1) (thickness 0.15)))
+  )
+  (gr_text GND (at 109.22 73.025 180) (layer F.SilkS)
+    (effects (font (size 1 1) (thickness 0.15)))
+  )
+  (gr_text +6.3VDC (at 87.63 73.025 180) (layer F.SilkS)
+    (effects (font (size 1 1) (thickness 0.15)))
+  )
+  (gr_text +200VDC (at 118.745 73.025 180) (layer F.SilkS)
+    (effects (font (size 1 1) (thickness 0.15)))
+  )
+  (gr_text OUT (at 154.94 88.9 90) (layer F.SilkS)
+    (effects (font (size 1 1) (thickness 0.15)))
+  )
+  (gr_text OUT (at 154.94 128.905 90) (layer F.SilkS)
+    (effects (font (size 1 1) (thickness 0.15)))
+  )
+  (gr_text GND (at 154.94 119.38 90) (layer F.SilkS)
+    (effects (font (size 1 1) (thickness 0.15)))
+  )
+  (gr_text GND (at 154.94 98.425 90) (layer F.SilkS)
+    (effects (font (size 1 1) (thickness 0.15)))
+  )
+  (gr_text GND (at 41.275 102.235 270) (layer F.SilkS)
+    (effects (font (size 1 1) (thickness 0.15)))
+  )
+  (gr_text GND (at 41.275 123.19 270) (layer F.SilkS)
+    (effects (font (size 1 1) (thickness 0.15)))
+  )
+  (gr_text IN (at 41.275 132.715 270) (layer F.SilkS)
+    (effects (font (size 1 1) (thickness 0.15)))
+  )
+  (gr_text IN (at 41.275 93.345 270) (layer F.SilkS)
+    (effects (font (size 1 1) (thickness 0.15)))
+  )
+  (gr_text "ECC88 Tube Pre-Amp\nV1\nMichael Schenk\n2021.01.19" (at 137.16 156.845) (layer F.SilkS)
+    (effects (font (size 1 1) (thickness 0.15)))
+  )
+  (gr_text michaelschenk72@gmail.com (at 105.41 159.385) (layer F.SilkS)
+    (effects (font (size 1 1) (thickness 0.15)))
+  )
   (gr_line (start 157.48 71.12) (end 157.48 163.195) (layer Edge.Cuts) (width 0.1))
   (gr_line (start 38.735 71.12) (end 157.48 71.12) (layer Edge.Cuts) (width 0.1))
@@
   (segment (start 139.895 128.905) (end 145.415 128.905) (width 0.5) (layer F.Cu) (net 6))
   (segment (start 145.415 128.905) (end 151.765 128.905) (width 0.5) (layer F.Cu) (net 6))
+  (segment (start 139.895 128.905) (end 135.255 124.265) (width 0.5) (layer B.Cu) (net 6))
+  (via (at 121.285 124.46) (size 1) (drill 0.5) (layers F.Cu B.Cu) (net 6))
+  (segment (start 121.48 124.265) (end 121.285 124.46) (width 0.5) (layer B.Cu) (net 6))
+  (segment (start 135.255 124.265) (end 121.48 124.265) (width 0.5) (layer B.Cu) (net 6))
+  (via (at 116.205 124.46) (size 1) (drill 0.5) (layers F.Cu B.Cu) (net 6))
+  (segment (start 121.285 124.46) (end 116.205 124.46) (width 0.5) (layer F.Cu) (net 6))
+  (via (at 90.17 124.46) (size 1) (drill 0.5) (layers F.Cu B.Cu) (net 6))
+  (segment (start 116.205 124.46) (end 90.17 124.46) (width 0.5) (layer B.Cu) (net 6))
+  (via (at 85.09 124.46) (size 1) (drill 0.5) (layers F.Cu B.Cu) (net 6))
+  (segment (start 90.17 124.46) (end 85.09 124.46) (width 0.5) (layer F.Cu) (net 6))
+  (via (at 70.485 125.73) (size 1) (drill 0.5) (layers F.Cu B.Cu) (net 6))
+  (segment (start 71.755 124.46) (end 70.485 125.73) (width 0.5) (layer B.Cu) (net 6))
+  (segment (start 85.09 124.46) (end 71.755 124.46) (width 0.5) (layer B.Cu) (net 6))
+  (segment (start 70.485 125.73) (end 70.485 127.815) (width 0.5) (layer F.Cu) (net 6))
   (segment (start 87.63 103.41864) (end 84.43976 106.60888) (width 1) (layer B.Cu) (net 7))
   (segment (start 87.63 142.78864) (end 84.43976 145.97888) (width 1) (layer B.Cu) (net 7))
@@
   (segment (start 94.12952 139.245) (end 93.94952 139.065) (width 0.5) (layer F.Cu) (net 10))
   (segment (start 99.06 139.245) (end 94.12952 139.245) (width 0.5) (layer F.Cu) (net 10))
-  (segment (start 44.45 93.345) (end 48.895 93.345) (width 0.5) (layer B.Cu) (net 11))
+  (via (at 84.455 139.065) (size 1) (drill 0.5) (layers F.Cu B.Cu) (net 10))
+  (segment (start 93.94952 139.065) (end 84.455 139.065) (width 0.5) (layer F.Cu) (net 10))
+  (segment (start 78.5622 133.879306) (end 78.5622 127.889) (width 0.5) (layer B.Cu) (net 10))
+  (segment (start 83.747894 139.065) (end 78.5622 133.879306) (width 0.5) (layer B.Cu) (net 10))
+  (segment (start 84.455 139.065) (end 83.747894 139.065) (width 0.5) (layer B.Cu) (net 10))
+  (segment (start 43.815 93.345) (end 48.895 93.345) (width 0.5) (layer B.Cu) (net 11))
   (segment (start 53.895 93.345) (end 57.785 93.345) (width 0.5) (layer F.Cu) (net 12))
   (segment (start 57.785 93.345) (end 61.595 93.345) (width 0.5) (layer F.Cu) (net 12))
@@
   (segment (start 139.895 88.9) (end 145.415 88.9) (width 0.5) (layer F.Cu) (net 14))
   (segment (start 145.415 88.9) (end 151.765 88.9) (width 0.5) (layer F.Cu) (net 14))
+  (segment (start 139.895 88.9) (end 134.815 83.82) (width 0.5) (layer B.Cu) (net 14))
+  (via (at 121.285 83.82) (size 1) (drill 0.5) (layers F.Cu B.Cu) (net 14))
+  (segment (start 134.815 83.82) (end 121.285 83.82) (width 0.5) (layer B.Cu) (net 14))
+  (via (at 116.205 83.82) (size 1) (drill 0.5) (layers F.Cu B.Cu) (net 14))
+  (segment (start 121.285 83.82) (end 116.205 83.82) (width 0.5) (layer F.Cu) (net 14))
+  (via (at 90.17 83.82) (size 1) (drill 0.5) (layers F.Cu B.Cu) (net 14))
+  (segment (start 116.205 83.82) (end 90.17 83.82) (width 0.5) (layer B.Cu) (net 14))
+  (via (at 84.455 83.82) (size 1) (drill 0.5) (layers F.Cu B.Cu) (net 14))
+  (segment (start 90.17 83.82) (end 84.455 83.82) (width 0.5) (layer F.Cu) (net 14))
+  (via (at 70.485 85.725) (size 1) (drill 0.5) (layers F.Cu B.Cu) (net 14))
+  (segment (start 72.39 83.82) (end 70.485 85.725) (width 0.5) (layer B.Cu) (net 14))
+  (segment (start 84.455 83.82) (end 72.39 83.82) (width 0.5) (layer B.Cu) (net 14))
+  (segment (start 70.485 85.725) (end 70.485 88.445) (width 0.5) (layer F.Cu) (net 14))
   (segment (start 66.495 93.345) (end 70.485 93.345) (width 0.5) (layer F.Cu) (net 15))
   (segment (start 74.7522 93.345) (end 74.93 93.5228) (width 0.5) (layer F.Cu) (net 15))
@@
   (segment (start 94.12952 99.875) (end 93.94952 99.695) (width 0.5) (layer F.Cu) (net 17))
   (segment (start 99.06 99.875) (end 94.12952 99.875) (width 0.5) (layer F.Cu) (net 17))
+  (via (at 84.455 99.695) (size 1) (drill 0.5) (layers F.Cu B.Cu) (net 17))
+  (segment (start 93.94952 99.695) (end 84.455 99.695) (width 0.5) (layer F.Cu) (net 17))
+  (segment (start 78.5622 94.509306) (end 78.5622 88.519) (width 0.5) (layer B.Cu) (net 17))
+  (segment (start 83.747894 99.695) (end 78.5622 94.509306) (width 0.5) (layer B.Cu) (net 17))
+  (segment (start 84.455 99.695) (end 83.747894 99.695) (width 0.5) (layer B.Cu) (net 17))
   (zone (net 3) (net_name GND) (layer F.Cu) (hatch edge 0.508)
     (connect_pads (clearance 0.508))
