File: pre-amp-discret-elektor-v1/pre-amp-discret.kicad_pcb (KiCad board)
At the start: 2 copper layers, 81.9 x 52.1 mm, 66 parts, among them J1 Conn_01x01, J2 Conn_01x01, J3 Conn_01x01, J4 Conn_01x01, J5 Conn_01x01, J6 Conn_01x01, J7 Conn_01x01, Q1 BCM857DS,115, Q10 BC860C, Q11 BCM847DS,115, Q13 BCM847DS,115, Q14 BCM857DS,115, Q18 BC860C, Q19 BC860C, Q2 BCM847DS,115, Q20 BC850C, Q3 BCM857DS,115, Q6 BC850C, Q7 BC860C, Q8 BC850C, Q9 BCM857DS,115

Commit message: WIP
Parts:
- removed Q10, Q18, Q19: BC860C, Package_TO_SOT_SMD:SOT-23
- removed Q14: BCM857DS,115, Package_SO:SC-74-6_1.5x2.9mm_P0.95mm
- removed Q20: BC850C, Package_TO_SOT_SMD:SOT-23
- added C10: 2.2uF, Capacitor_THT:C_Rect_L7.2mm_W7.2mm_P5.00mm_FKS2_FKP2_MKS2_MKP2, F.Cu at (145.8, 171.6)
- added C11: 100nF, Capacitor_SMD:C_0805_2012Metric_Pad1.18x1.45mm_HandSolder, F.Cu at (146.4, 178.4)
- added C20: 2.2uF, Capacitor_THT:C_Rect_L7.2mm_W7.2mm_P5.00mm_FKS2_FKP2_MKS2_MKP2, F.Cu at (134.7, 184.5)
- added C8: 150p, Capacitor_SMD:C_0805_2012Metric_Pad1.18x1.45mm_HandSolder, F.Cu at (162.2, 135.3)
- added C9: 1uF, Capacitor_THT:C_Rect_L7.2mm_W5.5mm_P5.00mm_FKS2_FKP2_MKS2_MKP2, F.Cu at (179.5, 126.2)
- added D1: 1N4148W, Diode_SMD:D_SOD-123, F.Cu at (146.8, 175.3)
- added D2: 1N4148W, Diode_SMD:D_SOD-123, F.Cu at (155.6, 171.2)
- added Q4: BC550C, Package_TO_SOT_THT:TO-92_Inline, F.Cu at (177.4, 113.8)
- added Q5: BC560C, Package_TO_SOT_THT:TO-92_Inline, F.Cu at (179.1, 133.1)
- added R14: 390R, Resistor_SMD:R_0805_2012Metric_Pad1.20x1.40mm_HandSolder, F.Cu at (167.9, 116.7)
- added R16: 10R, Resistor_SMD:R_0805_2012Metric_Pad1.20x1.40mm_HandSolder, F.Cu at (181.3, 117.8)
- added R18: 392k, Resistor_SMD:R_0805_2012Metric_Pad1.20x1.40mm_HandSolder, F.Cu at (152.1, 175.1)
- added R19: 100k, Resistor_SMD:R_0805_2012Metric_Pad1.20x1.40mm_HandSolder, F.Cu at (160.8, 171.0)
- added R31: 475k, Resistor_SMD:R_0805_2012Metric_Pad1.20x1.40mm_HandSolder, F.Cu at (148.7, 184.4)
- added RV1: 10k, Potentiometer_THT:Potentiometer_Bourns_3266W_Vertical, F.Cu at (174.0, 120.9)
- added RV2: 100k, Potentiometer_THT:Potentiometer_Bourns_3266W_Vertical, F.Cu at (140.9, 179.2)
- added U1: OP77, Package_SO:SO-8_3.9x4.9mm_P1.27mm, F.Cu at (181.4, 170.6)
- C17: value 270pF -> 100nF
- C7: value 270pF -> 150p
- Q2: value BCM847DS,115 -> BC850C; footprint Package_SO:SC-74-6_1.5x2.9mm_P0.95mm -> Package_TO_SOT_SMD:SOT-23
- Q6: value BC850C -> BC337-40; footprint Package_TO_SOT_SMD:SOT-23 -> Package_TO_SOT_THT:TO-92_Inline
- Q8: value BC850C -> BC327-40; footprint Package_TO_SOT_SMD:SOT-23 -> Package_TO_SOT_THT:TO-92_Inline
- Q9: value BCM857DS,115 -> BC850C; footprint Package_SO:SC-74-6_1.5x2.9mm_P0.95mm -> Package_TO_SOT_SMD:SOT-23
- R10: value 2k2 -> 10k
- R11, R27: value 39R -> 249R
- R12: value 100R -> 10k
- R15: value 1k -> 390R
- R17: value 47k -> 10R
- R2, R21, R24, R5: value 100R -> 80.6R
- R20, R23, R3, R6: value 68R -> 806R
- R22, R4: value 100R -> 140R
- R26: value 2k2 -> 392k
- R28: value 10k -> 3.9k
- R29: value 47k -> 27k
- R30: value 1k -> 475k
- moved R28 73.7 mm to (148.7, 181.4), turned to 0 degrees
- moved C17 73.2 mm to (144.0, 183.9), turned to 0 degrees
- moved R26 71.4 mm to (152.1, 178.0), turned to 0 degrees
- moved Q9 59.9 mm to (161.4, 174.8), turned to 0 degrees
- moved R29 44.7 mm to (156.8, 174.4), turned to 0 degrees
- moved R30 40.1 mm to (156.8, 177.3), turned to 0 degrees
- moved R17 39.4 mm to (184.7, 126.5), turned to 270 degrees
- moved R15 32.7 mm to (174.1, 126.6), turned to 0 degrees
- moved C5 31.6 mm to (194.8, 155.6)
- moved C4 25.8 mm to (187.7, 86.6)
- moved Q6 25.7 mm to (181.5, 111.2), turned to 270 degrees
- moved R10 25.5 mm to (165.9, 110.1), turned to 0 degrees
- moved Q2 25.5 mm to (171.6, 129.7), turned to 0 degrees
- moved R12 22.2 mm to (164.1, 132.0)
- moved C7 16.0 mm to (166.3, 113.0), turned to 0 degrees
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Connections:
- C17 pad 1: Net-(C17-Pad1) -> GND
- C17 pad 2: Net-(C17-Pad2) -> -15V
- C7 pad 1: Net-(C17-Pad1) -> GND
- Q1 pad 6: Net-(C7-Pad2) -> Net-(Q1-Pad6)
- Q13 pad 6: Net-(C17-Pad2) -> Net-(Q13-Pad6)
- Q2 pad 1: Net-(Q2-Pad1) -> Net-(Q1-Pad6)
- Q2 pad 3: Net-(Q1-Pad3) -> Net-(C9-Pad1)
- Q6 pad 1: Net-(C7-Pad2) -> +15V
- Q6 pad 2: Net-(Q6-Pad2) -> Net-(C9-Pad2)
- Q6 pad 3: GND -> Net-(Q6-Pad3)
- Q7 pad 1: Net-(Q18-Pad2) -> Net-(Q13-Pad6)
- Q7 pad 3: Net-(C17-Pad1) -> Net-(C9-Pad2)
- Q8 pad 1: Net-(Q6-Pad2) -> -15V
- Q8 pad 2: Net-(Q8-Pad2) -> Net-(C9-Pad1)
- Q8 pad 3: Net-(C17-Pad1) -> Net-(Q8-Pad3)
- Q9 pad 3: Net-(Q9-Pad2) -> Net-(Q9-Pad3)
- R10 pad 1: Net-(Q6-Pad2) -> Net-(C9-Pad2)
- R10 pad 2: -15V -> Net-(C7-Pad2)
- R12 pad 1: +15V -> Net-(C8-Pad1)
- R12 pad 2: Net-(Q9-Pad1) -> Net-(Q5-Pad2)
- R15 pad 1: +15V -> Net-(Q5-Pad2)
- R15 pad 2: Net-(Q14-Pad2) -> Net-(C9-Pad1)
- R17 pad 1: Net-(Q13-Pad3) -> Net-(C12-Pad1)
- R17 pad 2: Net-(C17-Pad2) -> Net-(Q8-Pad3)
- R20 pad 2: Net-(Q14-Pad1) -> Net-(Q13-Pad6)
- R23 pad 2: Net-(Q14-Pad4) -> Net-(Q13-Pad3)
- R26 pad 1: +15V -> Net-(C12-Pad2)
- R26 pad 2: Net-(Q18-Pad2) -> Net-(Q9-Pad3)
- R27 pad 1: Net-(Q8-Pad2) -> Net-(Q2-Pad2)
- R28 pad 1: Net-(Q9-Pad2) -> Net-(Q9-Pad1)
- R28 pad 2: GND -> -15V
- R29 pad 1: Net-(Q1-Pad3) -> Net-(C10-Pad1)
- R29 pad 2: Net-(C7-Pad2) -> Net-(Q9-Pad1)
- R3 pad 1: Net-(Q2-Pad1) -> Net-(Q1-Pad6)
- R30 pad 1: Net-(Q2-Pad2) -> Net-(C10-Pad2)
- R30 pad 2: -15V -> GND
- R6 pad 1: Net-(Q2-Pad4) -> Net-(Q1-Pad3)
Routing:
- net Net-(C17-Pad2): track 32.7 -> 0.00 mm, vias 3 -> 0
- net Net-(C7-Pad2): track 28.3 -> 0.00 mm, vias 2 -> 0
- net Net-(C17-Pad1): track 26.5 -> 0.00 mm, vias 4 -> 0
- net Net-(C12-Pad2): track 43.4 -> 17.1 mm, vias 3 -> 2
- net Net-(C12-Pad1): track 20.6 -> 0.12 mm, vias 4 -> 0
- net -15V: track 104.1 -> 87.2 mm, vias 3 -> 1
- net +15V: track 93.4 -> 80.4 mm, vias 3 -> 1
- net Net-(Q13-Pad6): track 0.00 -> 10.00 mm, vias 0 -> 2
- net Net-(Q1-Pad6): track 0.00 -> 8.58 mm, vias 0 -> 1
- net Net-(Q6-Pad2): track 7.45 -> 0.00 mm
- net Net-(Q18-Pad2): track 6.94 -> 0.00 mm
- net Net-(Q9-Pad1): track 6.71 -> 0.00 mm
- net Net-(C6-Pad1): track 3.88 -> 0.00 mm
- net Net-(Q9-Pad2): track 2.99 -> 0.00 mm
- net Net-(J6-Pad1): track 2.65 -> 0.02 mm
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
Commit message: WIP
Parts:
- U1: value OP77 -> OPA188xxDBV; footprint Package_SO:SO-8_3.9x4.9mm_P1.27mm -> Package_TO_SOT_SMD:TSOT-23-5
- moved U1 48.5 mm to (132.8, 169.5)
- moved Q9 43.0 mm to (120.5, 161.4)
- moved R26 34.4 mm to (118.5, 170.6)
- moved R18 34.1 mm to (118.9, 167.3)
- moved R29 29.5 mm to (127.9, 168.5), turned to 180 degrees
- moved C10 22.0 mm to (124.8, 178.3)
- moved C17 20.6 mm to (127.9, 170.9)
- moved RV2 20.4 mm to (121.4, 173.4)
- moved C11 13.2 mm to (138.1, 168.1), turned to 180 degrees
- moved C13 7.50 mm to (146.8, 108.1), turned to 90 degrees
- moved R15 6.20 mm to (167.9, 126.4)
- moved R16 5.10 mm to (186.1, 119.7)
- moved R23 4.76 mm to (144.9, 112.9)
- moved C15 4.65 mm to (138.3, 103.1), turned to 90 degrees
- moved R6 4.23 mm to (145.7, 136.4)
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Connections:
- U1 pad 1: (no net) -> Net-(C10-Pad1)
- U1 pad 2: Net-(C10-Pad2) -> -15V
- U1 pad 4: -15V -> Net-(C10-Pad2)
- U1 pad 5: (no net) -> +15V
Routing:
- net +15V: track 80.4 -> 55.2 mm
- net Net-(Q1-Pad3): track 20.1 -> 0.02 mm, vias 3 -> 0
- net -15V: track 87.2 -> 75.6 mm
- net Net-(Q14-Pad2): track 11.3 -> 0.00 mm
- net Net-(Q13-Pad3): track 15.3 -> 5.35 mm, vias 4 -> 3
- net Net-(Q13-Pad6): track 10.00 -> 1.21 mm, vias 2 -> 1
- net Net-(Q1-Pad6): track 8.58 -> 0.00 mm, vias 1 -> 0
- net Net-(Q2-Pad2): track 8.55 -> 0.00 mm

Commit message: WIP
Parts:
- C10, C20: footprint Capacitor_THT:C_Rect_L7.2mm_W7.2mm_P5.00mm_FKS2_FKP2_MKS2_MKP2 -> Capacitor_SMD:C_1210_3225Metric_Pad1.33x2.70mm_HandSolder
- moved C20 55.0 mm to (162.2, 136.8), turned to 270 degrees
- moved R31 54.4 mm to (163.8, 132.1), turned to 270 degrees
- moved C10 49.6 mm to (146.6, 133.7)
- moved R28 48.5 mm to (140.0, 133.7)
- moved R26 48.0 mm to (138.8, 127.1), turned to 270 degrees
- moved R19 44.3 mm to (134.9, 135.0), turned to 270 degrees
- moved R18 43.8 mm to (136.4, 127.1), turned to 270 degrees
- moved RV2 41.4 mm to (143.5, 138.3)
- moved D1 40.4 mm to (159.3, 136.8), turned to 270 degrees
- moved R29 39.8 mm to (141.2, 131.1)
- moved C17 38.1 mm to (146.9, 137.9), turned to 270 degrees
- moved R30 37.1 mm to (154.1, 140.4), turned to 270 degrees
- moved C11 36.1 mm to (154.2, 135.9), turned to 270 degrees
- moved U1 35.9 mm to (150.7, 138.4)
- moved Q9 33.9 mm to (136.0, 131.2), turned to 270 degrees
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Connections:
- R12 pad 2: Net-(Q5-Pad2) -> Net-(C9-Pad1)
Routing:
- net +15V: track 55.2 -> 77.4 mm, vias 1 -> 0
- net Net-(C9-Pad2): track 0.05 -> 20.6 mm, vias 0 -> 1
- net Net-(C12-Pad1): track 0.12 -> 18.9 mm, vias 0 -> 1
- net Net-(C9-Pad1): track 0.00 -> 17.6 mm
- net Net-(Q5-Pad2): track 0.00 -> 15.7 mm, vias 0 -> 1
- net Net-(Q4-Pad3): track 0.00 -> 14.7 mm
- net Net-(Q11-Pad6): track 21.2 -> 8.09 mm
- net Net-(Q3-Pad6): track 21.5 -> 9.68 mm
- net Net-(Q4-Pad2): track 0.00 -> 11.0 mm, vias 0 -> 2
- net Net-(Q8-Pad3): track 0.00 -> 9.90 mm, vias 0 -> 1
- net Net-(C12-Pad2): track 17.1 -> 25.9 mm, vias 2 -> 3
- net -15V: track 75.6 -> 83.9 mm
- net Net-(C2-Pad2): track 8.29 -> 0.00 mm
- net Net-(Q6-Pad3): track 0.00 -> 7.56 mm, vias 0 -> 1
- net Net-(J6-Pad1): track 0.02 -> 2.60 mm
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Other:
- board text added: "Pre-Amp Elektor V1 Michael Schenk 2021.01.24"
- board text removed: "Pre-Amp Symetrical Discret V2 Michael Schenk 2021.01.02"

Commit message: Update pre-amp-discret.kicad_pcb
Parts:
- moved D2 29.3 mm to (158.6, 110.9), turned to 90 degrees
- moved D1 26.0 mm to (161.4, 110.9)
- moved C20 25.9 mm to (164.5, 111.0)
- moved R30 23.5 mm to (159.8, 117.6)
- moved U1 23.5 mm to (156.4, 115.6)
- moved C10 23.4 mm to (154.8, 111.8)
- moved C16 23.1 mm to (151.4, 134.9)
- moved C11 22.3 mm to (161.1, 114.7), turned to 180 degrees
- moved C17 21.6 mm to (152.3, 117.0), turned to 0 degrees
- moved R31 16.4 mm to (164.5, 115.7), turned to 90 degrees
- moved C13 9.31 mm to (150.6, 98.4), turned to 270 degrees
- moved C15 8.25 mm to (143.1, 103.4)
- moved R22 6.58 mm to (157.0, 120.8), turned to 270 degrees
- moved R23 4.60 mm to (139.6, 109.5)
- moved R3 4.47 mm to (146.9, 123.4)
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Routing:
- net Net-(Q1-Pad6): track 0.00 -> 32.3 mm, vias 0 -> 2
- net Net-(Q13-Pad6): track 1.21 -> 33.1 mm, vias 1 -> 4
- net Net-(C10-Pad1): track 0.00 -> 28.1 mm, vias 0 -> 3
- net +15V: track 77.4 -> 101.6 mm, vias 0 -> 5
- net Net-(C12-Pad2): track 25.9 -> 49.2 mm, vias 3 -> 4
- net -15V: track 83.9 -> 105.2 mm, vias 1 -> 4
- net Net-(C20-Pad2): track 0.00 -> 13.9 mm
- net Net-(C12-Pad1): track 18.9 -> 32.0 mm, vias 1 -> 3
- net Net-(Q11-Pad6): track 8.09 -> 17.2 mm
- net Net-(C10-Pad2): track 0.00 -> 7.44 mm, vias 0 -> 2
- net Net-(C2-Pad1): track 23.0 -> 29.4 mm, vias 3 -> 4
- net Net-(Q3-Pad6): track 9.68 -> 15.7 mm
- net Net-(C2-Pad2): track 0.00 -> 4.27 mm
- net Net-(Q13-Pad3): track 5.35 -> 2.47 mm, vias 3 -> 0
- net Net-(Q1-Pad3): track 0.02 -> 2.84 mm
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
Commit message: 1. Layout completed
Parts:
- moved RV2 6.51 mm to (138.4, 134.2)
- moved R19 4.40 mm to (133.3, 130.9)
- moved J7 2.70 mm to (190.2, 114.0)
- moved Q9 1.69 mm to (137.6, 130.9)
- moved R29 1.20 mm to (141.6, 129.9)
- moved R28 1.08 mm to (140.6, 132.8), turned to 270 degrees
- moved J6 0.13 mm to (190.2, 121.9)
Routing:
- net -15V: track 105.2 -> 122.6 mm
- net Net-(Q9-Pad3): track 0.00 -> 6.24 mm
- net Net-(Q9-Pad1): track 0.00 -> 4.00 mm
- net Net-(Q9-Pad2): track 0.00 -> 3.31 mm
- net Net-(R19-Pad2): track 0.00 -> 2.32 mm
- net Net-(C10-Pad1): track 28.1 -> 28.3 mm, vias 3 -> 4

Commit message: Ready to create gerber
Parts:
- added C21: 33p, Capacitor_SMD:C_0805_2012Metric_Pad1.18x1.45mm_HandSolder, F.Cu at (137.9, 120.2)
- added R32: 470R, Resistor_SMD:R_0805_2012Metric_Pad1.20x1.40mm_HandSolder, F.Cu at (136.9, 117.2)
- moved R1 1.92 mm to (137.9, 114.3)
- moved C2 1.22 mm to (133.5, 117.2)
Connections:
- Q1 pad 2: Net-(C2-Pad1) -> Net-(C21-Pad2)
- Q13 pad 2: Net-(C2-Pad1) -> Net-(C21-Pad2)
- R1 pad 1: Net-(C2-Pad1) -> Net-(C21-Pad2)
- R18 pad 1: Net-(C2-Pad1) -> Net-(C21-Pad2)
Routing:
- net Net-(C21-Pad2): track 0.00 -> 28.8 mm, vias 0 -> 4
- net Net-(C2-Pad1): track 29.4 -> 2.38 mm, vias 4 -> 0
- net Net-(C2-Pad2): track 4.27 -> 3.05 mm
