File: pre-amp-discret-elektor-v3/pre-amp-discret.kicad_pcb (KiCad board)
At the start: 2 copper layers, 81.9 x 52.1 mm, 64 parts, among them J1 Conn_01x01, J2 Conn_01x01, J3 Conn_01x01, J4 Conn_01x01, J5 Conn_01x01, J6 Conn_01x01, J7 Conn_01x01, Q1 BCM857DS,115, Q11 BCM847DS,115, Q13 BCM847DS,115, Q2 BC850C, Q3 BCM857DS,115, Q4 BC550C, Q5 BC560C, Q6 BC337-40, Q7 BC860C, Q8 BC327-40

Commit message: V3 Layout completed
Parts:
- removed Q13: BCM847DS,115, Package_SO:SC-74-6_1.5x2.9mm_P0.95mm
- Q1: value BCM857DS,115 -> THAT340; footprint Package_SO:SC-74-6_1.5x2.9mm_P0.95mm -> Package_SO:SOIC-14_3.9x8.7mm_P1.27mm
- moved Q1 10.5 mm to (147.1, 121.8)
- moved R6 8.91 mm to (149.6, 132.3)
- moved R23 8.77 mm to (149.6, 111.3)
- moved R5 8.18 mm to (152.7, 124.1), turned to 90 degrees
- moved R24 8.15 mm to (152.7, 119.5), turned to 90 degrees
- moved R2 4.50 mm to (141.6, 124.1), turned to 90 degrees
- moved R21 4.40 mm to (141.6, 119.5), turned to 90 degrees
- moved R20 3.69 mm to (144.7, 111.3)
- moved R3 3.57 mm to (144.7, 132.3)
Connections:
- Q1 pad 4: Net-(Q1-Pad4) -> (no net)
- Q1 pad 5: Net-(C12-Pad2) -> Net-(Q1-Pad5)
- Q1 pad 6: Net-(Q1-Pad6) -> Net-(C21-Pad2)
- Q2 pad 1: Net-(Q1-Pad6) -> Net-(Q1-Pad7)
- Q7 pad 1: Net-(Q13-Pad6) -> Net-(Q1-Pad1)
- R2 pad 2: Net-(Q1-Pad1) -> Net-(Q1-Pad5)
- R20 pad 2: Net-(Q13-Pad6) -> Net-(Q1-Pad1)
- R21 pad 1: Net-(Q13-Pad1) -> Net-(Q1-Pad3)
- R23 pad 2: Net-(Q13-Pad3) -> Net-(Q1-Pad14)
- R24 pad 1: Net-(Q13-Pad4) -> Net-(Q1-Pad12)
- R3 pad 1: Net-(Q1-Pad6) -> Net-(Q1-Pad7)
- R5 pad 2: Net-(Q1-Pad4) -> Net-(Q1-Pad10)
- R6 pad 1: Net-(Q1-Pad3) -> Net-(Q1-Pad8)
Routing:
- net Net-(Q1-Pad1): track 1.78 -> 37.8 mm, vias 0 -> 3
- net Net-(Q1-Pad7): track 0.00 -> 34.5 mm, vias 0 -> 3
- net Net-(Q13-Pad6): track 29.9 -> 0.00 mm, vias 3 -> 0
- net Net-(Q1-Pad6): track 27.4 -> 0.00 mm, vias 2 -> 0
- net Net-(C12-Pad2): track 44.2 -> 26.3 mm
- net Net-(C21-Pad2): track 30.6 -> 17.6 mm
- net Net-(Q1-Pad8): track 0.00 -> 5.73 mm, vias 0 -> 2
- net Net-(Q1-Pad14): track 0.00 -> 5.72 mm, vias 0 -> 2
- net Net-(Q13-Pad1): track 5.14 -> 0.00 mm
- net Net-(Q1-Pad4): track 4.77 -> 0.00 mm
- net Net-(Q1-Pad5): track 0.00 -> 3.05 mm
- net Net-(Q1-Pad12): track 0.00 -> 3.05 mm
- net Net-(Q1-Pad10): track 0.00 -> 3.05 mm
- net Net-(Q13-Pad3): track 2.47 -> 0.00 mm
- net Net-(Q13-Pad4): track 1.95 -> 0.00 mm
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Other:
- board text added: "Pre-Amp Elektor V3 Michael Schenk 2021.02.10"
- board text removed: "Pre-Amp Elektor V2 Michael Schenk 2021.02.10"
