File: hv-power-supply-v1d/hv-power-supply-v1.sch (KiCad schematic (older format))
At the start: 113 parts, among them J1 AC-HV, J10 HV, J11 GND_HV, J12 LED, J13 GND_LED, J14 +5V, J15 GND_5V, J2 AC-HV, J3 EARTH, J4 AC-LV, J5 AC-LV, J6 LV1, J7 GND_LV1, J8 LV2, J9 GND_LV2, Q1 IRF840, Q2 MMBT3904-TP, Q3 MMBT3904-TP, Q4 IRF840, U1 LM4040DBZ-10, U2 LM7805_TO220, U3 LM321, U4 LM317_3PinPackage, U5 LM317_3PinPackage, U6 TLC555CDR

Commit message: WIP
Parts:
- D11, D12: footprint Diode_THT:D_DO-41_SOD81_P10.16mm_Horizontal -> Diode_SMD:D_SOD-123F
Connections:
- net at D9.3, R5.2, U3.1 (+): no longer C20.1
- net at RV1.2, U3.3 (-): now also C20.1
Changed lines of the file:
@@
 	4350 2500 4350 3650
 Wire Wire Line
-	6650 3600 6200 3600
+	6650 3600 6350 3600
 Wire Wire Line
 	6050 2500 6050 3450
@@
 Wire Wire Line
 	6500 3400 6650 3400
-Wire Wire Line
-	6500 3400 6500 2950
-Wire Wire Line
-	6500 2950 7050 2950
-Connection ~ 6500 3400
 $Comp
 L Mechanical:Heatsink HS3
@@
 F 0 "D11" H 8250 5117 50  0000 C CNN
 F 1 "1N4007" H 8250 5026 50  0000 C CNN
-F 2 "Diode_THT:D_DO-41_SOD81_P10.16mm_Horizontal" H 8250 4725 50  0001 C CNN
+F 2 "Diode_SMD:D_SOD-123F" H 8250 4725 50  0001 C CNN
 F 3 "http://www.vishay.com/docs/88503/1n4001.pdf" H 8250 4900 50  0001 C CNN
 	1    8250 4900
@@
 F 0 "D12" H 8250 6717 50  0000 C CNN
 F 1 "1N4007" H 8250 6626 50  0000 C CNN
-F 2 "Diode_THT:D_DO-41_SOD81_P10.16mm_Horizontal" H 8250 6325 50  0001 C CNN
+F 2 "Diode_SMD:D_SOD-123F" H 8250 6325 50  0001 C CNN
 F 3 "http://www.vishay.com/docs/88503/1n4001.pdf" H 8250 6500 50  0001 C CNN
 	1    8250 6500
@@
 Wire Wire Line
 	9050 7750 10350 7750
+Wire Wire Line
+	6350 2950 6350 3600
+Wire Wire Line
+	6350 2950 7050 2950
+Connection ~ 6350 3600
+Wire Wire Line
+	6350 3600 6200 3600
 $EndSCHEMATC

Commit message: WIP
Parts:
- D11, D12: footprint Diode_SMD:D_SOD-123F -> Diode_SMD:D_SMA_Handsoldering
Changed lines of the file:
@@
 F 0 "D11" H 8250 5117 50  0000 C CNN
 F 1 "1N4007" H 8250 5026 50  0000 C CNN
-F 2 "Diode_SMD:D_SOD-123F" H 8250 4725 50  0001 C CNN
+F 2 "Diode_SMD:D_SMA_Handsoldering" H 8250 4725 50  0001 C CNN
 F 3 "http://www.vishay.com/docs/88503/1n4001.pdf" H 8250 4900 50  0001 C CNN
 	1    8250 4900
@@
 F 0 "D12" H 8250 6717 50  0000 C CNN
 F 1 "1N4007" H 8250 6626 50  0000 C CNN
-F 2 "Diode_SMD:D_SOD-123F" H 8250 6325 50  0001 C CNN
+F 2 "Diode_SMD:D_SMA_Handsoldering" H 8250 6325 50  0001 C CNN
 F 3 "http://www.vishay.com/docs/88503/1n4001.pdf" H 8250 6500 50  0001 C CNN
 	1    8250 6500
