File: dac-pcm1702-v1/kicad-asrc-v3/dac.sch (KiCad schematic (older format))
At the start: 99 parts, among them J1 Conn_01x06_Male, J10 B, J11 IN, J12 PORTB, J13 CLK, J14 PORTA, J15 A, J16 +5VIN, J17 GND, J18 I2C2, J2 LED, J3 GND, J4 +5VOUT, J5 GND, J6 IN, J7 I2C1, J8 AC, J9 AC, U1 PLR135-T10, U10 TLV1117-33, U11 TLV1117-18, U2 PLR135-T10, U3 SRC4382/SRC4392, U4 74LVC1G125, U5 PIC16F18446-I/SO, U6 PL133-37TI-R, U7 74LVC1G125, U8 ASDMB-xxxMHz, U9 TLV1117-50

Commit message: WIP
Parts:
- added C? (x2): 33pF, Capacitor_SMD:C_0603_1608Metric_Pad1.08x0.95mm_HandSolder, symbol Device:C
- added JP?: SolderJumper_3_Open, Jumper:SolderJumper-3_P1.3mm_Open_RoundedPad1.0x1.5mm_NumberLabels, symbol Jumper:SolderJumper_3_Open
- added L? (x2): 47uH, Inductor_SMD:L_0805_2012Metric_Pad1.05x1.20mm_HandSolder, symbol Device:L
- R1, R30: value 0R -> NC
Connections:
- net +3V3: now also JP?.3 (B); no longer C3.2, C4.2, U1.1 (VCC), U2.1 (VCC)
- net GND: now also C?.1, C?.1
- net at J11.3 (Pin_3), R1.1, R5.2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: now also C?.2
- net at J11.2 (Pin_2), R30.1, R4.1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: now also C?.2
- net +5V: now reaches C17.1, C18.1, C19.1, C20.1, J4.1 (Pin_1), R10.2, TP2.1, U10.3 (VI), U11.3 (VI), U9.2 (VO)
- net +5V: now also JP?.1 (A)
- new net: C3.2, L?.1, U1.1 (VCC)
- new net: C4.2, L?.1, U2.1 (VCC)
- new net: JP?.2 (C), L?.2, L?.2
Other:
- moved on the sheet: C1, C11, C12, C13, C14, C15, C16, C2, C25, C26, C27, C28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

Commit message: Update dac.sch
Parts:
- gave numbers to parts that had none: 5
Changed lines of the file:
@@
 	13150 8900 13150 8850
 $Comp
-L Device:L L?
+L Device:L L1
 U 1 1 60762620
 P 2000 1700
-F 0 "L?" V 2190 1700 50  0000 C CNN
+F 0 "L1" V 2190 1700 50  0000 C CNN
 F 1 "47uH" V 2099 1700 50  0000 C CNN
 F 2 "Inductor_SMD:L_0805_2012Metric_Pad1.05x1.20mm_HandSolder" H 2000 1700 50  0001 C CNN
@@
 $EndComp
 $Comp
-L Jumper:SolderJumper_3_Open JP?
+L Jumper:SolderJumper_3_Open JP1
 U 1 1 6076422D
 P 2200 4300
-F 0 "JP?" H 2200 4413 50  0000 C CNN
+F 0 "JP1" H 2200 4413 50  0000 C CNN
 F 1 "SolderJumper_3_Open" H 2200 4504 50  0000 C CNN
 F 2 "Jumper:SolderJumper-3_P1.3mm_Open_RoundedPad1.0x1.5mm_NumberLabels" H 2200 4300 50  0001 C CNN
@@
 $EndComp
 $Comp
-L Device:C C?
+L Device:C C29
 U 1 1 607655B6
 P 2600 1650
-F 0 "C?" H 2485 1604 50  0000 R CNN
+F 0 "C29" H 2485 1604 50  0000 R CNN
 F 1 "33pF" H 2485 1695 50  0000 R CNN
 F 2 "Capacitor_SMD:C_0603_1608Metric_Pad1.08x0.95mm_HandSolder" H 2638 1500 50  0001 C CNN
@@
 $EndComp
 $Comp
-L power:+5V #PWR?
+L power:+5V #PWR0103
 U 1 1 607D1DA9
 P 13100 8000
-F 0 "#PWR?" H 13100 7850 50  0001 C CNN
+F 0 "#PWR0103" H 13100 7850 50  0001 C CNN
 F 1 "+5V" H 13115 8173 50  0000 C CNN
 F 2 "" H 13100 8000 50  0001 C CNN
@@
 	13100 8050 13100 8000
 $Comp
-L power:+5V #PWR?
+L power:+5V #PWR0106
 U 1 1 60807BC9
 P 2550 4250
-F 0 "#PWR?" H 2550 4100 50  0001 C CNN
+F 0 "#PWR0106" H 2550 4100 50  0001 C CNN
 F 1 "+5V" H 2565 4423 50  0000 C CNN
 F 2 "" H 2550 4250 50  0001 C CNN
@@
 $EndComp
 $Comp
-L power:+3.3V #PWR?
+L power:+3.3V #PWR0168
 U 1 1 6080881A
 P 1850 4250
-F 0 "#PWR?" H 1850 4100 50  0001 C CNN
+F 0 "#PWR0168" H 1850 4100 50  0001 C CNN
 F 1 "+3.3V" H 1865 4423 50  0000 C CNN
 F 2 "" H 1850 4250 50  0001 C CNN
@@
 $EndComp
 $Comp
-L Device:C C?
+L Device:C C30
 U 1 1 60979B5B
 P 2600 3200
-F 0 "C?" H 2485 3154 50  0000 R CNN
+F 0 "C30" H 2485 3154 50  0000 R CNN
 F 1 "33pF" H 2485 3245 50  0000 R CNN
 F 2 "Capacitor_SMD:C_0603_1608Metric_Pad1.08x0.95mm_HandSolder" H 2638 3050 50  0001 C CNN
@@
 $EndComp
 $Comp
-L power:GND #PWR?
+L power:GND #PWR0169
 U 1 1 6097A1C9
 P 2600 3500
-F 0 "#PWR?" H 2600 3250 50  0001 C CNN
+F 0 "#PWR0169" H 2600 3250 50  0001 C CNN
 F 1 "GND" H 2605 3327 50  0000 C CNN
 F 2 "" H 2600 3500 50  0001 C CNN
@@
 $EndComp
 $Comp
-L power:GND #PWR?
+L power:GND #PWR0170
 U 1 1 6097A869
 P 2600 1950
-F 0 "#PWR?" H 2600 1700 50  0001 C CNN
+F 0 "#PWR0170" H 2600 1700 50  0001 C CNN
 F 1 "GND" H 2605 1777 50  0000 C CNN
 F 2 "" H 2600 1950 50  0001 C CNN
@@
 	2600 3500 2600 3350
 $Comp
-L Device:L L?
+L Device:L L2
 U 1 1 60AFA2C3
 P 2000 3250
-F 0 "L?" V 2190 3250 50  0000 C CNN
+F 0 "L2" V 2190 3250 50  0000 C CNN
 F 1 "47uH" V 2099 3250 50  0000 C CNN
 F 2 "Inductor_SMD:L_0805_2012Metric_Pad1.05x1.20mm_HandSolder" H 2000 3250 50  0001 C CNN
