File: xilinx-cpld-breakout-v1/kicad/xilinx-cpld-breakout.sch (KiCad schematic (older format))
At the start: 3 parts

Commit message: WIP
Parts:
- removed U?: XC2C64A-xVQ44, Package_QFP:TQFP-44_10x10mm_P0.8mm, symbol kicad-snk:XC2C64A-xVQ44
- removed U?: TPS7A2018, Package_TO_SOT_SMD:SOT-23-5, symbol Regulator_Linear:TPS7A0518PDBV
- removed U?: TPS7A0533PDBV, Package_TO_SOT_SMD:SOT-23-5, symbol Regulator_Linear:TPS7A0533PDBV
- added C1, C2, C3, C4: 100nF, Capacitor_SMD:C_0603_1608Metric_Pad1.08x0.95mm_HandSolder, symbol Device:C
- added C5: 10uF, Capacitor_Tantalum_SMD:CP_EIA-3528-21_Kemet-B_Pad1.50x2.35mm_HandSolder, symbol Device:CP
- added C6, C7, C8: 10uF, Capacitor_SMD:C_0805_2012Metric_Pad1.18x1.45mm_HandSolder, symbol Device:CP
- added J1, J3: Conn_01x20_Male, Connector_PinHeader_2.54mm:PinHeader_1x20_P2.54mm_Vertical, symbol Connector:Conn_01x20_Male
- added J8: Conn_01x06_Male, Connector_PinHeader_2.54mm:PinHeader_1x06_P2.54mm_Vertical, symbol Connector:Conn_01x06_Male
- added JP1, JP2: SolderJumper_3_Open, Jumper:SolderJumper-3_P1.3mm_Open_RoundedPad1.0x1.5mm_NumberLabels, symbol Jumper:SolderJumper_3_Open
- added U1: XC2C64A-xVQ44, Package_QFP:TQFP-44_10x10mm_P0.8mm, symbol kicad-snk:XC2C64A-xVQ44
- added U2: TC1185-5.0VCT713, Package_TO_SOT_SMD:SOT-23-5, symbol Regulator_Linear:TC1017-xCT
- added U3: TC1185-1.8VCT713, Package_TO_SOT_SMD:SOT-23-5, symbol Regulator_Linear:TC1017-xCT
- added U4: TC1185-3.3VCT713, Package_TO_SOT_SMD:SOT-23-5, symbol Regulator_Linear:TC1017-xCT
- added U5: CM1293A−04SO, Package_SO:SC-74-6_1.5x2.9mm_P0.95mm, symbol Power_Protection:USBLC6-4SC6
Connections:
- new net: C4.2, JP2.2 (C), U1.26 (VCCIO2)
- new net: C3.2, JP1.2 (C), U1.7 (VCCIO1)
- new net +1V8: C2.2, C7.1, JP1.3 (B), JP2.3 (B), U1.15 (VCC), U3.5 (VOUT)
- new net +3V3: C1.2, C8.1, J8.6 (Pin_6), JP1.1 (A), JP2.1 (A), U1.35 (VCCAUX), U4.5 (VOUT), U5.5 (VBUS)
- new net +5VIN: C5.1, J1.20 (Pin_20), U2.1 (VIN), U2.3 (~SHDN)
- new net +5VOUT: C6.1, J1.19 (Pin_19), U2.5 (VOUT), U3.1 (VIN), U3.3 (~SHDN), U4.1 (VIN), U4.3 (~SHDN)
- new net GND: C1.1, C2.1, C3.1, C4.1, C5.2, C6.2, C7.2, C8.2, J3.20 (Pin_20), J8.5 (Pin_5), U1.17 (GND), U1.25 (GND), U1.4 (GND), U2.2 (GND), U3.2 (GND), U4.2 (GND), U5.2 (GND)
- new net JTAG_TCK: J8.4 (Pin_4), U1.11 (TCK), U5.6 (I/O4)
- new net JTAG_TDI: J8.2 (Pin_2), U1.9 (TDI), U5.3 (I/O2)
- new net JTAG_TDO: J8.3 (Pin_3), U1.24 (TDO), U5.4 (I/O3)
- new net JTAG_TMS: J8.1 (Pin_1), U1.10 (TMS), U5.1 (I/O1)
- new net PIN1-IO1-GCK2: J3.1 (Pin_1), U1.1 (IO1/GCK2)
- new net PIN12-IO1: J3.11 (Pin_11), U1.12 (IO1)
- new net PIN13-IO1: J3.12 (Pin_12), U1.13 (IO1)
- new net PIN14-IO1: J3.13 (Pin_13), U1.14 (IO1)
- new net PIN16-IO1: J3.14 (Pin_14), U1.16 (IO1)
- new net PIN18-IO1: J3.15 (Pin_15), U1.18 (IO2)
- new net PIN19-IO1: J3.16 (Pin_16), U1.19 (IO2)
- new net PIN2-IO1: J3.2 (Pin_2), U1.2 (IO1)
- new net PIN20-IO1: J3.17 (Pin_17), U1.20 (IO2)
- new net PIN21-IO1: J3.18 (Pin_18), U1.21 (IO2)
- new net PIN22-IO1: J3.19 (Pin_19), U1.22 (IO2)
- new net PIN3-IO1: J3.3 (Pin_3), U1.3 (IO1)
- new net PIN33-IO2-GTS0: J1.8 (Pin_8), U1.33 (IO2/GTS0)
- new net PIN34-IO2-GTS1: J1.9 (Pin_9), U1.34 (IO2/GTS1)
- new net PIN36-IO2: J1.10 (Pin_10), U1.36 (IO2)
- new net PIN37-IO2: J1.11 (Pin_11), U1.37 (IO2)
- new net PIN38-IO2: J1.12 (Pin_12), U1.38 (IO2)
- new net PIN39-IO1: J1.13 (Pin_13), U1.39 (IO1)
- new net PIN40-IO1: J1.14 (Pin_14), U1.40 (IO1)
- new net PIN41-IO1: J1.15 (Pin_15), U1.41 (IO1)
- new net PIN42-IO1: J1.16 (Pin_16), U1.42 (IO1)
- new net PIN43-IO1-GCK0: J1.17 (Pin_17), U1.43 (IO1/GCK0)
- new net PIN44-IO1-GCK2: J1.18 (Pin_18), U1.44 (IO1/GCK1)
- new net PIN5-IO1: J3.4 (Pin_4), U1.5 (IO1)
- new net PIN6-IO1: J3.5 (Pin_5), U1.6 (IO1)
- new net PIN8-IO1: J3.6 (Pin_6), U1.8 (IO1)

Commit message: Layout completed
Connections:
- net PIN23-IO2: now reaches U1.23 (IO2)
- net PIN23-IO2: now also J1.1 (Pin_1)
- net PIN27-IO2: now reaches U1.27 (IO2)
- net PIN27-IO2: now also J1.2 (Pin_2)
- net PIN28-IO2: now reaches U1.28 (IO2)
- net PIN28-IO2: now also J1.3 (Pin_3)
- net PIN29-IO2: now reaches U1.29 (IO2)
- net PIN29-IO2: now also J1.4 (Pin_4)
- net PIN30-IO2-GSR: now reaches U1.30 (IO2/GSR)
- net PIN30-IO2-GSR: now also J1.5 (Pin_5)
- net PIN31-IO2-GTS2: now reaches U1.31 (IO2/GTS2)
- net PIN31-IO2-GTS2: now also J1.6 (Pin_6)
- net PIN32-IO2-GTS3: now reaches U1.32 (IO2/GTS3)
- net PIN32-IO2-GTS3: now also J1.7 (Pin_7)
- net PIN18-IO1 renamed PIN18-IO2
- net PIN19-IO1 renamed PIN19-IO2
- net PIN20-IO1 renamed PIN20-IO2
- net PIN21-IO1 renamed PIN21-IO2
- net PIN22-IO1 renamed PIN22-IO2
Changed lines of the file:
@@
 PIN16-IO1
 Text GLabel 3600 5650 2    50   BiDi ~ 0
-PIN18-IO1
+PIN18-IO2
 Text GLabel 3600 5750 2    50   BiDi ~ 0
-PIN19-IO1
+PIN19-IO2
 Text GLabel 3600 5850 2    50   BiDi ~ 0
-PIN20-IO1
+PIN20-IO2
 Text GLabel 3600 5950 2    50   BiDi ~ 0
-PIN21-IO1
+PIN21-IO2
 Text GLabel 3600 6050 2    50   BiDi ~ 0
-PIN22-IO1
+PIN22-IO2
 Wire Wire Line
 	1700 6950 1950 6950
@@
 	9250 3200 9500 3200
 Text GLabel 9250 3300 0    50   BiDi ~ 0
-PIN18-IO1
+PIN18-IO2
 Text GLabel 9250 3400 0    50   BiDi ~ 0
-PIN19-IO1
+PIN19-IO2
 Text GLabel 9250 3500 0    50   BiDi ~ 0
-PIN20-IO1
+PIN20-IO2
 Text GLabel 9250 3600 0    50   BiDi ~ 0
-PIN21-IO1
+PIN21-IO2
 Text GLabel 9250 3700 0    50   BiDi ~ 0
-PIN22-IO1
+PIN22-IO2
 Wire Wire Line
 	9500 3300 9250 3300
@@
 Wire Wire Line
 	9250 6350 9500 6350
+Text GLabel 3600 6850 2    50   BiDi ~ 0
+PIN32-IO2-GTS3
+Wire Wire Line
+	3600 6850 3350 6850
+Text GLabel 9250 5250 0    50   BiDi ~ 0
+PIN32-IO2-GTS3
+Text GLabel 3600 6750 2    50   BiDi ~ 0
+PIN31-IO2-GTS2
+Text GLabel 3600 6650 2    50   BiDi ~ 0
+PIN30-IO2-GSR
+Wire Wire Line
+	3600 6750 3350 6750
+Wire Wire Line
+	3600 6650 3350 6650
+Text GLabel 9250 5150 0    50   BiDi ~ 0
+PIN31-IO2-GTS2
+Text GLabel 9250 5050 0    50   BiDi ~ 0
+PIN30-IO2-GSR
+Wire Wire Line
+	9250 5150 9500 5150
+Wire Wire Line
+	9250 5050 9500 5050
+Wire Wire Line
+	9250 5250 9500 5250
+Text GLabel 3600 6450 2    50   BiDi ~ 0
+PIN29-IO2
+Text GLabel 3600 6350 2    50   BiDi ~ 0
+PIN28-IO2
+Text GLabel 3600 6250 2    50   BiDi ~ 0
+PIN27-IO2
+Text GLabel 3600 6150 2    50   BiDi ~ 0
+PIN23-IO2
+Wire Wire Line
+	3600 6150 3350 6150
+Wire Wire Line
+	3350 6250 3600 6250
+Wire Wire Line
+	3600 6350 3350 6350
+Wire Wire Line
+	3350 6450 3600 6450
+Text GLabel 9250 4950 0    50   BiDi ~ 0
+PIN29-IO2
+Text GLabel 9250 4850 0    50   BiDi ~ 0
+PIN28-IO2
+Text GLabel 9250 4750 0    50   BiDi ~ 0
+PIN27-IO2
+Text GLabel 9250 4650 0    50   BiDi ~ 0
+PIN23-IO2
+Wire Wire Line
+	9250 4650 9500 4650
+Wire Wire Line
+	9500 4750 9250 4750
+Wire Wire Line
+	9250 4850 9500 4850
+Wire Wire Line
+	9500 4950 9250 4950
 $EndSCHEMATC
