File: hv-psu-discrete/kicad/v1g/hv-power-supply-v1.sch (KiCad schematic (older format))
At the start: 100 parts, among them J1 AC-HV, J10 HV, J11 GND_HV, J12 LED, J13 GND_LED, J14 +5V, J15 GND_5V, J2 AC-HV, J3 EARTH, J4 AC-LV, J5 AC-LV, J6 LV1, J7 GND_LV1, Q1 IRF840, Q2 MMBT3904-TP, Q3 MMBT3904-TP, Q4 IRF840, U1 LM4040DBZ-10, U2 LM7805_TO220, U3 OPA188xxDBV, U4 LM317_3PinPackage, U6 TLC555CDR

Commit message: wip
Parts:
- removed D12: 1N4007, Diode_SMD:D_SMA_Handsoldering, symbol Diode:1N4007
- Q1: value IRF840 -> IPN50R3K0CE; footprint Package_TO_SOT_THT:TO-220-3_Vertical -> Package_TO_SOT_SMD:SOT-223-3_TabPin2
Changed lines of the file:
@@
 Sheet 1 1
 Title "Discrete HV Supply"
-Date "2021-07-17"
-Rev "V1f"
+Date "2021-07-20"
+Rev "V1g"
 Comp ""
 Comment1 ""
@@
 P 9000 3500
 F 0 "Q1" H 9108 3553 60  0000 L CNN
-F 1 "IRF840" H 9108 3447 60  0000 L CNN
-F 2 "Package_TO_SOT_THT:TO-220-3_Vertical" H 9200 3700 60  0001 L CNN
+F 1 "IPN50R3K0CE" H 9108 3447 60  0000 L CNN
+F 2 "Package_TO_SOT_SMD:SOT-223-3_TabPin2" H 9200 3700 60  0001 L CNN
 F 3 "http://www.vishay.com/docs/91015/sihf510.pdf" H 9200 3800 60  0001 L CNN
 F 4 "IRF510PBF-ND" H 9200 3900 60  0001 L CNN "Digi-Key_PN"
@@
 Wire Wire Line
 	3800 5250 3800 8500
-$Comp
-L Diode:1N4007 D12
-U 1 1 60EA1E2D
-P 13400 2600
-F 0 "D12" H 13400 2817 50  0000 C CNN
-F 1 "1N4007" H 13400 2726 50  0000 C CNN
-F 2 "Diode_SMD:D_SMA_Handsoldering" H 13400 2425 50  0001 C CNN
-F 3 "http://www.vishay.com/docs/88503/1n4001.pdf" H 13400 2600 50  0001 C CNN
-	1    13400 2600
-	0    1    1    0
-$EndComp
-Wire Wire Line
-	13400 3550 13400 2750
-Wire Wire Line
-	13400 2450 13400 1600
-Wire Wire Line
-	13400 1600 12650 1600
-Connection ~ 12650 1600
 Wire Wire Line
 	5900 8500 6250 8500

Commit message: Update hv-power-supply-v1.sch
Parts:
- Q1: value IPN50R3K0CE -> FQT1N60CTF
Changed lines of the file:
@@
 P 11500 2900
 F 0 "Q3" H 11688 2953 60  0000 L CNN
-F 1 "MMBT3904-TP" H 11688 2847 60  0000 L CNN
+F 1 "MMBT3904-TP" H 11650 3050 60  0000 L CNN
 F 2 "Package_TO_SOT_SMD:SOT-23" H 11700 3100 60  0001 L CNN
 F 3 "https://www.mccsemi.com/pdf/Products/MMBT3904(SOT-23).pdf" H 11700 3200 60  0001 L CNN
@@
 U 1 1 603EDCB9
 P 9000 3500
-F 0 "Q1" H 9108 3553 60  0000 L CNN
-F 1 "IPN50R3K0CE" H 9108 3447 60  0000 L CNN
+F 0 "Q1" H 9150 3650 60  0000 L CNN
+F 1 "FQT1N60CTF" H 9150 3350 60  0000 L CNN
 F 2 "Package_TO_SOT_SMD:SOT-223-3_TabPin2" H 9200 3700 60  0001 L CNN
 F 3 "http://www.vishay.com/docs/91015/sihf510.pdf" H 9200 3800 60  0001 L CNN
