File: pre-amp-discret/kicad/v6/pre-amp-discret.sch (KiCad schematic (older format))
At the start: 52 parts, among them J1 Conn_01x01, J2 Conn_01x01, J3 Conn_01x01, J4 Conn_01x01, J5 Conn_01x01, J6 Conn_01x01, J7 Conn_01x01, Q1 BCM857DS,115, Q10 BC860C, Q2 BCM847DS,115, Q3 BC860C, Q4 BC860C, Q6 BC850C, Q7 BC860C, Q8 BC850C, Q9 BC860C, U1 OPA188xxDBV

Commit message: Finalize v6 and create gerber
Parts:
- removed C1, C3: 220uF, Capacitor_THT:CP_Radial_D8.0mm_P3.50mm, symbol Device:CP
- added C1, C3: 100nF, Capacitor_SMD:C_1210_3225Metric_Pad1.33x2.70mm_HandSolder, symbol Device:C
- C10, C6: footprint Capacitor_SMD:C_0805_2012Metric_Pad1.18x1.45mm_HandSolder -> Capacitor_SMD:C_1210_3225Metric_Pad1.33x2.70mm_HandSolder
- C13, C14, C4, C5: footprint Capacitor_THT:C_Rect_L7.2mm_W2.5mm_P5.00mm_FKS2_FKP2_MKS2_MKP2 -> Capacitor_SMD:C_1210_3225Metric_Pad1.33x2.70mm_HandSolder
- C15, C16: value 220uF -> 10uF/25V; footprint Capacitor_THT:CP_Radial_D8.0mm_P3.50mm -> Capacitor_SMD:CP_Elec_6.3x5.8
Connections:
- net +15V: now also C3.2
- net -15V: now also C1.1
- net GND: now also C1.2, C3.1
Changed lines of the file:
@@
 encoding utf-8
 Sheet 1 1
-Title "Discrete Pre-Amp"
-Date "2021-05-19"
-Rev "V5"
+Title "Discrete Pre-Amp Servo"
+Date "2021-07-28"
+Rev "V6"
 Comp ""
 Comment1 ""
@@
 L power:+15V #PWR05
 U 1 1 5F8542B0
-P 1250 1050
-F 0 "#PWR05" H 1250 900 50  0001 C CNN
-F 1 "+15V" H 1265 1223 50  0000 C CNN
-F 2 "" H 1250 1050 50  0001 C CNN
-F 3 "" H 1250 1050 50  0001 C CNN
-	1    1250 1050
+P 1750 1050
+F 0 "#PWR05" H 1750 900 50  0001 C CNN
+F 1 "+15V" H 1765 1223 50  0000 C CNN
+F 2 "" H 1750 1050 50  0001 C CNN
+F 3 "" H 1750 1050 50  0001 C CNN
+	1    1750 1050
 	1    0    0    -1
 $EndComp
@@
 L power:-15V #PWR08
 U 1 1 5F85C667
-P 1250 6900
-F 0 "#PWR08" H 1250 7000 50  0001 C CNN
-F 1 "-15V" H 1265 7073 50  0000 C CNN
-F 2 "" H 1250 6900 50  0001 C CNN
-F 3 "" H 1250 6900 50  0001 C CNN
-	1    1250 6900
+P 1750 6750
+F 0 "#PWR08" H 1750 6850 50  0001 C CNN
+F 1 "-15V" H 1765 6923 50  0000 C CNN
+F 2 "" H 1750 6750 50  0001 C CNN
+F 3 "" H 1750 6750 50  0001 C CNN
+	1    1750 6750
 	-1   0    0    1
 $EndComp
@@
 $EndComp
 $Comp
-L Device:CP C3
-U 1 1 5F86C1B0
-P 1250 6250
-F 0 "C3" H 1368 6296 50  0000 L CNN
-F 1 "220uF" H 1368 6205 50  0000 L CNN
-F 2 "Capacitor_THT:CP_Radial_D8.0mm_P3.50mm" H 1288 6100 50  0001 C CNN
-F 3 "~" H 1250 6250 50  0001 C CNN
-	1    1250 6250
-	1    0    0    -1
-$EndComp
-$Comp
-L power:GND #PWR07
-U 1 1 5F870D74
-P 1250 6000
-F 0 "#PWR07" H 1250 5750 50  0001 C CNN
-F 1 "GND" H 1255 5827 50  0000 C CNN
-F 2 "" H 1250 6000 50  0001 C CNN
-F 3 "" H 1250 6000 50  0001 C CNN
-	1    1250 6000
-	-1   0    0    1
-$EndComp
-$Comp
 L power:GND #PWR011
 U 1 1 5F8716F0
@@
 Wire Wire Line
 	1750 6700 1750 6400
-Wire Wire Line
-	1250 6700 1250 6400
-Wire Wire Line
-	1250 6900 1250 6700
-Connection ~ 1250 6700
-Wire Wire Line
-	1250 6100 1250 6000
 Wire Wire Line
 	1750 6100 1750 6000
@@
 	0    1    1    0
 $EndComp
-Wire Wire Line
-	1250 1100 1250 1050
-$Comp
-L Device:CP C1
-U 1 1 5F87FECA
-P 1250 1450
-F 0 "C1" H 1368 1496 50  0000 L CNN
-F 1 "220uF" H 1368 1405 50  0000 L CNN
-F 2 "Capacitor_THT:CP_Radial_D8.0mm_P3.50mm" H 1288 1300 50  0001 C CNN
-F 3 "~" H 1250 1450 50  0001 C CNN
-	1    1250 1450
-	1    0    0    -1
-$EndComp
-$Comp
-L power:GND #PWR06
-U 1 1 5F88163E
-P 1250 1750
-F 0 "#PWR06" H 1250 1500 50  0001 C CNN
-F 1 "GND" H 1255 1577 50  0000 C CNN
-F 2 "" H 1250 1750 50  0001 C CNN
-F 3 "" H 1250 1750 50  0001 C CNN
-	1    1250 1750
-	1    0    0    -1
-$EndComp
 $Comp
 L power:GND #PWR010
@@
 	7000 4650 7000 4800
 Wire Wire Line
-	1250 1300 1250 1100
-Connection ~ 1250 1100
-Wire Wire Line
 	1750 1300 1750 1100
 Wire Wire Line
 	1750 1750 1750 1600
-Connection ~ 1750 1100
-Wire Wire Line
-	1250 1100 1750 1100
-Connection ~ 1750 6700
 Wire Wire Line
 	1750 6700 2300 6700
-Wire Wire Line
-	1250 6700 1750 6700
-Wire Wire Line
-	1250 1600 1250 1750
 Wire Wire Line
 	4950 5850 4950 6100
@@
 F 0 "C13" H 7085 1404 50  0000 R CNN
 F 1 "100nF" H 7085 1495 50  0000 R CNN
-F 2 "Capacitor_THT:C_Rect_L7.2mm_W2.5mm_P5.00mm_FKS2_FKP2_MKS2_MKP2" H 7238 1300 50  0001 C CNN
+F 2 "Capacitor_SMD:C_1210_3225Metric_Pad1.33x2.70mm_HandSolder" H 7238 1300 50  0001 C CNN
 F 3 "~" H 7200 1450 50  0001 C CNN
 	1    7200 1450
@@
 F 0 "C4" H 1635 1404 50  0000 R CNN
 F 1 "100nF" H 1635 1495 50  0000 R CNN
-F 2 "Capacitor_THT:C_Rect_L7.2mm_W2.5mm_P5.00mm_FKS2_FKP2_MKS2_MKP2" H 1788 1300 50  0001 C CNN
+F 2 "Capacitor_SMD:C_1210_3225Metric_Pad1.33x2.70mm_HandSolder" H 1788 1300 50  0001 C CNN
 F 3 "~" H 1750 1450 50  0001 C CNN
 	1    1750 1450
@@
 F 0 "C14" H 7085 6204 50  0000 R CNN
 F 1 "100nF" H 7085 6295 50  0000 R CNN
-F 2 "Capacitor_THT:C_Rect_L7.2mm_W2.5mm_P5.00mm_FKS2_FKP2_MKS2_MKP2" H 7238 6100 50  0001 C CNN
+F 2 "Capacitor_SMD:C_1210_3225Metric_Pad1.33x2.70mm_HandSolder" H 7238 6100 50  0001 C CNN
 F 3 "~" H 7200 6250 50  0001 C CNN
 	1    7200 6250
@@
 F 0 "C5" H 1635 6204 50  0000 R CNN
 F 1 "100nF" H 1635 6295 50  0000 R CNN
-F 2 "Capacitor_THT:C_Rect_L7.2mm_W2.5mm_P5.00mm_FKS2_FKP2_MKS2_MKP2" H 1788 6100 50  0001 C CNN
+F 2 "Capacitor_SMD:C_1210_3225Metric_Pad1.33x2.70mm_HandSolder" H 1788 6100 50  0001 C CNN
 F 3 "~" H 1750 6250 50  0001 C CNN
 	1    1750 6250
@@
 P 7700 1450
 F 0 "C15" H 7818 1496 50  0000 L CNN
-F 1 "220uF" H 7818 1405 50  0000 L CNN
-F 2 "Capacitor_THT:CP_Radial_D8.0mm_P3.50mm" H 7738 1300 50  0001 C CNN
+F 1 "10uF/25V" H 7818 1405 50  0000 L CNN
+F 2 "Capacitor_SMD:CP_Elec_6.3x5.8" H 7738 1300 50  0001 C CNN
 F 3 "~" H 7700 1450 50  0001 C CNN
 	1    7700 1450
@@
 P 7700 6250
 F 0 "C16" H 7818 6296 50  0000 L CNN
-F 1 "220uF" H 7818 6205 50  0000 L CNN
-F 2 "Capacitor_THT:CP_Radial_D8.0mm_P3.50mm" H 7738 6100 50  0001 C CNN
+F 1 "10uF/25V" H 7818 6205 50  0000 L CNN
+F 2 "Capacitor_SMD:CP_Elec_6.3x5.8" H 7738 6100 50  0001 C CNN
 F 3 "~" H 7700 6250 50  0001 C CNN
 	1    7700 6250
@@
 F 0 "C10" H 13585 8504 50  0000 R CNN
 F 1 "1uF" H 13585 8595 50  0000 R CNN
-F 2 "Capacitor_SMD:C_0805_2012Metric_Pad1.18x1.45mm_HandSolder" H 13738 8400 50  0001 C CNN
+F 2 "Capacitor_SMD:C_1210_3225Metric_Pad1.33x2.70mm_HandSolder" H 13738 8400 50  0001 C CNN
 F 3 "~" H 13700 8550 50  0001 C CNN
 	1    13700 8550
@@
 F 0 "C6" H 11585 8504 50  0000 R CNN
 F 1 "1uF" H 11585 8595 50  0000 R CNN
-F 2 "Capacitor_SMD:C_0805_2012Metric_Pad1.18x1.45mm_HandSolder" H 11738 8400 50  0001 C CNN
+F 2 "Capacitor_SMD:C_1210_3225Metric_Pad1.33x2.70mm_HandSolder" H 11738 8400 50  0001 C CNN
 F 3 "~" H 11700 8550 50  0001 C CNN
 	1    11700 8550
@@
 	2300 5450 2300 5550
 Wire Wire Line
-	3100 6700 4950 6700
+	3100 6700 4100 6700
 Connection ~ 3100 6700
 Wire Wire Line
@@
 	3650 2250 5200 2250
 Wire Wire Line
-	3650 1100 5700 1100
+	3650 1100 4650 1100
 Connection ~ 3650 1100
 Wire Wire Line
@@
 	1    0    0    1
 $EndComp
+Wire Wire Line
+	1750 1050 1750 1100
+Connection ~ 1750 1100
+Wire Wire Line
+	1750 6750 1750 6700
+Connection ~ 1750 6700
+$Comp
+L power:GND #PWR0111
+U 1 1 610EEBFC
+P 4650 1750
+F 0 "#PWR0111" H 4650 1500 50  0001 C CNN
+F 1 "GND" H 4655 1577 50  0000 C CNN
+F 2 "" H 4650 1750 50  0001 C CNN
+F 3 "" H 4650 1750 50  0001 C CNN
+	1    4650 1750
+	1    0    0    -1
+$EndComp
+Wire Wire Line
+	4650 1750 4650 1600
+$Comp
+L Device:C C3
+U 1 1 610EEC04
+P 4650 1450
+F 0 "C3" H 4535 1404 50  0000 R CNN
+F 1 "100nF" H 4535 1495 50  0000 R CNN
+F 2 "Capacitor_SMD:C_1210_3225Metric_Pad1.33x2.70mm_HandSolder" H 4688 1300 50  0001 C CNN
+F 3 "~" H 4650 1450 50  0001 C CNN
+	1    4650 1450
+	-1   0    0    1
+$EndComp
+Wire Wire Line
+	4650 1300 4650 1100
+Connection ~ 4650 1100
+Wire Wire Line
+	4650 1100 5700 1100
+$Comp
+L power:GND #PWR0112
+U 1 1 61104596
+P 4100 6000
+F 0 "#PWR0112" H 4100 5750 50  0001 C CNN
+F 1 "GND" H 4105 5827 50  0000 C CNN
+F 2 "" H 4100 6000 50  0001 C CNN
+F 3 "" H 4100 6000 50  0001 C CNN
+	1    4100 6000
+	-1   0    0    1
+$EndComp
+Wire Wire Line
+	4100 6700 4100 6400
+Wire Wire Line
+	4100 6100 4100 6000
+$Comp
+L Device:C C1
+U 1 1 611045A2
+P 4100 6250
+F 0 "C1" H 3985 6204 50  0000 R CNN
+F 1 "100nF" H 3985 6295 50  0000 R CNN
+F 2 "Capacitor_SMD:C_1210_3225Metric_Pad1.33x2.70mm_HandSolder" H 4138 6100 50  0001 C CNN
+F 3 "~" H 4100 6250 50  0001 C CNN
+	1    4100 6250
+	-1   0    0    1
+$EndComp
+Connection ~ 4100 6700
+Wire Wire Line
+	4100 6700 4950 6700
 $EndSCHEMATC
