File: lv-lownoise-psu/kicad/v3d/lv-lownoise-psu.kicad_pcb (KiCad board)
At the start: 2 copper layers, 71.1 x 61 mm, 57 parts, among them J1 AC, J10 GND, J11 GND, J12 -5V, J2 GND, J3 AC, J4 +15V, J5 GND, J6 -15V, J7 LED, J8 GND, J9 +5V, Q1 BD679, Q2 BD680, U1 LM7805_TO220, U2 LM7905_TO220, U3 LT3045xMSE, U4 LT3094xMSE

Commit message: WIP
Parts:
- removed C15, C16: 4.7uF, Capacitor_Tantalum_SMD:CP_EIA-2012-12_Kemet-R_Pad1.30x1.05mm_HandSolder
- removed R1, R2: 150k, Resistor_SMD:R_0805_2012Metric_Pad1.20x1.40mm_HandSolder
- removed R10, R11, R4, R9: 0R, Resistor_SMD:R_0805_2012Metric_Pad1.15x1.40mm_HandSolder
- added C19: 4.7uF/25V, Capacitor_SMD:C_1206_3216Metric_Pad1.33x1.80mm_HandSolder, F.Cu at (125.0, 52.6)
- added C20: 4.7uF/25V, Capacitor_SMD:C_1206_3216Metric_Pad1.33x1.80mm_HandSolder, F.Cu at (40.2, 1.18)
- added C21: 4.7uF/25V, Capacitor_SMD:C_1206_3216Metric_Pad1.33x1.80mm_HandSolder, F.Cu at (128.7, 55.4)
- added C22: 4.7uF/25V, Capacitor_SMD:C_1206_3216Metric_Pad1.33x1.80mm_HandSolder, F.Cu at (135.9, 81.3)
- added D5: MMSZ5247C/17V, Diode_SMD:D_SOD-123, F.Cu at (121.8, 56.9)
- added D6: MMSZ5247C/17V, Diode_SMD:D_SOD-123, F.Cu at (26.7, 18.2)
- C17, C18: value 47uF -> 33uF
- C3, C4: value 10nF -> Cx/10nF/50V
- C5, C6: value 10nF -> Cs/50V
- C7, C9: value 4.7uF -> 100nF; footprint Capacitor_Tantalum_SMD:CP_EIA-2012-12_Kemet-R_Pad1.30x1.05mm_HandSolder -> Capacitor_SMD:C_0805_2012Metric_Pad1.18x1.45mm_HandSolder
- Q1: value BD679 -> BD139
- Q2: value BD680 -> BD140
- R5: value 3.16k -> Rs/1/8W
- R6: value 21k -> Rs/1/8W
- R7: value 21k -> 430R/0.6W; footprint Resistor_SMD:R_0805_2012Metric_Pad1.20x1.40mm_HandSolder -> Resistor_THT:R_Axial_DIN0207_L6.3mm_D2.5mm_P10.16mm_Horizontal
- R8: value 3.16k -> 430R/0.6W; footprint Resistor_SMD:R_0805_2012Metric_Pad1.20x1.40mm_HandSolder -> Resistor_THT:R_Axial_DIN0207_L6.3mm_D2.5mm_P10.16mm_Horizontal
- moved Q2 126.3 mm to (11.7, 5.52), turned to 0 degrees
- moved R8 112.5 mm to (25.4, 1.53), turned to 0 degrees
- moved C9 110.2 mm to (26.0, 21.6), turned to 0 degrees
- moved R6 87.8 mm to (37.0, 14.7), turned to 0 degrees
- moved C4 74.8 mm to (41.8, 4.36), turned to 0 degrees
- moved C6 68.4 mm to (41.6, 8.41), turned to 0 degrees
- moved R5 37.8 mm to (82.4, 59.1), turned to 0 degrees
- moved C3 18.2 mm to (82.3, 53.9), turned to 270 degrees
- moved C7 14.9 mm to (118.2, 57.8), turned to 270 degrees
- moved C5 8.98 mm to (85.7, 53.1), turned to 270 degrees
- moved R7 7.40 mm to (115.4, 56.6), turned to 90 degrees
- moved Q1 2.20 mm to (120.1, 48.7), turned to 270 degrees
Connections:
- C2 pad 2: Net-(C2-Pad2) -> Net-(C10-Pad2)
- C3 pad 2: Net-(C2-Pad2) -> GND
- C4 pad 1: Net-(C2-Pad2) -> GND
- C5 pad 2: Net-(C1-Pad1) -> Net-(C5-Pad2)
- C6 pad 1: Net-(C1-Pad1) -> GND
- C6 pad 2: Net-(C4-Pad2) -> Net-(C6-Pad2)
- C8 pad 1: Net-(C8-Pad1) -> Net-(C1-Pad1)
- D1 pad 2: Net-(C2-Pad2) -> Net-(C10-Pad2)
- D2 pad 2: Net-(C2-Pad2) -> Net-(C10-Pad2)
- Q1 pad 1: Net-(C7-Pad1) -> Net-(C19-Pad1)
- Q1 pad 3: Net-(Q1-Pad3) -> Net-(C7-Pad1)
- Q2 pad 1: Net-(C9-Pad2) -> Net-(C20-Pad2)
- Q2 pad 2: Net-(C2-Pad2) -> Net-(C10-Pad2)
- Q2 pad 3: Net-(Q2-Pad3) -> Net-(C9-Pad2)
- R5 pad 1: Net-(C1-Pad1) -> Net-(C5-Pad2)
- R5 pad 2: Net-(Q1-Pad3) -> GND
- R6 pad 1: Net-(Q1-Pad3) -> Net-(C6-Pad2)
- R6 pad 2: GND -> Net-(C4-Pad2)
- R7 pad 1: GND -> Net-(C1-Pad1)
- R7 pad 2: Net-(Q2-Pad3) -> Net-(C7-Pad1)
- R8 pad 1: Net-(Q2-Pad3) -> Net-(C9-Pad2)
- R8 pad 2: Net-(C2-Pad2) -> Net-(C10-Pad2)
- U1 pad 1: Net-(C8-Pad1) -> Net-(C1-Pad1)
- U3 pad 1: Net-(C7-Pad1) -> Net-(C19-Pad1)
- U3 pad 2: Net-(C7-Pad1) -> Net-(C19-Pad1)
- U3 pad 3: Net-(C7-Pad1) -> Net-(C19-Pad1)
- U3 pad 4: Net-(C7-Pad1) -> Net-(C19-Pad1)
- U3 pad 7: Net-(C7-Pad1) -> Net-(C19-Pad1)
- U4 pad 1: Net-(C9-Pad2) -> Net-(C20-Pad2)
- U4 pad 13: Net-(C9-Pad2) -> Net-(C20-Pad2)
- U4 pad 2: Net-(C9-Pad2) -> Net-(C20-Pad2)
- U4 pad 3: Net-(C9-Pad2) -> Net-(C20-Pad2)
- U4 pad 5: Net-(C9-Pad2) -> Net-(C20-Pad2)
Routing:
- net Net-(C10-Pad2): track 7.28 -> 44.4 mm, vias 0 -> 1
- net Net-(C2-Pad2): track 42.9 -> 5.79 mm, vias 1 -> 0
- net Net-(C1-Pad1): track 43.7 -> 19.1 mm
- net Net-(C7-Pad1): track 20.1 -> 0.00 mm, vias 2 -> 0
- net Net-(C9-Pad2): track 16.6 -> 0.00 mm
- net Net-(C20-Pad2): track 0.00 -> 16.6 mm
- net Net-(C19-Pad1): track 0.00 -> 10.1 mm, vias 0 -> 2
- net Net-(C8-Pad1): track 9.39 -> 0.00 mm
- net Net-(Q1-Pad3): track 6.74 -> 0.00 mm
- net Net-(C3-Pad1): track 34.4 -> 31.0 mm
- net Net-(C4-Pad2): track 25.5 -> 22.1 mm

Commit message: finish layout
Parts:
- C13, C14: value 100uF -> 10uF/25V; footprint Capacitor_THT:CP_Radial_D8.0mm_P3.50mm -> Capacitor_SMD:C_1206_3216Metric_Pad1.33x1.80mm_HandSolder
- moved Q2 124.7 mm to (118.8, 69.3), turned to 90 degrees
- moved C20 108.5 mm to (123.4, 70.8), turned to 90 degrees
- moved R8 107.1 mm to (114.3, 61.2), turned to 270 degrees
- moved C9 105.3 mm to (122.3, 64.2), turned to 180 degrees
- moved D6 103.1 mm to (120.5, 61.2), turned to 180 degrees
- moved C4 64.8 mm to (83.9, 53.6), turned to 90 degrees
- moved C6 58.0 mm to (86.9, 44.6), turned to 180 degrees
- moved R6 56.2 mm to (83.9, 45.6), turned to 270 degrees
- moved C5 18.2 mm to (83.9, 71.2)
- moved C8 14.8 mm to (128.0, 34.3), turned to 0 degrees
- moved C12 14.2 mm to (128.0, 82.5), turned to 180 degrees
- moved R5 13.9 mm to (86.9, 72.3)
- moved C14 12.4 mm to (124.4, 85.5), turned to 180 degrees
- moved C22 10.6 mm to (137.0, 70.8), turned to 90 degrees
- moved R7 10.2 mm to (114.3, 46.5), turned to 270 degrees
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Routing:
- net Net-(C1-Pad1): track 19.1 -> 51.4 mm
- net Net-(C11-Pad1): track 33.7 -> 22.8 mm
- net Net-(C7-Pad1): track 0.00 -> 10.1 mm
- net Net-(C19-Pad1): track 10.1 -> 20.1 mm
- net Net-(C9-Pad2): track 0.00 -> 9.99 mm
- net Net-(C18-Pad2): track 15.7 -> 23.6 mm
- net Net-(C17-Pad1): track 15.4 -> 23.3 mm
- net Net-(C12-Pad2): track 17.3 -> 11.0 mm
- net Net-(C10-Pad2): track 44.4 -> 50.5 mm
- net Net-(Q2-Pad3): track 5.90 -> 0.00 mm
- net Net-(C2-Pad2): track 5.79 -> 0.00 mm
- net Net-(C4-Pad2): track 22.1 -> 26.0 mm
- net GND: track 8.28 -> 12.1 mm
- net Net-(J7-Pad1): track 5.86 -> 2.86 mm
- net Net-(C3-Pad1): track 31.0 -> 33.5 mm
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Other:
- board text added: "+"
- board text added: "K"
- board text added: "Low noise dual power supply V3d Michael Schenk, 2021.09.07"
- board text added: "°"
- board text removed: "Low noise dual power supply V3c Michael Schenk, 2020.12.27"
