File: lv-lownoise-psu/kicad/v3d-1.0/lv-lownoise-psu.kicad_pcb (KiCad board)
At the start: 2 copper layers, 71.1 x 61 mm, 55 parts, among them J1 AC, J10 GND, J11 GND, J12 -5V, J2 GND, J3 AC, J4 +15V, J5 GND, J6 -15V, J7 LED, J8 GND, J9 +5V, Q1 BD139, Q2 BD140, U1 LM7805_TO220, U2 LM7905_TO220, U3 LT3045xMSE, U4 LT3094xMSE

Commit message: ready to order
Parts:
- added D10: MMSZ5232B/5.6V, Diode_SMD:D_SOD-123, F.Cu at (125.2, 60.3)
- added D7: MMSZ5232B/5.6V, Diode_SMD:D_SOD-123, F.Cu at (124.5, 57.7)
- added D8: MMSZ5232B/5.6V, Diode_SMD:D_SOD-123, F.Cu at (129.3, 57.7)
- added D9: MMSZ5232B/5.6V, Diode_SMD:D_SOD-123, F.Cu at (130.0, 60.3)
- D5, D6: value MMSZ5247C/17V -> MMSZ5232B/5.6V
- J10, J11, J12, J4, J5, J6, J7, J8, J9: footprint Connector_Pin:Pin_D1.3mm_L11.0mm -> Connector_Pin:Pin_D1.0mm_L10.0mm
Connections:
- D5 pad 2: GND -> Net-(D5-Pad2)
- D6 pad 1: GND -> Net-(D10-Pad2)
Routing:
- net Net-(D5-Pad2): track 0.00 -> 1.91 mm
- net Net-(D10-Pad2): track 0.00 -> 1.86 mm
- net Net-(D7-Pad2): track 0.00 -> 1.46 mm
- net Net-(D10-Pad1): track 0.00 -> 1.46 mm
Other:
- board text added: "Low noise dual power supply V3d-1.0 Michael Schenk, 2021.09.15"
- board text removed: "Low noise dual power supply V3d Michael Schenk, 2021.09.07"
