File: lv-lownoise-psu/kicad/lm317-lm337-die-noiser-v1a/lv-lownoise-psu.kicad_pcb (KiCad board)
At the start: 2 copper layers, 71.1 x 61 mm, 67 parts, among them J1 AC, J10 GND, J11 GND, J12 -5V, J2 GND, J3 AC, J4 +15V, J5 GND, J6 -15V, J7 LED, J8 GND, J9 +5V, Q1 BC817-40, Q2 BC807-40, U1 LM7805_TO220, U2 LM7905_TO220, U5 LM317_TO-220, U6 LM337_TO220

Commit message: WIP
Parts:
- added NT1: Net-Tie_2, NetTie:NetTie-2_SMD_Pad0.5mm, F.Cu at (143.5, 58.0)
- added Q3: BC807-40, Package_TO_SOT_SMD:SOT-23, F.Cu at (134.2, 48.7)
- added R14: 270R, Resistor_SMD:R_0805_2012Metric_Pad1.20x1.40mm_HandSolder, F.Cu at (137.0, 48.8)
- C16: value 10nF -> 22nF
- moved D5 13.3 mm to (139.6, 55.9), turned to 180 degrees
- moved Q1 11.7 mm to (137.0, 52.5)
- moved C16 10.4 mm to (133.1, 51.5), turned to 0 degrees
- moved R10 9.24 mm to (140.2, 52.6), turned to 270 degrees
- moved R9 8.51 mm to (139.0, 48.8), turned to 270 degrees
- moved R7 7.76 mm to (115.8, 54.6)
- moved R1 7.75 mm to (115.8, 50.8)
- moved R8 7.45 mm to (141.0, 48.8)
- moved C21 6.33 mm to (144.0, 51.4), turned to 270 degrees
- moved C15 2.41 mm to (126.8, 52.3)
- moved RV1 2.01 mm to (129.5, 58.9)
- moved C19 0.08 mm to (148.0, 53.9)
Connections:
- net Net-(C17-Pad1) renamed /Force+
- C1 pad 2: GND -> (no net)
- C16 pad 2: GND -> /Sense-
- C18 pad 1: GND -> (no net)
- C2 pad 1: GND -> (no net)
- C22 pad 1: GND -> (no net)
- C24 pad 1: GND -> (no net)
- C9 pad 1: GND -> (no net)
- D1 pad 2: Net-(C10-Pad2) -> Net-(D1-Pad2)
- D2 pad 2: Net-(C10-Pad2) -> Net-(D1-Pad2)
- D3 pad 1: Net-(C1-Pad1) -> Net-(D3-Pad1)
- D4 pad 1: Net-(C1-Pad1) -> Net-(D3-Pad1)
- D5 pad 2: GND -> /Sense-
- D6 pad 1: GND -> (no net)
- Q1 pad 2: GND -> /Sense-
- Q1 pad 3: Net-(C15-Pad2) -> Net-(Q1-Pad3)
- Q2 pad 2: GND -> (no net)
- R2 pad 1: GND -> (no net)
- RV2 pad 2: GND -> (no net)
- RV2 pad 3: GND -> (no net)
Routing:
- net /Sense-: track 0.00 -> 15.3 mm
- net Net-(C15-Pad1): track 19.8 -> 6.86 mm, vias 1 -> 0
- net Net-(C15-Pad2): track 10.4 -> 19.4 mm
- net Net-(Q1-Pad3): track 0.00 -> 2.86 mm
- net Net-(C21-Pad2): track 2.55 -> 4.77 mm
- net GND: track 0.00 -> 2.10 mm
- net Net-(D5-Pad1): track 9.54 -> 8.00 mm
- net /Force+: track 41.2 -> 41.9 mm, vias 0 -> 1

Commit message: WIP
Parts:
- added NT2: Net-Tie_2, NetTie:NetTie-2_SMD_Pad0.5mm, F.Cu at (143.5, 59.5)
- added Q4: BC817-40, Package_TO_SOT_SMD:SOT-23, F.Cu at (131.4, 63.0)
- added R15: 270R, Resistor_SMD:R_0805_2012Metric_Pad1.20x1.40mm_HandSolder, F.Cu at (136.9, 67.4)
- C22: value 10nF -> 22nF
- moved C23 7.44 mm to (143.9, 62.6)
- moved R11 7.41 mm to (141.0, 68.5)
- moved R12 5.85 mm to (137.9, 64.0)
- moved Q2 5.85 mm to (135.1, 64.1)
- moved D6 2.72 mm to (139.7, 60.5), turned to 0 degrees
- moved C22 2.42 mm to (128.6, 62.8)
- moved R13 2.14 mm to (140.0, 64.0)
- moved RV1 1.65 mm to (129.5, 57.3)
- moved NT1 1.40 mm to (143.5, 56.6)
- moved RV2 0.64 mm to (129.5, 77.0)
Connections:
- C1 pad 2: (no net) -> GND
- C18 pad 1: (no net) -> GND
- C2 pad 1: (no net) -> GND
- C22 pad 1: (no net) -> Net-(C22-Pad1)
- C24 pad 1: (no net) -> GND
- C9 pad 1: (no net) -> GND
- D1 pad 2: Net-(D1-Pad2) -> Net-(C10-Pad2)
- D2 pad 2: Net-(D1-Pad2) -> Net-(C10-Pad2)
- D3 pad 1: Net-(D3-Pad1) -> Net-(C1-Pad1)
- D4 pad 1: Net-(D3-Pad1) -> Net-(C1-Pad1)
- D6 pad 1: (no net) -> Net-(C22-Pad1)
- Q2 pad 2: (no net) -> Net-(C22-Pad1)
- Q2 pad 3: Net-(C20-Pad1) -> Net-(Q2-Pad3)
- R2 pad 1: (no net) -> GND
- RV2 pad 2: (no net) -> GND
- RV2 pad 3: (no net) -> GND
Routing:
- net Net-(C15-Pad1): track 6.86 -> 24.0 mm
- net Net-(C22-Pad1): track 0.00 -> 16.6 mm
- net Net-(C20-Pad1): track 10.4 -> 19.5 mm
- net Net-(Q2-Pad3): track 0.00 -> 7.80 mm
- net GND: track 2.10 -> 7.99 mm
- net Net-(Q1-Pad3): track 2.86 -> 6.54 mm
- net /Force+: track 41.9 -> 44.4 mm
- net Net-(C23-Pad1): track 2.42 -> 4.88 mm
- net Net-(D6-Pad2): track 9.54 -> 7.14 mm
- net Net-(C20-Pad2): track 20.8 -> 20.2 mm
- net Net-(C18-Pad2): track 43.3 -> 43.7 mm, vias 0 -> 1

Commit message: Create gerber, ready to order
Parts:
- moved R4 7.85 mm to (115.8, 69.2)
- moved Q4 6.08 mm to (134.1, 68.4), turned to 270 degrees
- moved C22 5.05 mm to (133.1, 65.2), turned to 180 degrees
- moved R12 4.53 mm to (138.9, 68.4)
- moved C9 3.47 mm to (115.8, 74.4), turned to 90 degrees
- moved C20 2.48 mm to (126.7, 67.2)
- moved Q2 1.91 mm to (137.0, 64.0)
- moved R15 1.00 mm to (137.0, 68.4), turned to 270 degrees
Routing:
- net Net-(C20-Pad2): track 20.2 -> 26.5 mm, vias 1 -> 0
- net Net-(Q2-Pad3): track 7.80 -> 4.35 mm
- net Net-(D6-Pad2): track 7.14 -> 10.2 mm
- net Net-(C18-Pad2): track 43.7 -> 46.1 mm
- net Net-(C10-Pad2): track 58.0 -> 59.4 mm
- net Net-(C20-Pad1): track 19.5 -> 20.7 mm
Other:
- board text added: "Low noise dual PSU LM317/337 with die-noiser V1a Michael Schenk, 2021.10.12"
- board text removed: "Low noise dual PSU LM317/337 with denoiser V1a Michael Schenk, 2021.10.3"
