File: lv-lownoise-psu/kicad/v3d-2.0/lv-lownoise-psu.kicad_pcb (KiCad board)
At the start: 2 copper layers, 71.1 x 61 mm, 59 parts, among them J1 AC, J10 GND, J11 GND, J12 -5V, J2 GND, J3 AC, J4 +15V, J5 GND, J6 -15V, J7 LED, J8 GND, J9 +5V, Q1 BD139, Q2 BD140, U1 LM7805_TO220, U2 LM7905_TO220, U3 LT3045xMSE, U4 LT3094xMSE

Commit message: Gerber created, ready to order
Parts:
- added C15: 4.7uF/35V, Capacitor_Tantalum_SMD:CP_EIA-3528-15_AVX-H_Pad1.50x2.35mm_HandSolder, F.Cu at (128.1, 48.2)
- added C16: 4.7uF/35V, Capacitor_Tantalum_SMD:CP_EIA-3528-15_AVX-H_Pad1.50x2.35mm_HandSolder, F.Cu at (137.0, 52.1)
- C19, C20: value 4.7uF/25V -> 4.7uF/35V; footprint Capacitor_SMD:C_1206_3216Metric_Pad1.33x1.80mm_HandSolder -> Capacitor_Tantalum_SMD:CP_EIA-3528-15_AVX-H_Pad1.50x2.35mm_HandSolder
- C21, C22: value 4.7uF/25V -> 4.7uF/50V
- C7, C9: value 100nF -> 4.7uF/50V; footprint Capacitor_SMD:C_0805_2012Metric_Pad1.18x1.45mm_HandSolder -> Capacitor_SMD:C_1206_3216Metric_Pad1.33x1.80mm_HandSolder
- U3: value LT3045xMSE -> LT3045xDD-10DFN; footprint Package_SO:MSOP-12-1EP_3x4mm_P0.65mm_EP1.65x2.85mm -> Package_DFN_QFN:DFN-10-1EP_3x3mm_P0.5mm_EP1.65x2.38mm
- U4: value LT3094xMSE -> LT3094xDD-12DFN; footprint Package_SO:MSOP-12-1EP_3x4mm_P0.65mm_EP1.65x2.85mm -> Package_DFN_QFN:DFN-12-1EP_3x3mm_P0.45mm_EP1.66x2.38mm
- moved C19 17.3 mm to (128.0, 66.3), turned to 270 degrees
- moved C22 14.6 mm to (123.0, 66.7), turned to 180 degrees
- moved C21 14.1 mm to (123.0, 51.1), turned to 0 degrees
- moved C20 9.50 mm to (132.8, 72.4), turned to 0 degrees
- moved RV1 7.43 mm to (135.4, 56.6), turned to 180 degrees
- moved RV2 4.23 mm to (138.2, 72.4), turned to 180 degrees
- moved C18 3.72 mm to (136.5, 64.0), turned to 270 degrees
- moved C17 3.56 mm to (136.8, 45.8), turned to 90 degrees
- moved U4 2.02 mm to (131.8, 68.8)
- moved U3 2.01 mm to (132.0, 50.3)
- moved D7 1.08 mm to (124.5, 56.6)
- moved D8 1.08 mm to (129.3, 56.6)
- moved D10 0.95 mm to (125.2, 61.2)
- moved D9 0.95 mm to (130.0, 61.2)
- moved J4 0.83 mm to (148.0, 49.0)
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Connections:
- C19 pad 1: Net-(C19-Pad1) -> GND
- C19 pad 2: GND -> Net-(C19-Pad2)
- C21 pad 1: Net-(C21-Pad1) -> Net-(C1-Pad1)
- C22 pad 2: Net-(C22-Pad2) -> Net-(C10-Pad2)
- Q1 pad 1: Net-(C19-Pad1) -> Net-(C15-Pad1)
- Q2 pad 1: Net-(C20-Pad2) -> Net-(C19-Pad2)
- RV1 pad 1: Net-(C21-Pad1) -> Net-(C16-Pad1)
- RV2 pad 1: Net-(C22-Pad2) -> Net-(C20-Pad2)
- U3 pad 1: Net-(C19-Pad1) -> Net-(C15-Pad1)
- U3 pad 11: Net-(C17-Pad1) -> GND
- U3 pad 2: Net-(C19-Pad1) -> Net-(C15-Pad1)
- U3 pad 3: Net-(C19-Pad1) -> Net-(C15-Pad1)
- U3 pad 4: Net-(C19-Pad1) -> (no net)
- U3 pad 5: (no net) -> GND
- U3 pad 6: GND -> Net-(C15-Pad1)
- U3 pad 7: Net-(C19-Pad1) -> Net-(C16-Pad1)
- U3 pad 8: Net-(C21-Pad1) -> GND
- U3 pad 9: GND -> Net-(C17-Pad1)
- U4 pad 1: Net-(C20-Pad2) -> Net-(C19-Pad2)
- U4 pad 13: Net-(C20-Pad2) -> Net-(C19-Pad2)
- U4 pad 2: Net-(C20-Pad2) -> Net-(C19-Pad2)
- U4 pad 3: Net-(C20-Pad2) -> Net-(C19-Pad2)
- U4 pad 5: Net-(C20-Pad2) -> Net-(C19-Pad2)
- U4 pad 8: Net-(C22-Pad2) -> Net-(C20-Pad2)
Routing:
- net Net-(C15-Pad1): track 0.00 -> 23.7 mm, vias 0 -> 2
- net Net-(C19-Pad2): track 0.00 -> 22.0 mm
- net Net-(C19-Pad1): track 20.1 -> 0.00 mm, vias 2 -> 0
- net Net-(C22-Pad2): track 8.94 -> 0.00 mm
- net Net-(C21-Pad1): track 8.78 -> 0.00 mm
- net Net-(C16-Pad1): track 0.00 -> 7.45 mm
- net Net-(C20-Pad2): track 15.1 -> 7.74 mm
- net Net-(C17-Pad1): track 23.3 -> 19.2 mm, vias 1 -> 0
- net Net-(C1-Pad1): track 51.4 -> 54.6 mm
- net Net-(C10-Pad2): track 50.5 -> 53.1 mm
- net GND: track 12.1 -> 13.5 mm
- net Net-(C18-Pad2): track 23.6 -> 22.5 mm, vias 1 -> 0
Other:
- board text added: "Low noise dual power supply V3d-2.0 Michael Schenk, 2021.10.15"
- board text removed: "Low noise dual power supply V3d-1.0 Michael Schenk, 2021.09.15"
