File: pre-amp-discret-elektor/kicad/v2b-servo/pre-amp-discret.kicad_pcb (KiCad board)
At the start: 2 copper layers, 81.9 x 52.1 mm, 71 parts, among them J1 Conn_01x01, J2 Conn_01x01, J3 Conn_01x01, J4 Conn_01x01, J5 Conn_01x01, J6 Conn_01x01, J7 Conn_01x01, Q1 BCM857DS,115, Q11 BCM847DS,115, Q13 BCM847DS,115, Q2 BC850C, Q3 BCM857DS,115, Q4 BC550C, Q5 BC560C, Q6 BC337-40, Q7 BC860C, Q8 BC327-40, U1 OPA188xxDBV

Commit message: WIP
Parts:
- removed C1, C18, C19, C3: 220uF, Capacitor_THT:CP_Radial_D8.0mm_P3.50mm
- C13, C14, C4, C5: footprint Capacitor_THT:C_Rect_L7.2mm_W2.5mm_P5.00mm_FKS2_FKP2_MKS2_MKP2 -> Capacitor_SMD:C_1210_3225Metric_Pad1.33x2.70mm_HandSolder
- C15, C16: value 220uF -> 10uF/25V; footprint Capacitor_THT:CP_Radial_D8.0mm_P3.50mm -> Capacitor_SMD:CP_Elec_6.3x5.8
- moved C4 41.1 mm to (144.4, 107.1), turned to 270 degrees
- moved C15 39.6 mm to (182.5, 106.8), turned to 0 degrees
- moved C16 39.4 mm to (182.2, 137.5), turned to 180 degrees
- moved C5 38.2 mm to (144.9, 137.4), turned to 270 degrees
- moved C13 25.5 mm to (175.2, 105.2)
- moved C14 24.1 mm to (174.9, 139.0)
- moved R25 20.6 mm to (140.6, 118.4), turned to 270 degrees
- moved R4 20.6 mm to (141.1, 124.6), turned to 270 degrees
- moved R7 18.0 mm to (147.6, 125.5), turned to 270 degrees
- moved Q3 16.4 mm to (144.5, 124.5)
- moved Q11 15.8 mm to (143.8, 119.4)
- moved R22 15.6 mm to (147.2, 119.3)
- moved C7 6.03 mm to (162.9, 115.8)
- moved C8 6.03 mm to (163.0, 127.3)
- moved C9 6.03 mm to (175.4, 124.8)
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Routing:
- net Net-(Q3-Pad6): track 25.4 -> 4.78 mm, vias 4 -> 0
- net Net-(Q11-Pad6): track 24.2 -> 4.51 mm, vias 4 -> 0
- net Net-(Q13-Pad6): track 29.9 -> 23.9 mm
- net Net-(Q1-Pad6): track 27.4 -> 21.4 mm
- net DCSERVO_IN: track 33.8 -> 30.2 mm
- net Net-(C12-Pad1): track 26.2 -> 22.5 mm
- net Net-(C12-Pad2): track 45.8 -> 43.5 mm
- net +15V: track 113.8 -> 111.7 mm
- net Net-(Q3-Pad1): track 6.23 -> 5.32 mm
- net -15V: track 115.9 -> 115.2 mm
Other:
- board text added: "Pre-Amp Elektor V2b DC Servo Michael Schenk 2021.10.27"
- board text removed: "Pre-Amp Elektor V2a DC Servo Michael Schenk 2021.05.19"
