File: amp-mosfet-160W/kicad/v1/amp-mosfet-160w/amp-mosfet-160w.kicad_pcb (KiCad board)
At the start: 2 copper layers, 160 x 100.3 mm, 74 parts, among them J1 Conn_01x01, J2 Conn_01x01, J3 +69V, J4 -69V, J5 LS+, J6 LS-, J7 GND, Q1 BC556, Q10 MJE340, Q11 ECX10P20, Q12 ECX10N20, Q2 MJE340, Q3 MJE350, Q4 ECX10P20, Q5 ECX10N20, Q6 BC556, Q7 BC556, Q8 BC556, Q9 MJE350

Commit message: WIP
Parts:
- moved MK1 185.2 mm to (67.2, 43.7)
- moved C3 129.0 mm to (137.5, 78.4), turned to 180 degrees
- moved R9 93.4 mm to (140.6, 73.7), turned to 180 degrees
- moved R12 91.3 mm to (116.1, 68.1)
- moved R8 87.4 mm to (138.4, 68.7)
- moved R20 87.2 mm to (146.3, 65.4), turned to 180 degrees
- moved MK2 52.5 mm to (203.1, 43.6)
- moved J3 6.67 mm to (205.2, 77.5)
- moved R15 6.54 mm to (80.4, 96.6)
- moved R22 6.33 mm to (160.3, 67.8)
- moved R21 5.84 mm to (181.7, 67.8)
- moved R16 5.27 mm to (101.6, 96.6)
- moved R18 5.13 mm to (69.8, 102.5)
- moved R24 4.83 mm to (189.7, 71.2)
- moved C17 3.66 mm to (189.7, 67.8)
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Connections:
- Q11 pad 2: Net-(C18-Pad2) -> Net-(Q11-Pad2)
- Q11 pad 3: Net-(Q11-Pad3) -> Net-(C18-Pad2)
- Q4 pad 2: Net-(C18-Pad2) -> Net-(Q4-Pad2)
- Q4 pad 3: Net-(Q4-Pad3) -> Net-(C18-Pad2)
- R15 pad 2: Net-(Q4-Pad3) -> Net-(Q4-Pad2)
- R16 pad 2: Net-(Q11-Pad3) -> Net-(Q11-Pad2)
Routing:
- net Net-(C18-Pad2): track 24.2 -> 0.00 mm
Other:
- board size 160 x 100.3 mm -> 165.1 x 100.3 mm

Commit message: WIP
Parts:
- R10: value 22k -> 1k
- moved C4 116.2 mm to (108.3, 109.6)
- moved C6 105.1 mm to (117.1, 109.6)
- moved R5 104.6 mm to (147.2, 122.7)
- moved Q6 98.5 mm to (160.0, 115.3)
- moved C5 88.5 mm to (116.4, 100.3)
- moved Q7 83.1 mm to (151.9, 115.6)
- moved R11 75.8 mm to (113.8, 95.4)
- moved R3 68.2 mm to (158.6, 119.9)
- moved R10 66.3 mm to (111.6, 104.5)
Changed lines of the file:
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@@
   )
   (module Resistor_THT:R_Axial_DIN0207_L6.3mm_D2.5mm_P10.16mm_Horizontal (layer F.Cu)
-    (at 183.184001 125.920001)
+    (at 113.792 95.377)
     (descr "Resistor, Axial_DIN0207 series, Axial, Horizontal, pin pitch=10.16mm, 0.25W = 1/4W, length*diameter=6.3*2.5mm^2, http://cdn-reichelt.de/documents/datenblatt/B400/1_4W%23YAG.pdf")
     (tags "Resistor Axial_DIN0207 series Axial Horizontal pin pitch 10.16mm 0.25W = 1/4W length 6.3mm diameter 2.5mm")
@@
   )
   (module Resistor_THT:R_Axial_DIN0207_L6.3mm_D2.5mm_P10.16mm_Horizontal (layer F.Cu)
-    (at 171.014001 134.020001)
+    (at 111.633 104.521)
     (descr "Resistor, Axial_DIN0207 series, Axial, Horizontal, pin pitch=10.16mm, 0.25W = 1/4W, length*diameter=6.3*2.5mm^2, http://cdn-reichelt.de/documents/datenblatt/B400/1_4W%23YAG.pdf")
     (tags "Resistor Axial_DIN0207 series Axial Horizontal pin pitch 10.16mm 0.25W = 1/4W length 6.3mm diameter 2.5mm")
@@
       (effects (font (size 1 1) (thickness 0.15)))
     )
-    (fp_text value 22k (at 5.08 2.37) (layer F.Fab)
+    (fp_text value 1k (at 5.08 2.37) (layer F.Fab)
       (effects (font (size 1 1) (thickness 0.15)))
     )
@@
   )
   (module Resistor_THT:R_Axial_DIN0207_L6.3mm_D2.5mm_P10.16mm_Horizontal (layer F.Cu)
-    (at 243.074001 80.840001)
+    (at 147.193 122.682)
     (descr "Resistor, Axial_DIN0207 series, Axial, Horizontal, pin pitch=10.16mm, 0.25W = 1/4W, length*diameter=6.3*2.5mm^2, http://cdn-reichelt.de/documents/datenblatt/B400/1_4W%23YAG.pdf")
     (tags "Resistor Axial_DIN0207 series Axial Horizontal pin pitch 10.16mm 0.25W = 1/4W length 6.3mm diameter 2.5mm")
@@
   )
   (module Resistor_THT:R_Axial_DIN0207_L6.3mm_D2.5mm_P10.16mm_Horizontal (layer F.Cu)
-    (at 223.274001 98.290001)
+    (at 158.623 119.888)
     (descr "Resistor, Axial_DIN0207 series, Axial, Horizontal, pin pitch=10.16mm, 0.25W = 1/4W, length*diameter=6.3*2.5mm^2, http://cdn-reichelt.de/documents/datenblatt/B400/1_4W%23YAG.pdf")
     (tags "Resistor Axial_DIN0207 series Axial Horizontal pin pitch 10.16mm 0.25W = 1/4W length 6.3mm diameter 2.5mm")
@@
   )
   (module Package_TO_SOT_THT:TO-92_Inline (layer F.Cu)
-    (at 234.624001 123.820001)
+    (at 151.892 115.57)
     (descr "TO-92 leads in-line, narrow, oval pads, drill 0.75mm (see NXP sot054_po.pdf)")
     (tags "to-92 sc-43 sc-43a sot54 PA33 transistor")
@@
   )
   (module Package_TO_SOT_THT:TO-92_Inline (layer F.Cu)
-    (at 257.554001 101.710001)
+    (at 160.02 115.316)
     (descr "TO-92 leads in-line, narrow, oval pads, drill 0.75mm (see NXP sot054_po.pdf)")
     (tags "to-92 sc-43 sc-43a sot54 PA33 transistor")
@@
   )
   (module Capacitor_THT:C_Rect_L7.2mm_W2.5mm_P5.00mm_FKS2_FKP2_MKS2_MKP2 (layer F.Cu)
-    (at 221.784001 118.540001)
+    (at 117.094 109.601)
     (descr "C, Rect series, Radial, pin pitch=5.00mm, , length*width=7.2*2.5mm^2, Capacitor, http://www.wima.com/EN/WIMA_FKS_2.pdf")
     (tags "C Rect series Radial pin pitch 5.00mm  length 7.2mm width 2.5mm Capacitor")
@@
   )
   (module Capacitor_THT:C_Rect_L7.2mm_W2.5mm_P5.00mm_FKS2_FKP2_MKS2_MKP2 (layer F.Cu)
-    (at 197.934001 134.840001)
+    (at 116.412 100.33)
     (descr "C, Rect series, Radial, pin pitch=5.00mm, , length*width=7.2*2.5mm^2, Capacitor, http://www.wima.com/EN/WIMA_FKS_2.pdf")
     (tags "C Rect series Radial pin pitch 5.00mm  length 7.2mm width 2.5mm Capacitor")
@@
   )
   (module Capacitor_THT:CP_Radial_D5.0mm_P2.00mm (layer F.Cu)
-    (at 222.403776 131.790001)
+    (at 108.331 109.601)
     (descr "CP, Radial series, Radial, pin pitch=2.00mm, , diameter=5mm, Electrolytic Capacitor")
     (tags "CP Radial series Radial pin pitch 2.00mm  diameter 5mm Electrolytic Capacitor")

Commit message: WIP
Parts:
- R15, R16, R23, R24: moved to F.Cu
- moved J2 162.0 mm to (93.3, 127.5)
- moved J1 158.5 mm to (101.6, 127.5)
- moved R2 68.9 mm to (114.3, 112.4), turned to 270 degrees
- moved R1 67.7 mm to (108.0, 119.4), turned to 180 degrees
- moved C2 63.6 mm to (111.3, 112.4), turned to 180 degrees
- moved C1 60.5 mm to (108.0, 122.5), turned to 270 degrees
- moved R7 41.3 mm to (104.5, 109.2), turned to 180 degrees
- moved Q1 38.1 mm to (112.8, 106.7), turned to 270 degrees
- moved Q8 34.4 mm to (108.6, 109.2), turned to 90 degrees
- moved R4 31.4 mm to (112.8, 103.4), turned to 180 degrees
- moved C4 27.5 mm to (128.5, 128.3), turned to 270 degrees
- moved R11 20.6 mm to (132.1, 104.9), turned to 270 degrees
- moved R10 19.9 mm to (128.5, 115.1), turned to 270 degrees
- moved C6 17.0 mm to (123.7, 125.2), turned to 270 degrees
- moved D3 15.1 mm to (118.4, 92.6)
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Routing:
- net GND: track 33.7 -> 155.0 mm
- net Net-(C13-Pad1): track 0.00 -> 113.6 mm
- net Net-(C7-Pad1): track 0.00 -> 93.7 mm
- net Net-(C18-Pad2): track 0.00 -> 75.5 mm
- net Net-(C7-Pad2): track 0.00 -> 71.9 mm
- net Net-(C14-Pad1): track 0.00 -> 54.5 mm
- net Net-(Q2-Pad3): track 0.00 -> 52.7 mm
- net Net-(C10-Pad2): track 0.00 -> 51.3 mm
- net Net-(C8-Pad1): track 0.00 -> 49.3 mm
- net Net-(C3-Pad1): track 0.00 -> 35.7 mm
- net Net-(C5-Pad2): track 0.00 -> 21.2 mm
- net Net-(C16-Pad1): track 0.00 -> 20.5 mm
- net Net-(C3-Pad2): track 0.00 -> 19.5 mm
- net Net-(Q10-Pad1): track 0.00 -> 15.8 mm
- net Net-(C15-Pad1): track 0.00 -> 12.6 mm
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
Commit message: WIP
Parts:
- moved J2 18.0 mm to (111.1, 130.2)
- moved R17 7.90 mm to (191.3, 102.0)
- moved D5 7.27 mm to (201.4, 98.9)
- moved JP1 7.16 mm to (201.4, 85.1)
- moved C14 6.74 mm to (205.2, 82.5)
- moved R1 6.48 mm to (113.7, 122.4), turned to 0 degrees
- moved C11 5.90 mm to (191.2, 109.2)
- moved C9 5.24 mm to (191.2, 118.0)
- moved R2 3.43 mm to (110.9, 112.3)
- moved C2 2.92 mm to (114.2, 112.3), turned to 270 degrees
- moved J1 2.73 mm to (101.5, 130.2)
- moved C1 1.40 mm to (106.6, 122.4), turned to 180 degrees
Routing:
- net GND: track 155.0 -> 282.4 mm
- net Net-(Q7-Pad1): track 0.00 -> 32.0 mm
- net Net-(C10-Pad2): track 51.3 -> 77.7 mm
- net Net-(C11-Pad1): track 8.70 -> 24.7 mm
- net Net-(C13-Pad1): track 113.6 -> 125.9 mm
- net Net-(C5-Pad2): track 21.2 -> 33.0 mm
- net Net-(C14-Pad1): track 54.5 -> 63.4 mm
- net Net-(C4-Pad1): track 0.00 -> 7.87 mm
- net Net-(C1-Pad2): track 0.00 -> 7.82 mm
- net Net-(C1-Pad1): track 0.00 -> 7.11 mm
- net Net-(C13-Pad2): track 0.00 -> 4.59 mm
- net Net-(Q2-Pad3): track 52.7 -> 56.9 mm
- net Net-(C2-Pad1): track 5.27 -> 9.14 mm
- net Net-(D5-Pad2): track 0.00 -> 3.68 mm
- net Net-(C8-Pad1): track 49.3 -> 52.6 mm
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
Commit message: Update amp-mosfet-160w.kicad_pcb
Parts:
- moved R3 4.05 mm to (161.3, 116.8), turned to 270 degrees
- moved Q6 3.98 mm to (156.6, 116.8)
- moved Q7 3.98 mm to (152.4, 119.4)
- moved R5 0.44 mm to (147.2, 123.1), turned to 90 degrees
- moved J2 0.19 mm to (111.1, 130.4)
- moved C6 0.19 mm to (123.7, 125.4)
- moved C4 0.16 mm to (128.5, 128.4)
Routing:
- net Net-(C11-Pad1): track 24.7 -> 144.2 mm
- net Net-(Q6-Pad2): track 0.00 -> 11.5 mm
- net Net-(Q6-Pad1): track 0.00 -> 9.42 mm
- net GND: track 282.4 -> 290.3 mm
- net Net-(Q7-Pad1): track 32.0 -> 35.1 mm

Commit message: Update amp-mosfet-160w.kicad_pcb
Parts:
- moved MK1 1.14 mm to (67.2, 42.5)
- moved MK2 1.02 mm to (203.1, 42.5)
Other:
- board size 165.1 x 100.3 mm -> 147.3 x 100.3 mm
Changed lines of the file:
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@@
   (general
     (thickness 1.6)
-    (drawings 13)
+    (drawings 15)
     (tracks 207)
     (zones 0)
@@
   )
   (module MountingHole:MountingHole_3.2mm_M3_Pad_Via (layer F.Cu)
-    (at 203.073 43.561)
+    (at 203.073 42.545)
     (descr "Mounting Hole 3.2mm, M3")
     (tags "mounting hole 3.2mm m3")
@@
   )
   (module MountingHole:MountingHole_3.2mm_M3_Pad_Via (layer F.Cu)
-    (at 67.183 43.688)
+    (at 67.183 42.545)
     (descr "Mounting Hole 3.2mm, M3")
     (tags "mounting hole 3.2mm m3")
@@
     )
   )
+  (dimension 5.715 (width 0.15) (layer Dwgs.User)
+    (gr_text "5.715 mm" (at 72.293 39.6875 90) (layer Dwgs.User)
+      (effects (font (size 1 1) (thickness 0.15)))
+    )
+    (feature1 (pts (xy 61.214 36.83) (xy 71.579421 36.83)))
+    (feature2 (pts (xy 61.214 42.545) (xy 71.579421 42.545)))
+    (crossbar (pts (xy 70.993 42.545) (xy 70.993 36.83)))
+    (arrow1a (pts (xy 70.993 36.83) (xy 71.579421 37.956504)))
+    (arrow1b (pts (xy 70.993 36.83) (xy 70.406579 37.956504)))
+    (arrow2a (pts (xy 70.993 42.545) (xy 71.579421 41.418496)))
+    (arrow2b (pts (xy 70.993 42.545) (xy 70.406579 41.418496)))
+  )
+  (dimension 5.715 (width 0.15) (layer Dwgs.User)
+    (gr_text "5.715 mm" (at 205.9305 39.213) (layer Dwgs.User)
+      (effects (font (size 1 1) (thickness 0.15)))
+    )
+    (feature1 (pts (xy 203.073 44.196) (xy 203.073 39.926579)))
+    (feature2 (pts (xy 208.788 44.196) (xy 208.788 39.926579)))
+    (crossbar (pts (xy 208.788 40.513) (xy 203.073 40.513)))
+    (arrow1a (pts (xy 203.073 40.513) (xy 204.199504 39.926579)))
+    (arrow1b (pts (xy 203.073 40.513) (xy 204.199504 41.099421)))
+    (arrow2a (pts (xy 208.788 40.513) (xy 207.661496 39.926579)))
+    (arrow2b (pts (xy 208.788 40.513) (xy 207.661496 41.099421)))
+  )
   (dimension 17.78 (width 0.15) (layer Dwgs.User)
     (gr_text "17.780 mm" (at 127.254 91.664) (layer Dwgs.User)
@@
     (arrow2b (pts (xy 176.8475 28.2575) (xy 177.974004 27.671079)))
   )
-  (gr_line (start 62.23 137.16) (end 62.23 36.83) (layer Edge.Cuts) (width 0.05))
-  (gr_line (start 222.25 137.16) (end 62.23 137.16) (layer Edge.Cuts) (width 0.05))
-  (gr_line (start 227.33 36.83) (end 227.33 137.16) (layer Edge.Cuts) (width 0.05))
-  (gr_line (start 62.23 36.83) (end 222.25 36.83) (layer Edge.Cuts) (width 0.05))
+  (gr_line (start 61.468 137.16) (end 61.468 36.83) (layer Edge.Cuts) (width 0.05))
+  (gr_line (start 208.788 137.16) (end 61.468 137.16) (layer Edge.Cuts) (width 0.05))
+  (gr_line (start 208.788 36.83) (end 208.788 137.16) (layer Edge.Cuts) (width 0.05))
+  (gr_line (start 61.468 36.83) (end 208.788 36.83) (layer Edge.Cuts) (width 0.05))
   (dimension 29.21 (width 0.15) (layer Dwgs.User)
     (gr_text "29.210 mm" (at 44.928 45.085 90) (layer Dwgs.User)

Commit message: Update amp-mosfet-160w.kicad_pcb
Parts:
- moved MK3 222.6 mm to (67.2, 131.4)
- moved MK4 124.9 mm to (203.1, 131.4)
Changed lines of the file:
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@@
   (general
     (thickness 1.6)
-    (drawings 15)
+    (drawings 4)
     (tracks 207)
     (zones 0)
@@
   )
   (module MountingHole:MountingHole_3.2mm_M3_Pad_Via (layer F.Cu)
-    (at 268.397056 24.972944)
+    (at 203.073 131.445)
     (descr "Mounting Hole 3.2mm, M3")
     (tags "mounting hole 3.2mm m3")
@@
   )
   (module MountingHole:MountingHole_3.2mm_M3_Pad_Via (layer F.Cu)
-    (at 269.24 38.1)
+    (at 67.183 131.445)
     (descr "Mounting Hole 3.2mm, M3")
     (tags "mounting hole 3.2mm m3")
@@
     )
   )
-  (dimension 5.715 (width 0.15) (layer Dwgs.User)
-    (gr_text "5.715 mm" (at 72.293 39.6875 90) (layer Dwgs.User)
-      (effects (font (size 1 1) (thickness 0.15)))
-    )
-    (feature1 (pts (xy 61.214 36.83) (xy 71.579421 36.83)))
-    (feature2 (pts (xy 61.214 42.545) (xy 71.579421 42.545)))
-    (crossbar (pts (xy 70.993 42.545) (xy 70.993 36.83)))
-    (arrow1a (pts (xy 70.993 36.83) (xy 71.579421 37.956504)))
-    (arrow1b (pts (xy 70.993 36.83) (xy 70.406579 37.956504)))
-    (arrow2a (pts (xy 70.993 42.545) (xy 71.579421 41.418496)))
-    (arrow2b (pts (xy 70.993 42.545) (xy 70.406579 41.418496)))
-  )
-  (dimension 5.715 (width 0.15) (layer Dwgs.User)
-    (gr_text "5.715 mm" (at 205.9305 39.213) (layer Dwgs.User)
-      (effects (font (size 1 1) (thickness 0.15)))
-    )
-    (feature1 (pts (xy 203.073 44.196) (xy 203.073 39.926579)))
-    (feature2 (pts (xy 208.788 44.196) (xy 208.788 39.926579)))
-    (crossbar (pts (xy 208.788 40.513) (xy 203.073 40.513)))
-    (arrow1a (pts (xy 203.073 40.513) (xy 204.199504 39.926579)))
-    (arrow1b (pts (xy 203.073 40.513) (xy 204.199504 41.099421)))
-    (arrow2a (pts (xy 208.788 40.513) (xy 207.661496 39.926579)))
-    (arrow2b (pts (xy 208.788 40.513) (xy 207.661496 41.099421)))
-  )
-  (dimension 17.78 (width 0.15) (layer Dwgs.User)
-    (gr_text "17.780 mm" (at 127.254 91.664) (layer Dwgs.User)
-      (effects (font (size 1 1) (thickness 0.15)))
-    )
-    (feature1 (pts (xy 118.364 100.203) (xy 118.364 92.377579)))
-    (feature2 (pts (xy 136.144 100.203) (xy 136.144 92.377579)))
-    (crossbar (pts (xy 136.144 92.964) (xy 118.364 92.964)))
-    (arrow1a (pts (xy 118.364 92.964) (xy 119.490504 92.377579)))
-    (arrow1b (pts (xy 118.364 92.964) (xy 119.490504 93.550421)))
-    (arrow2a (pts (xy 136.144 92.964) (xy 135.017496 92.377579)))
-    (arrow2b (pts (xy 136.144 92.964) (xy 135.017496 93.550421)))
-  )
-  (dimension 10.033 (width 0.15) (layer Dwgs.User)
-    (gr_text "10.033 mm" (at 69.9135 50.897) (layer Dwgs.User)
-      (effects (font (size 1 1) (thickness 0.15)))
-    )
-    (feature1 (pts (xy 64.897 63.5) (xy 64.897 51.610579)))
-    (feature2 (pts (xy 74.93 63.5) (xy 74.93 51.610579)))
-    (crossbar (pts (xy 74.93 52.197) (xy 64.897 52.197)))
-    (arrow1a (pts (xy 64.897 52.197) (xy 66.023504 51.610579)))
-    (arrow1b (pts (xy 64.897 52.197) (xy 66.023504 52.783421)))
-    (arrow2a (pts (xy 74.93 52.197) (xy 73.803496 51.610579)))
-    (arrow2b (pts (xy 74.93 52.197) (xy 73.803496 52.783421)))
-  )
-  (dimension 10.033 (width 0.15) (layer Dwgs.User)
-    (gr_text "10.033 mm" (at 200.2155 71.785) (layer Dwgs.User)
-      (effects (font (size 1 1) (thickness 0.15)))
-    )
-    (feature1 (pts (xy 195.199 63.5) (xy 195.199 71.071421)))
-    (feature2 (pts (xy 205.232 63.5) (xy 205.232 71.071421)))
-    (crossbar (pts (xy 205.232 70.485) (xy 195.199 70.485)))
-    (arrow1a (pts (xy 195.199 70.485) (xy 196.325504 69.898579)))
-    (arrow1b (pts (xy 195.199 70.485) (xy 196.325504 71.071421)))
-    (arrow2a (pts (xy 205.232 70.485) (xy 204.105496 69.898579)))
-    (arrow2b (pts (xy 205.232 70.485) (xy 204.105496 71.071421)))
-  )
-  (dimension 10.033 (width 0.15) (layer Dwgs.User)
-    (gr_text "10.033 mm" (at 69.9135 71.785) (layer Dwgs.User)
-      (effects (font (size 1 1) (thickness 0.15)))
-    )
-    (feature1 (pts (xy 64.897 63.5) (xy 64.897 71.071421)))
-    (feature2 (pts (xy 74.93 63.5) (xy 74.93 71.071421)))
-    (crossbar (pts (xy 74.93 70.485) (xy 64.897 70.485)))
-    (arrow1a (pts (xy 64.897 70.485) (xy 66.023504 69.898579)))
-    (arrow1b (pts (xy 64.897 70.485) (xy 66.023504 71.071421)))
-    (arrow2a (pts (xy 74.93 70.485) (xy 73.803496 69.898579)))
-    (arrow2b (pts (xy 74.93 70.485) (xy 73.803496 71.071421)))
-  )
-  (dimension 2.54 (width 0.15) (layer Dwgs.User)
-    (gr_text "2.540 mm" (at 142.621 37.943) (layer Dwgs.User)
-      (effects (font (size 1 1) (thickness 0.15)))
-    )
-    (feature1 (pts (xy 143.891 43.307) (xy 143.891 38.656579)))
-    (feature2 (pts (xy 141.351 43.307) (xy 141.351 38.656579)))
-    (crossbar (pts (xy 141.351 39.243) (xy 143.891 39.243)))
-    (arrow1a (pts (xy 143.891 39.243) (xy 142.764496 39.829421)))
-    (arrow1b (pts (xy 143.891 39.243) (xy 142.764496 38.656579)))
-    (arrow2a (pts (xy 141.351 39.243) (xy 142.477504 39.829421)))
-    (arrow2b (pts (xy 141.351 39.243) (xy 142.477504 38.656579)))
-  )
-  (dimension 5.08 (width 0.15) (layer Dwgs.User)
-    (gr_text "5.080 mm" (at 179.3875 26.9575) (layer Dwgs.User)
-      (effects (font (size 1 1) (thickness 0.15)))
-    )
-    (feature1 (pts (xy 181.9275 35.982608) (xy 181.9275 27.671079)))
-    (feature2 (pts (xy 176.8475 35.982608) (xy 176.8475 27.671079)))
-    (crossbar (pts (xy 176.8475 28.2575) (xy 181.9275 28.2575)))
-    (arrow1a (pts (xy 181.9275 28.2575) (xy 180.800996 28.843921)))
-    (arrow1b (pts (xy 181.9275 28.2575) (xy 180.800996 27.671079)))
-    (arrow2a (pts (xy 176.8475 28.2575) (xy 177.974004 28.843921)))
-    (arrow2b (pts (xy 176.8475 28.2575) (xy 177.974004 27.671079)))
-  )
   (gr_line (start 61.468 137.16) (end 61.468 36.83) (layer Edge.Cuts) (width 0.05))
   (gr_line (start 208.788 137.16) (end 61.468 137.16) (layer Edge.Cuts) (width 0.05))
   (gr_line (start 208.788 36.83) (end 208.788 137.16) (layer Edge.Cuts) (width 0.05))
   (gr_line (start 61.468 36.83) (end 208.788 36.83) (layer Edge.Cuts) (width 0.05))
-  (dimension 29.21 (width 0.15) (layer Dwgs.User)
-    (gr_text "29.210 mm" (at 44.928 45.085 90) (layer Dwgs.User)
-      (effects (font (size 1 1) (thickness 0.15)))
-    )
-    (feature1 (pts (xy 65.278 30.48) (xy 45.641579 30.48)))
-    (feature2 (pts (xy 65.278 59.69) (xy 45.641579 59.69)))
-    (crossbar (pts (xy 46.228 59.69) (xy 46.228 30.48)))
-    (arrow1a (pts (xy 46.228 30.48) (xy 46.814421 31.606504)))
-    (arrow1b (pts (xy 46.228 30.48) (xy 45.641579 31.606504)))
-    (arrow2a (pts (xy 46.228 59.69) (xy 46.814421 58.563496)))
-    (arrow2b (pts (xy 46.228 59.69) (xy 45.641579 58.563496)))
-  )
-  (dimension 100.33 (width 0.15) (layer Dwgs.User)
-    (gr_text "100.330 mm" (at 29.688 88.265 270) (layer Dwgs.User)
-      (effects (font (size 1 1) (thickness 0.15)))
-    )
-    (feature1 (pts (xy 62.738 138.43) (xy 30.401579 138.43)))
-    (feature2 (pts (xy 62.738 38.1) (xy 30.401579 38.1)))
-    (crossbar (pts (xy 30.988 38.1) (xy 30.988 138.43)))
-    (arrow1a (pts (xy 30.988 138.43) (xy 30.401579 137.303496)))
-    (arrow1b (pts (xy 30.988 138.43) (xy 31.574421 137.303496)))
-    (arrow2a (pts (xy 30.988 38.1) (xy 30.401579 39.226504)))
-    (arrow2b (pts (xy 30.988 38.1) (xy 31.574421 39.226504)))
-  )
-  (dimension 160.02 (width 0.15) (layer Dwgs.User)
-    (gr_text "160.020 mm" (at 147.32 21.56) (layer Dwgs.User)
-      (effects (font (size 1 1) (thickness 0.15)))
-    )
-    (feature1 (pts (xy 227.33 38.1) (xy 227.33 22.273579)))
-    (feature2 (pts (xy 67.31 38.1) (xy 67.31 22.273579)))
-    (crossbar (pts (xy 67.31 22.86) (xy 227.33 22.86)))
-    (arrow1a (pts (xy 227.33 22.86) (xy 226.203496 23.446421)))
-    (arrow1b (pts (xy 227.33 22.86) (xy 226.203496 22.273579)))
-    (arrow2a (pts (xy 67.31 22.86) (xy 68.436504 23.446421)))
-    (arrow2b (pts (xy 67.31 22.86) (xy 68.436504 22.273579)))
-  )
   (segment (start 101.5365 122.4445) (end 101.553 122.428) (width 0.5) (layer B.Cu) (net 1))
   (segment (start 101.5365 130.2385) (end 101.5365 122.4445) (width 0.5) (layer B.Cu) (net 1))

Commit message: Ready to order V1
Parts:
- D1, D3: value 1N4148 -> 1N914
- R11: value 22k -> 33k
- moved MK1 1.65 mm to (65.5, 42.5)
- moved MK3 1.57 mm to (65.6, 131.4)
- moved MK2 1.40 mm to (204.5, 42.5)
- moved MK4 1.40 mm to (204.5, 131.4)
Other:
- board size 147.3 x 100.3 mm -> 150.4 x 100.3 mm
- board text added: "+69V"
- board text added: "-69V"
- board text added: "IN"
- board text added: "IN_GND"
- board text added: "LS+"
- board text added: "LS-"
- board text added: "Lateral MOSFET Power Amplifier 160W V1 2021.11.16"
- board text added: "michaelschenk72@gmail.com"
- board text added: "°"
