File: amp-mosfet-80W/kicad/V3/amp-mosfet-80w.kicad_pcb (KiCad board)
At the start: 2 copper layers, 100.3 x 55.2 mm, 60 parts, among them J1 Conn_01x01, J2 Conn_01x01, J3 +50V, J4 -50V, J5 LS+, J6 LS-, J7 GND, Q1 BC856BS, Q11 ECX10P20, Q12 ECX10N20, Q2 BC856BS, Q3 DZT5551, Q4 DZT5401, Q5 DZT5401, Q6 DZT5551

Commit message: WIP
Parts:
- removed C17: 470p, Capacitor_SMD:C_0805_2012Metric_Pad1.18x1.45mm_HandSolder
- added Q7: BC856B, Package_TO_SOT_SMD:SOT-23, F.Cu at (172.1, 62.4)
- added Q8: BC846, Package_TO_SOT_SMD:SOT-23, F.Cu at (141.8, 65.0)
- added R13: 1k, Resistor_SMD:R_0805_2012Metric_Pad1.20x1.40mm_HandSolder, F.Cu at (175.0, 115.9)
- added R15: 100R, Resistor_SMD:R_0805_2012Metric_Pad1.20x1.40mm_HandSolder, F.Cu at (179.8, 118.8)
- added R16: 22k, Resistor_SMD:R_0805_2012Metric_Pad1.20x1.40mm_HandSolder, F.Cu at (122.9, 71.6)
- added R22: 100R, Resistor_SMD:R_0805_2012Metric_Pad1.20x1.40mm_HandSolder, F.Cu at (179.8, 109.9)
- added R23: 2.2k, Resistor_SMD:R_0805_2012Metric_Pad1.20x1.40mm_HandSolder, F.Cu at (184.6, 109.9)
- added R24: 2.2k, Resistor_SMD:R_0805_2012Metric_Pad1.20x1.40mm_HandSolder, F.Cu at (179.8, 112.9)
- added R25: 33R, Resistor_SMD:R_0805_2012Metric_Pad1.20x1.40mm_HandSolder, F.Cu at (175.0, 113.0)
- C1: value 2.2uF -> 3.3uF
- C3: value 10n -> 47p; footprint Capacitor_THT:C_Rect_L7.2mm_W2.5mm_P5.00mm_FKS2_FKP2_MKS2_MKP2 -> Capacitor_SMD:C_0805_2012Metric_Pad1.18x1.45mm_HandSolder
- C8: value 18p -> 47p
- Q3: value DZT5551 -> BC856BS; footprint Package_TO_SOT_SMD:SOT-223-3_TabPin2 -> Package_TO_SOT_SMD:SOT-363_SC-70-6
- Q4: value DZT5401 -> BC846BDW1; footprint Package_TO_SOT_SMD:SOT-223-3_TabPin2 -> Package_TO_SOT_SMD:SOT-363_SC-70-6
- R12: value 100R -> 220R
- R20: value 100R -> 33R
- R4, R7: value 3k9 -> 1k
- R5: value 430R -> 220R
- R6: value 22k -> 100R
- R8: value 100R -> 1k
- R9: value 12k/1W -> 100R; footprint Resistor_SMD:R_1206_3216Metric_Pad1.30x1.75mm_HandSolder -> Resistor_SMD:R_0805_2012Metric_Pad1.20x1.40mm_HandSolder
- moved Q3 60.3 mm to (184.3, 116.3), turned to 0 degrees
- moved R9 56.2 mm to (189.3, 109.9), turned to 0 degrees
- moved R8 47.7 mm to (175.0, 118.9), turned to 0 degrees
- moved Q4 43.6 mm to (127.4, 70.6), turned to 0 degrees
- moved R12 18.4 mm to (124.0, 68.6), turned to 0 degrees
- moved C3 14.7 mm to (176.3, 63.0), turned to 0 degrees
- moved C8 7.52 mm to (146.3, 64.0)
Connections:
- C2 pad 1: Net-(C2-Pad1) -> Net-(Q1-Pad2)
- C3 pad 1: Net-(Q4-Pad1) -> Net-(C7-Pad2)
- C3 pad 2: Net-(Q3-Pad2) -> Net-(C3-Pad2)
- C5 pad 2: Net-(C5-Pad2) -> Net-(Q1-Pad5)
- C8 pad 1: Net-(C8-Pad1) -> Net-(C7-Pad1)
- C8 pad 2: Net-(C7-Pad1) -> Net-(Q1-Pad6)
- Q1 pad 2: Net-(C2-Pad1) -> Net-(Q1-Pad2)
- Q1 pad 3: Net-(Q1-Pad3) -> Net-(R7-Pad1)
- Q1 pad 4: Net-(Q1-Pad1) -> Net-(Q1-Pad4)
- Q1 pad 5: Net-(C5-Pad2) -> Net-(Q1-Pad5)
- Q1 pad 6: Net-(C8-Pad1) -> Net-(Q1-Pad6)
- Q3 pad 1: Net-(Q1-Pad3) -> Net-(Q3-Pad1)
- Q3 pad 2: Net-(Q3-Pad2) -> Net-(Q1-Pad5)
- Q3 pad 3: Net-(Q3-Pad3) -> Net-(C3-Pad2)
- Q4 pad 2: Net-(Q4-Pad1) -> Net-(Q4-Pad2)
- Q4 pad 3: Net-(Q4-Pad3) -> Net-(Q4-Pad2)
- Q5 pad 1: Net-(Q4-Pad1) -> Net-(Q5-Pad1)
- Q6 pad 1: Net-(C8-Pad1) -> Net-(Q6-Pad1)
- Q6 pad 3: Net-(Q3-Pad3) -> Net-(Q6-Pad3)
- R10 pad 1: Net-(C5-Pad2) -> Net-(Q1-Pad5)
- R11 pad 2: Net-(C5-Pad2) -> Net-(Q1-Pad5)
- R12 pad 1: Net-(Q3-Pad3) -> Net-(C10-Pad2)
- R12 pad 2: Net-(C10-Pad2) -> Net-(Q4-Pad1)
- R2 pad 1: Net-(C2-Pad1) -> Net-(Q1-Pad2)
- R4 pad 1: Net-(C8-Pad1) -> Net-(Q1-Pad6)
- R7 pad 1: Net-(Q1-Pad3) -> Net-(R7-Pad1)
- R8 pad 1: Net-(C11-Pad1) -> Net-(C3-Pad2)
- R8 pad 2: Net-(Q4-Pad3) -> Net-(C11-Pad1)
- R9 pad 1: Net-(Q4-Pad1) -> Net-(Q4-Pad6)
- R9 pad 2: Net-(Q3-Pad2) -> Net-(Q3-Pad4)
Routing:
- net Net-(C11-Pad1): track 61.9 -> 16.4 mm
- net Net-(Q4-Pad1): track 30.1 -> 0.00 mm
- net Net-(C8-Pad1): track 21.5 -> 0.00 mm, vias 2 -> 0
- net Net-(Q3-Pad2): track 21.3 -> 0.00 mm
- net Net-(Q1-Pad3): track 18.0 -> 0.00 mm, vias 2 -> 0
- net Net-(Q1-Pad5): track 0.00 -> 17.1 mm
- net Net-(C5-Pad2): track 17.1 -> 0.00 mm
- net Net-(Q1-Pad6): track 0.00 -> 17.1 mm, vias 0 -> 2
- net Net-(Q3-Pad3): track 8.42 -> 0.00 mm
- net Net-(Q1-Pad2): track 0.00 -> 7.55 mm
- net Net-(C2-Pad1): track 7.55 -> 0.00 mm
- net Net-(Q4-Pad3): track 5.48 -> 0.00 mm
- net Net-(Q1-Pad1): track 4.78 -> 0.00 mm
- net Net-(C10-Pad2): track 56.1 -> 51.7 mm
- net Net-(Q12-Pad1): track 6.57 -> 3.46 mm
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- removed copper zone on F.Cu, net Net-(Q3-Pad2)
- removed copper zone on F.Cu, net Net-(Q4-Pad1)

Commit message: WIP
Parts:
- removed JP1, JP2: Jump, Connector_PinHeader_2.54mm:PinHeader_1x02_P2.54mm_Vertical
- moved R24 60.6 mm to (141.2, 66.2)
- moved R25 59.6 mm to (142.2, 63.2), turned to -90 degrees
- moved R15 50.7 mm to (168.5, 69.3)
- moved R8 48.3 mm to (174.4, 70.6)
- moved R22 47.9 mm to (148.1, 74.1), turned to 180 degrees
- moved Q3 46.1 mm to (170.2, 72.4), turned to -90 degrees
- moved R23 44.1 mm to (179.7, 66.2), turned to 180 degrees
- moved R9 43.5 mm to (167.5, 72.3), turned to -90 degrees
- moved R13 42.6 mm to (174.4, 73.3)
- moved R12 14.9 mm to (137.3, 75.2), turned to 180 degrees
- moved R16 11.2 mm to (133.6, 75.2), turned to 180 degrees
- moved R4 9.65 mm to (141.2, 75.2), turned to 180 degrees
- moved Q4 9.16 mm to (136.3, 72.8)
- moved C8 6.42 mm to (140.0, 63.2), turned to -90 degrees
- moved Q8 4.73 mm to (137.1, 65.2), turned to -90 degrees
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Connections:
- C18 pad 2: Net-(C18-Pad2) -> Net-(D6-Pad1)
- D5 pad 2: Net-(D5-Pad2) -> Net-(C14-Pad1)
- J4 pad 1: Net-(C18-Pad2) -> Net-(D6-Pad1)
- Q11 pad 3: Net-(C18-Pad2) -> Net-(D6-Pad1)
- Q8 pad 3: unconnected-(Q8-Pad3) -> GND
Routing:
- net Net-(C18-Pad2): track 36.5 -> 0.00 mm
- net Net-(D6-Pad1): track 2.86 -> 39.2 mm
- net GND: track 259.4 -> 292.3 mm, vias 0 -> 1
- net Net-(Q4-Pad6): track 0.00 -> 32.8 mm, vias 0 -> 2
- net Net-(Q1-Pad2): track 7.55 -> 28.5 mm, vias 0 -> 1
- net Net-(Q1-Pad5): track 17.1 -> 32.9 mm
- net Net-(R6-Pad1): track 24.6 -> 10.2 mm
- net Net-(Q6-Pad1): track 0.00 -> 9.93 mm
- net Net-(Q4-Pad1): track 0.00 -> 4.84 mm
- net Net-(C3-Pad2): track 0.00 -> 4.74 mm, vias 0 -> 2
- net Net-(C10-Pad2): track 51.7 -> 47.8 mm
- net Net-(Q1-Pad1): track 0.00 -> 3.72 mm
- net Net-(Q4-Pad2): track 0.00 -> 2.80 mm
- net Net-(D5-Pad2): track 2.79 -> 0.00 mm
- net Net-(Q3-Pad1): track 0.00 -> 2.63 mm
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Other:
- board text added: "Lateral MOSFET Power Amplifier 80W V3 2022.01.01"
- board text removed: "Lateral MOSFET Power Amplifier 80W V2 2021.12.28"

Commit message: Layout completed
Parts:
- moved R3 4.26 mm to (174.1, 80.8), turned to 0 degrees
- moved R5 3.22 mm to (171.8, 77.2), turned to 180 degrees
Routing:
- net Net-(C11-Pad1): track 15.6 -> 58.1 mm
- net GND: track 292.3 -> 307.4 mm, vias 1 -> 3
- net Net-(R6-Pad1): track 10.2 -> 24.6 mm
- net Net-(C3-Pad2): track 4.74 -> 15.0 mm, vias 2 -> 3
- net Net-(Q5-Pad1): track 0.00 -> 9.72 mm
- net Net-(Q1-Pad2): track 28.5 -> 36.3 mm, vias 1 -> 2
- net Net-(Q3-Pad6): track 0.00 -> 2.59 mm
- net Net-(Q5-Pad3): track 0.02 -> 2.21 mm
- net Net-(C7-Pad2): track 43.5 -> 45.7 mm
- net Net-(C7-Pad1): track 48.1 -> 50.3 mm
- net Net-(Q3-Pad4): track 0.00 -> 2.07 mm
- net Net-(C10-Pad2): track 47.8 -> 49.7 mm
- net Net-(Q2-Pad1): track 5.63 -> 3.89 mm

Commit message: Update amp-mosfet-80w.kicad_pcb
Routing:
- net Net-(C13-Pad1): track 104.0 -> 100.8 mm
