File: amp-mosfet-80W/kicad/V4/amp-mosfet-80w.kicad_pcb (KiCad board)
At the start: 2 copper layers, 100.3 x 55.2 mm, 59 parts, among them J1 Conn_01x01, J2 Conn_01x01, J3 +50V, J4 -50V, J5 LS+, J6 LS-, J7 GND, Q1 BC856BS, Q11 ECX10P20, Q12 ECX10N20, Q2 BC856BS, Q3 BC846BDW1, Q4 BC846B, Q5 BC856B, Q6 DZT5551, Q7 DZT5401, Q8 BC846

Commit message: WIP
Parts:
- added C15: 1n, Capacitor_SMD:C_0805_2012Metric_Pad1.18x1.45mm_HandSolder, F.Cu at (129.6, 68.2)
- added C3: 100p, Capacitor_SMD:C_0805_2012Metric_Pad1.18x1.45mm_HandSolder, F.Cu at (140.7, 89.2)
- added R12: 68R, Resistor_SMD:R_0805_2012Metric_Pad1.20x1.40mm_HandSolder, F.Cu at (138.4, 91.1)
- added R13: 1k, Resistor_SMD:R_0805_2012Metric_Pad1.20x1.40mm_HandSolder, F.Cu at (126.0, 72.2)
- added R15: 4k7, Resistor_SMD:R_0805_2012Metric_Pad1.20x1.40mm_HandSolder, F.Cu at (124.1, 66.2)
- added R16: 470R, Resistor_SMD:R_0805_2012Metric_Pad1.20x1.40mm_HandSolder, F.Cu at (136.0, 61.9)
- C2: value 1n -> 470p; footprint Capacitor_THT:C_Rect_L7.2mm_W2.5mm_P5.00mm_FKS2_FKP2_MKS2_MKP2 -> Capacitor_SMD:C_0805_2012Metric_Pad1.18x1.45mm_HandSolder
- Q8: value BC846 -> BC846B
- R24: value 470R -> 1k
- R25: value 22R -> 33R
- R4, R7: value 470 -> 220
- R5: value 430R -> 180R
- R9: value 100R (70R) -> 75R
- moved Q3 40.1 mm to (130.1, 71.0)
- moved R7 21.5 mm to (125.2, 69.7)
- moved R9 13.4 mm to (180.4, 68.8)
- moved R4 11.4 mm to (129.8, 75.1)
- moved Q7 8.81 mm to (178.4, 56.9), turned to 90 degrees
- moved Q5 7.28 mm to (178.9, 64.1), turned to -90 degrees
- moved C1 3.71 mm to (140.9, 82.4)
- moved Q4 2.70 mm to (134.4, 70.8)
Connections:
- C7 pad 1: Net-(C7-Pad2) -> Net-(C7-Pad1)
- C8 pad 1: Net-(C7-Pad2) -> Net-(C7-Pad1)
- D4 pad 2: Net-(C7-Pad2) -> Net-(C7-Pad1)
- J1 pad 1: Net-(C1-Pad2) -> Net-(J1-Pad1)
- Q6 pad 1: Net-(Q8-Pad2) -> Net-(Q6-Pad1)
- Q6 pad 2: Net-(C7-Pad2) -> Net-(C7-Pad1)
- R14 pad 2: Net-(C7-Pad2) -> Net-(C7-Pad1)
- RV1 pad 2: Net-(C7-Pad2) -> Net-(C7-Pad1)
- RV1 pad 3: Net-(C7-Pad2) -> Net-(C7-Pad1)
Routing:
- net Net-(C11-Pad1): track 90.8 -> 16.3 mm, vias 2 -> 0
- net Net-(C7-Pad2): track 105.7 -> 36.8 mm
- net Net-(C7-Pad1): track 0.00 -> 48.1 mm
- net GND: track 307.3 -> 262.6 mm, vias 3 -> 2
- net Net-(Q1-Pad2): track 36.3 -> 0.00 mm, vias 2 -> 0
- net Net-(C10-Pad2): track 49.6 -> 13.4 mm
- net Net-(Q1-Pad3): track 21.7 -> 0.00 mm, vias 3 -> 0
- net Net-(C5-Pad2): track 32.9 -> 16.6 mm
- net Net-(Q1-Pad6): track 19.1 -> 5.58 mm, vias 2 -> 1
- net Net-(Q8-Pad2): track 9.93 -> 0.00 mm
- net Net-(C1-Pad2): track 5.72 -> 0.00 mm
- net Net-(Q3-Pad5): track 2.80 -> 0.00 mm
- net Net-(Q3-Pad1): track 2.63 -> 0.00 mm
- net Net-(C1-Pad1): track 4.33 -> 1.78 mm
- net Net-(Q5-Pad3): track 2.21 -> 0.00 mm
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- added copper zone on F.Cu, net Net-(C7-Pad1)
Other:
- board text added: "Lateral MOSFET Power Amplifier 80W V4 2022.01.23"
- board text removed: "Lateral MOSFET Power Amplifier 80W V3 2022.01.01"

Commit message: WIP
Parts:
- added C16: 1n, Capacitor_THT:C_Rect_L7.2mm_W2.5mm_P5.00mm_FKS2_FKP2_MKS2_MKP2, F.Cu at (146.0, 83.1)
- R2: value 1k -> 470R
- moved C15 12.3 mm to (133.0, 80.0), turned to 180 degrees
- moved Q4 12.2 mm to (132.8, 83.0), turned to -90 degrees
- moved R15 12.0 mm to (132.9, 74.4), turned to 180 degrees
- moved R7 7.42 mm to (132.2, 72.3)
- moved Q3 6.79 mm to (132.5, 77.3), turned to 90 degrees
- moved R13 6.04 mm to (129.2, 77.3), turned to 180 degrees
- moved R6 4.44 mm to (145.8, 80.0)
- moved R4 4.30 mm to (129.2, 79.3)
- moved R8 2.75 mm to (176.1, 68.4), turned to -90 degrees
- moved R22 2.55 mm to (149.2, 76.4)
- moved C2 2.47 mm to (146.0, 85.6)
- moved C1 2.39 mm to (138.5, 82.4), turned to -90 degrees
- moved Q8 2.12 mm to (137.6, 67.3)
- moved R16 2.10 mm to (137.7, 63.2), turned to -90 degrees
- moved C3 1.67 mm to (140.6, 90.9), turned to 90 degrees
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Routing:
- net Net-(C5-Pad2): track 16.6 -> 4.04 mm
- net GND: track 262.6 -> 253.0 mm, vias 2 -> 1
- net Net-(Q1-Pad2): track 0.00 -> 9.62 mm
- net Net-(Q1-Pad6): track 5.58 -> 0.00 mm, vias 1 -> 0
- net Net-(Q3-Pad5): track 0.00 -> 4.25 mm
- net Net-(Q3-Pad1): track 0.00 -> 2.13 mm
- net Net-(Q1-Pad1): track 3.72 -> 1.84 mm
- net Net-(R6-Pad1): track 24.6 -> 26.4 mm

Commit message: Update amp-mosfet-80w.kicad_pcb
Parts:
- moved Q4 11.6 mm to (142.3, 76.4), turned to 180 degrees
- moved C15 6.67 mm to (139.6, 79.2)
- moved R15 6.43 mm to (139.2, 73.1)
- moved Q3 6.25 mm to (138.6, 75.8)
- moved R13 6.25 mm to (135.2, 75.8)
- moved R4 6.25 mm to (135.2, 77.8)
- moved R7 6.16 mm to (138.2, 71.2)
- moved C16 3.50 mm to (148.3, 85.7)
- moved C2 3.50 mm to (148.3, 88.2)
- moved J1 3.50 mm to (138.2, 94.5)
- moved J2 3.50 mm to (145.7, 94.5)
- moved R1 3.50 mm to (145.7, 89.7)
- moved R2 3.50 mm to (145.7, 86.0)
- moved C1 3.50 mm to (140.8, 85.0)
- moved R12 3.47 mm to (140.8, 93.4)
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Routing:
- net Net-(C10-Pad2): track 13.4 -> 50.7 mm, vias 0 -> 2
- net GND: track 253.0 -> 283.8 mm, vias 1 -> 3
- net Net-(Q1-Pad6): track 0.00 -> 20.2 mm, vias 0 -> 2
- net Net-(Q1-Pad3): track 0.00 -> 14.3 mm
- net Net-(C5-Pad2): track 4.04 -> 14.5 mm
- net Net-(Q3-Pad5): track 4.25 -> 11.4 mm, vias 0 -> 2
- net Net-(Q8-Pad2): track 0.00 -> 6.74 mm, vias 0 -> 2
- net Net-(C1-Pad1): track 1.78 -> 7.52 mm
- net Net-(C1-Pad2): track 0.00 -> 4.46 mm
- net Net-(Q3-Pad4): track 0.00 -> 3.67 mm
- net Net-(J1-Pad1): track 0.00 -> 2.63 mm
- net Net-(Q6-Pad3): track 0.00 -> 2.18 mm
- net Net-(C7-Pad1): track 48.1 -> 50.3 mm
- net Net-(Q6-Pad1): track 0.00 -> 2.18 mm
- net Net-(Q1-Pad2): track 9.62 -> 11.6 mm

Commit message: Update amp-mosfet-80w.kicad_pcb
Parts:
- moved Q5 1.10 mm to (179.8, 63.4)
Routing:
- net Net-(C7-Pad2): track 36.8 -> 43.1 mm
Changed lines of the file:
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@@
     (property "Sheetname" "")
     (attr smd)
-    (fp_text reference "C2" (at 0 -1.68 -90) (layer "F.SilkS")
+    (fp_text reference "C2" (at 0 -2.2 -90) (layer "F.SilkS")
       (effects (font (size 1 1) (thickness 0.15)))
     )
@@
     (property "Sheetname" "")
     (attr through_hole)
-    (fp_text reference "J2" (at -2.6035 0) (layer "F.SilkS")
+    (fp_text reference "J2" (at 2.5035 0) (layer "F.SilkS")
       (effects (font (size 1 1) (thickness 0.15)))
     )
@@
     (property "Sheetname" "")
     (attr smd)
-    (fp_text reference "R1" (at 2.683 -0.5715 90) (layer "F.SilkS")
+    (fp_text reference "R1" (at 2.5065 -0.0035 90) (layer "F.SilkS")
       (effects (font (size 1 1) (thickness 0.15)))
     )
@@
     (property "Sheetname" "")
     (attr smd)
-    (fp_text reference "R2" (at -1.928 2.0465 180) (layer "F.SilkS")
+    (fp_text reference "R2" (at -2.7155 -0.0035 -90) (layer "F.SilkS")
       (effects (font (size 1 1) (thickness 0.15)))
     )
@@
     (property "Sheetname" "")
     (attr smd)
-    (fp_text reference "R6" (at -2.85 0 180) (layer "F.SilkS")
+    (fp_text reference "R6" (at 0 -1.5 180) (layer "F.SilkS")
       (effects (font (size 1 1) (thickness 0.15)))
     )
@@
     (property "Sheetname" "")
     (attr smd)
-    (fp_text reference "R4" (at 0 1.6) (layer "F.SilkS")
+    (fp_text reference "R4" (at 2.7 2.025) (layer "F.SilkS")
       (effects (font (size 1 1) (thickness 0.15)))
     )
@@
   )
   (footprint "Package_TO_SOT_SMD:SOT-23" (layer "F.Cu")
-    (at 178.95 64.1375 -90)
+    (at 179.8 63.4375 -90)
     (descr "SOT, 3 Pin (https://www.jedec.org/system/files/docs/to-236h.pdf variant AB), generated with kicad-footprint-generator ipc_gullwing_generator.py")
     (tags "SOT TO_SOT_SMD")
@@
     (property "Sheetname" "")
     (attr smd)
-    (fp_text reference "R15" (at 0 -1.65) (layer "F.SilkS")
+    (fp_text reference "R15" (at 3.2 -0.125) (layer "F.SilkS")
       (effects (font (size 1 1) (thickness 0.15)))
     )
@@
     (property "Sheetname" "")
     (attr smd)
-    (fp_text reference "Q3" (at 2.4354 -0.0258) (layer "F.SilkS")
+    (fp_text reference "Q3" (at -1.975 -0.0258) (layer "F.SilkS")
       (effects (font (size 1 1) (thickness 0.15)))
     )
@@
     (property "Sheetname" "")
     (attr through_hole)
-    (fp_text reference "C16" (at 2.5 -2.5 90) (layer "F.SilkS")
+    (fp_text reference "C16" (at 5.0125 -2.2 90) (layer "F.SilkS")
       (effects (font (size 1 1) (thickness 0.15)))
     )
@@
     (property "Sheetname" "")
     (attr smd)
-    (fp_text reference "R24" (at 0 1.95) (layer "F.SilkS")
+    (fp_text reference "R24" (at 3.25 0.05) (layer "F.SilkS")
       (effects (font (size 1 1) (thickness 0.15)))
     )
@@
     (property "Sheetname" "")
     (attr smd)
-    (fp_text reference "C15" (at 0 -1.68) (layer "F.SilkS")
+    (fp_text reference "C15" (at 0.1125 -1.8) (layer "F.SilkS")
       (effects (font (size 1 1) (thickness 0.15)))
     )
@@
     (property "Sheetname" "")
     (attr smd)
-    (fp_text reference "R25" (at 0 -1.65 90) (layer "F.SilkS")
+    (fp_text reference "R25" (at 0 -1.65 -90) (layer "F.SilkS")
       (effects (font (size 1 1) (thickness 0.15)))
     )
@@
     (property "Sheetname" "")
     (attr smd)
-    (fp_text reference "C8" (at -0.9421 2.054 180) (layer "F.SilkS")
+    (fp_text reference "C8" (at 0.0079 4.704 -90) (layer "F.SilkS")
       (effects (font (size 1 1) (thickness 0.15)))
     )
@@
     (property "Sheetname" "")
     (attr smd)
-    (fp_text reference "R13" (at 0 -1.65) (layer "F.SilkS")
+    (fp_text reference "R13" (at 3.2 -2.225) (layer "F.SilkS")
       (effects (font (size 1 1) (thickness 0.15)))
     )
@@
     (property "Sheetname" "")
     (attr smd)
-    (fp_text reference "Q4" (at 2.6375 -4.7) (layer "F.SilkS")
+    (fp_text reference "Q4" (at -0.6875 2.4) (layer "F.SilkS")
       (effects (font (size 1 1) (thickness 0.15)))
     )
@@
     (property "Sheetname" "")
     (attr smd)
-    (fp_text reference "R12" (at 0 -1.65 90) (layer "F.SilkS")
+    (fp_text reference "R12" (at -1.15 2.55 180) (layer "F.SilkS")
       (effects (font (size 1 1) (thickness 0.15)))
     )
@@
     (property "Sheetname" "")
     (attr smd)
-    (fp_text reference "R16" (at 0 -1.65 90) (layer "F.SilkS")
+    (fp_text reference "R16" (at 0 3.9 90) (layer "F.SilkS")
       (effects (font (size 1 1) (thickness 0.15)))
     )
@@
     (property "Sheetname" "")
     (attr smd)
-    (fp_text reference "C3" (at 0 -1.68 90) (layer "F.SilkS")
+    (fp_text reference "C3" (at -2.5625 -0.65 180) (layer "F.SilkS")
       (effects (font (size 1 1) (thickness 0.15)))
     )
@@
     (effects (font (size 1 1) (thickness 0.15)))
   )
-  (gr_text "IN" (at 135.89 94.488) (layer "F.SilkS")
+  (gr_text "IN" (at 138.25 97) (layer "F.SilkS")
     (effects (font (size 1 1) (thickness 0.15)))
   )
@@
     (effects (font (size 1 1) (thickness 0.15)))
   )
-  (gr_text "michaelschenk72@gmail.com" (at 133.477 97.282) (layer "F.SilkS")
+  (gr_text "michaelschenk72@gmail.com" (at 130.05 98.5) (layer "F.SilkS")
     (effects (font (size 1 1) (thickness 0.15)))
   )
@@
   (segment (start 166.243 51.308) (end 176.008 51.308) (width 1) (layer "F.Cu") (net 34))
   (segment (start 180.7 51.4) (end 191.989 51.4) (width 1) (layer "F.Cu") (net 34))
+  (segment (start 178.4 60) (end 178.4 53.7) (width 1) (layer "F.Cu") (net 34))
   (segment (start 161.798 51.308) (end 161.798 46.689) (width 1) (layer "B.Cu") (net 34))
   (segment (start 137.9 73.425) (end 138.2 73.125) (width 0.25) (layer "F.Cu") (net 35))

Commit message: Update amp-mosfet-80w.kicad_pcb
Parts:
- moved R9 6.00 mm to (179.7, 62.3), turned to 0 degrees
- moved Q5 1.96 mm to (179.8, 65.4)
- moved R8 1.10 mm to (176.1, 67.3)
Routing:
- net Net-(C11-Pad1): track 16.3 -> 50.7 mm, vias 0 -> 2
- net GND: track 283.8 -> 313.9 mm, vias 3 -> 4
- net Net-(Q5-Pad3): track 0.00 -> 10.0 mm
- net Net-(Q5-Pad1): track 0.00 -> 4.46 mm
Changed lines of the file:
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@@
   )
   (footprint "Package_TO_SOT_SMD:SOT-23" (layer "F.Cu")
-    (at 179.8 63.4375 -90)
+    (at 179.75 65.4 -90)
     (descr "SOT, 3 Pin (https://www.jedec.org/system/files/docs/to-236h.pdf variant AB), generated with kicad-footprint-generator ipc_gullwing_generator.py")
     (tags "SOT TO_SOT_SMD")
@@
   )
   (footprint "Resistor_SMD:R_0805_2012Metric_Pad1.20x1.40mm_HandSolder" (layer "F.Cu")
-    (at 179.9 68.3 90)
+    (at 179.7 62.3)
     (descr "Resistor SMD 0805 (2012 Metric), square (rectangular) end terminal, IPC_7351 nominal with elongated pad for handsoldering. (Body size source: IPC-SM-782 page 72, https://www.pcb-3d.com/wordpress/wp-content/uploads/ipc-sm-782a_amendment_1_and_2.pdf), generated with kicad-footprint-generator")
     (tags "resistor handsolder")
@@
     (property "Sheetname" "")
     (attr smd)
-    (fp_text reference "R9" (at -0.0298 1.5622 90) (layer "F.SilkS")
-      (effects (font (size 1 1) (thickness 0.15)))
-    )
-    (fp_text value "75R" (at 0 1.65 90) (layer "F.Fab")
-      (effects (font (size 1 1) (thickness 0.15)))
-    )
-    (fp_text user "${REFERENCE}" (at 0 0 90) (layer "F.Fab")
+    (fp_text reference "R9" (at 2.7 0) (layer "F.SilkS")
+      (effects (font (size 1 1) (thickness 0.15)))
+    )
+    (fp_text value "75R" (at 0 1.65) (layer "F.Fab")
+      (effects (font (size 1 1) (thickness 0.15)))
+    )
+    (fp_text user "${REFERENCE}" (at 0 0) (layer "F.Fab")
       (effects (font (size 0.5 0.5) (thickness 0.08)))
     )
@@
     (fp_line (start 1 -0.625) (end 1 0.625) (layer "F.Fab") (width 0.1))
     (fp_line (start 1 0.625) (end -1 0.625) (layer "F.Fab") (width 0.1))
-    (pad "1" smd roundrect locked (at -1 0 90) (size 1.2 1.4) (layers "F.Cu" "F.Paste" "F.Mask") (roundrect_rratio 0.208333)
+    (pad "1" smd roundrect locked (at -1 0) (size 1.2 1.4) (layers "F.Cu" "F.Paste" "F.Mask") (roundrect_rratio 0.208333)
       (net 9 "Net-(C11-Pad1)") (pintype "passive"))
-    (pad "2" smd roundrect locked (at 1 0 90) (size 1.2 1.4) (layers "F.Cu" "F.Paste" "F.Mask") (roundrect_rratio 0.208333)
+    (pad "2" smd roundrect locked (at 1 0) (size 1.2 1.4) (layers "F.Cu" "F.Paste" "F.Mask") (roundrect_rratio 0.208333)
       (net 29 "Net-(Q5-Pad1)") (pintype "passive"))
     (model "${KICAD6_3DMODEL_DIR}/Resistor_SMD.3dshapes/R_0805_2012Metric.wrl"
@@
   )
   (footprint "Resistor_SMD:R_0805_2012Metric_Pad1.20x1.40mm_HandSolder" (layer "F.Cu")
-    (at 176.1 68.4 -90)
+    (at 176.1 67.3 -90)
     (descr "Resistor SMD 0805 (2012 Metric), square (rectangular) end terminal, IPC_7351 nominal with elongated pad for handsoldering. (Body size source: IPC-SM-782 page 72, https://www.pcb-3d.com/wordpress/wp-content/uploads/ipc-sm-782a_amendment_1_and_2.pdf), generated with kicad-footprint-generator")
     (tags "resistor handsolder")
@@
     (effects (font (size 1 1) (thickness 0.15)))
   )
-  (gr_text "°" (at 143.5 79) (layer "F.SilkS")
+  (gr_text "°" (at 144.25 79) (layer "F.SilkS")
     (effects (font (size 1 1) (thickness 0.15)))
   )
@@
     (effects (font (size 1 1) (thickness 0.15)))
   )
-  (gr_text "°" (at 137.25 77.15) (layer "F.SilkS")
+  (gr_text "°" (at 137.05 77.2) (layer "F.SilkS")
     (effects (font (size 1 1) (thickness 0.15)))
   )
@@
   (segment (start 148.3 90.7375) (end 154.563 90.7375) (width 1) (layer "F.Cu") (net 3))
   (segment (start 196.201998 97.536) (end 160.9725 97.536) (width 3) (layer "F.Cu") (net 3))
-  (segment (start 176.55 80.3) (end 175.1 80.3) (width 0.5) (layer "F.Cu") (net 3))
   (segment (start 145.7465 90.7435) (end 148.652 90.7435) (width 1) (layer "F.Cu") (net 3))
   (segment (start 145.7465 94.4585) (end 142.9165 94.4585) (width 1) (layer "F.Cu") (net 3))
@@
   (segment (start 160.9725 97.536) (end 159.4485 96.012) (width 3) (layer "F.Cu") (net 3))
   (segment (start 159.385 81.1) (end 159.385 85.7885) (width 3) (layer "F.Cu") (net 3))
+  (segment (start 175.1 80.3) (end 176.3 80.3) (width 0.5) (layer "F.Cu") (net 3))
   (segment (start 204.978 88.759998) (end 196.201998 97.536) (width 3) (layer "F.Cu") (net 3))
+  (segment (start 176.1 68.3) (end 176.1 69.5) (width 0.5) (layer "F.Cu") (net 3))
   (segment (start 113.665 88.632998) (end 122.695002 97.663) (width 3) (layer "F.Cu") (net 3))
   (segment (start 145.7465 94.4585) (end 145.7465 90.7435) (width 1) (layer "F.Cu") (net 3))
@@
   (segment (start 157.7975 97.663) (end 159.4485 96.012) (width 3) (layer "F.Cu") (net 3))
   (via (at 140.15 76.4) (size 0.6) (drill 0.3) (layers "F.Cu" "B.Cu") (net 3))
-  (via (at 176.55 80.3) (size 0.6) (drill 0.3) (layers "F.Cu" "B.Cu") (net 3))
+  (via (at 176.3 80.3) (size 0.6) (drill 0.3) (layers "F.Cu" "B.Cu") (net 3))
+  (via (at 176.1 69.5) (size 0.6) (drill 0.3) (layers "F.Cu" "B.Cu") (net 3))
   (via (at 137.2 69.85) (size 0.6) (drill 0.3) (layers "F.Cu" "B.Cu") (net 3))
   (segment (start 137.150978 76.4) (end 137.150489 76.399511) (width 0.5) (layer "B.Cu") (net 3))
@@
   (segment (start 137.150489 69.899511) (end 137.150489 76.399511) (width 0.5) (layer "B.Cu") (net 3))
   (segment (start 161.0865 97.65) (end 159.4485 96.012) (width 2) (layer "B.Cu") (net 3))
+  (segment (start 179.65 80.3) (end 179.6955 80.2545) (width 0.5) (layer "B.Cu") (net 3))
   (segment (start 137.15 97.7) (end 157.7605 97.7) (width 2) (layer "B.Cu") (net 3))
+  (segment (start 176.1 76.659) (end 176.1 69.5) (width 0.5) (layer "B.Cu") (net 3))
   (segment (start 189.23 89.789) (end 181.369 97.65) (width 2) (layer "B.Cu") (net 3))
+  (segment (start 176.3 80.3) (end 179.65 80.3) (width 0.5) (layer "B.Cu") (net 3))
   (segment (start 129.286 89.836) (end 137.15 97.7) (width 2) (layer "B.Cu") (net 3))
   (segment (start 137.150489 81.971511) (end 129.286 89.836) (width 0.5) (layer "B.Cu") (net 3))
   (segment (start 137.2 69.85) (end 137.150489 69.899511) (width 0.5) (layer "B.Cu") (net 3))
   (segment (start 189.23 89.789) (end 197.8495 89.789) (width 2) (layer "B.Cu") (net 3))
+  (segment (start 189.23 89.789) (end 179.6955 80.2545) (width 0.5) (layer "B.Cu") (net 3))
   (segment (start 137.150489 76.399511) (end 137.150489 81.971511) (width 0.5) (layer "B.Cu") (net 3))
   (segment (start 140.15 76.4) (end 137.150978 76.4) (width 0.5) (layer "B.Cu") (net 3))
   (segment (start 129.286 89.836) (end 120.904 89.836) (width 2) (layer "B.Cu") (net 3))
+  (segment (start 179.6955 80.2545) (end 176.1 76.659) (width 0.5) (layer "B.Cu") (net 3))
   (segment (start 147.428 84.9655) (end 148.2 85.7375) (width 0.25) (layer "F.Cu") (net 4))
   (segment (start 148.3 87.1625) (end 148.3 85.7375) (width 0.25) (layer "F.Cu") (net 4))
@@
   (segment (start 155.448 70.326) (end 153.474 70.326) (width 0.25) (layer "F.Cu") (net 8))
   (segment (start 145.75 75.825) (end 151.175 70.4) (width 0.25) (layer "F.Cu") (net 8))
+  (segment (start 178.8 64.4625) (end 178.8 65.588) (width 0.5) (layer "F.Cu") (net 9))
   (segment (start 172.0805 78.4195) (end 171.4015 78.4195) (width 0.25) (layer "F.Cu") (net 9))
   (segment (start 172.75 77.75) (end 172.0805 78.4195) (width 0.25) (layer "F.Cu") (net 9))
   (segment (start 197.866 84.7725) (end 197.866 79.766) (width 1) (layer "F.Cu") (net 9))
+  (segment (start 178.8 62.4) (end 178.7 62.3) (width 0.5) (layer "F.Cu") (net 9))
   (segment (start 172.75 76.7) (end 172.75 77.75) (width 0.25) (layer "F.Cu") (net 9))
+  (segment (start 172.75 76.7) (end 178.8 76.7) (width 0.5) (layer "F.Cu") (net 9))
+  (segment (start 178.8 64.4625) (end 178.8 62.4) (width 0.5) (layer "F.Cu") (net 9))
+  (via (at 178.8 76.7) (size 0.6) (drill 0.3) (layers "F.Cu" "B.Cu") (net 9))
+  (via (at 178.8 65.588) (size 0.6) (drill 0.3) (layers "F.Cu" "B.Cu") (net 9))
+  (segment (start 178.8 65.588) (end 178.8 76.7) (width 0.5) (layer "B.Cu") (net 9))
+  (segment (start 189.23 84.789) (end 186.789 84.789) (width 0.5) (layer "B.Cu") (net 9))
   (segment (start 197.866 84.7725) (end 189.2465 84.7725) (width 1) (layer "B.Cu") (net 9))
+  (segment (start 186.789 84.789) (end 178.75 76.75) (width 0.5) (layer "B.Cu") (net 9))
+  (segment (start 178.8 76.7) (end 178.75 76.75) (width 0.5) (layer "B.Cu") (net 9))
   (segment (start 159.385 73.326) (end 159.385 76.2) (width 3) (layer "F.Cu") (net 10))
   (segment (start 166.243 56.895) (end 166.242 56.896) (width 1) (layer "F.Cu") (net 11))
@@
   (segment (start 115.443 51.308) (end 115.465 51.33) (width 3) (layer "F.Cu") (net 18))
   (segment (start 113.665 74.1045) (end 113.665 69.723) (width 3) (layer "B.Cu") (net 18))
+  (segment (start 176.1375 66.3375) (end 176.1 66.3) (width 0.5) (layer "F.Cu") (net 19))
+  (segment (start 176.5375 66.3375) (end 176.5 66.3) (width 0.5) (layer "F.Cu") (net 19))
+  (segment (start 179.75 66.3375) (end 176.1375 66.3375) (width 0.5) (layer "F.Cu") (net 19))
+  (segment (start 176.1 66.3) (end 176.1 60) (width 0.5) (layer "F.Cu") (net 19))
   (segment (start 173.1 80.3) (end 171.421 80.3) (width 0.25) (layer "F.Cu") (net 20))
   (segment (start 170.7515 80.3195) (end 171.4015 80.3195) (width 0.25) (layer "F.Cu") (net 20))
@@
   (via (at 139.2 66.2) (size 0.6) (drill 0.3) (layers "F.Cu" "B.Cu") (net 28))
   (segment (start 139.2 66.2) (end 137.05 66.2) (width 0.25) (layer "B.Cu") (net 28))
+  (segment (start 180.7 64.4625) (end 180.7 62.3) (width 0.5) (layer "F.Cu") (net 29))
+  (segment (start 180.7 62.3) (end 180.7 60) (width 0.5) (layer "F.Cu") (net 29))
   (segment (start 142.24 60.035) (end 142.254 60.021) (width 0.5) (layer "F.Cu") (net 30))
   (segment (start 142.24 62.2) (end 142.24 60.035) (width 0.5) (layer "F.Cu") (net 30))
