File: amp-mosfet-80W/kicad-inrush-relais/v2/inrush-current-limiter-relais.kicad_pcb (KiCad board)
At the start: 2 copper layers, 63.2 x 50.8 mm, 30 parts, among them J1 Conn_01x02, J2 Screw_Terminal_01x02, J3 Conn_01x02, J4 Conn_01x02, J5 Conn_01x02, J6 Screw_Terminal_01x02, K1 Omrom G5Q-1 DC24, Q1 BC559, Q2 2N7000

Commit message: WIP
Parts:
- moved R7 1.52 mm to (128.8, 73.9)
Routing:
- net Net-(K1-Pad3): track 67.9 -> 69.5 mm
- net Net-(K1-Pad4): track 23.3 -> 23.9 mm
Other:
- board text added: "AC IN Neutral"
- board text added: "AC IN Phase"
- board text added: "AC OUT Neutral"
- board text added: "AC OUT Phase"
- board text added: "Inrush Current Limiter Relais V2 2022.02.23"
- board text removed: "AC Neutral"
- board text removed: "AC Phase"
- board text removed: "Inrush Current Limiter Relais V1 2022.02.08"
Changed lines of the file:
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@@
   )
   (footprint "Resistor_THT:R_Axial_Power_L25.0mm_W9.0mm_P30.48mm" (layer "F.Cu")
-    (at 127.254 73.914 -90)
+    (at 128.778 73.914 -90)
     (descr "Resistor, Axial_Power series, Box, pin pitch=30.48mm, 7W, length*width*height=25*9*9mm^3, http://cdn-reichelt.de/documents/datenblatt/B400/5WAXIAL_9WAXIAL_11WAXIAL_17WAXIAL%23YAG.pdf")
     (tags "Resistor Axial_Power series Box pin pitch 30.48mm 7W length 25mm width 9mm height 9mm")
@@
   )
   (gr_rect (start 80.772 55.88) (end 144.018 106.68) (layer "Edge.Cuts") (width 0.1) (fill none))
-  (gr_text "Inrush Current\nLimiter Relais\nV1\n2022.02.08" (at 95.758 103.124) (layer "F.SilkS")
+  (gr_text "Inrush Current\nLimiter Relais\nV2\n2022.02.23" (at 95.758 103.124) (layer "F.SilkS")
     (effects (font (size 1 1) (thickness 0.15)))
   )
@@
     (effects (font (size 1 1) (thickness 0.15)))
   )
-  (gr_text "AC Phase" (at 82.042 70.866 270) (layer "F.SilkS")
-    (effects (font (size 1 1) (thickness 0.15)))
-  )
-  (gr_text "AC Phase" (at 142.748 71.374 90) (layer "F.SilkS")
-    (effects (font (size 1 1) (thickness 0.15)))
-  )
-  (gr_text "AC Neutral" (at 81.788 90.424 270) (layer "F.SilkS")
-    (effects (font (size 1 1) (thickness 0.15)))
-  )
-  (gr_text "AC Neutral" (at 143.002 90.424 90) (layer "F.SilkS")
+  (gr_text "AC IN Phase" (at 82.042 69.85 270) (layer "F.SilkS")
+    (effects (font (size 1 1) (thickness 0.15)))
+  )
+  (gr_text "AC OUT Phase" (at 142.748 69.596 90) (layer "F.SilkS")
+    (effects (font (size 1 1) (thickness 0.15)))
+  )
+  (gr_text "AC IN Neutral" (at 81.788 91.694 270) (layer "F.SilkS")
+    (effects (font (size 1 1) (thickness 0.15)))
+  )
+  (gr_text "AC OUT Neutral" (at 143.002 92.456 90) (layer "F.SilkS")
     (effects (font (size 1 1) (thickness 0.15)))
   )
@@
   (segment (start 93.472 83.566) (end 93.472 87.884) (width 1) (layer "F.Cu") (net 6))
   (via (at 93.472 87.884) (size 1) (drill 0.5) (layers "F.Cu" "B.Cu") (net 6))
-  (segment (start 127.254 104.394) (end 121.426 104.394) (width 1) (layer "B.Cu") (net 6))
   (segment (start 93.472 87.884) (end 98.044 92.456) (width 1) (layer "B.Cu") (net 6))
+  (segment (start 121.426 104.394) (end 120.41 103.378) (width 1) (layer "B.Cu") (net 6))
   (segment (start 98.044 92.456) (end 108.204 92.456) (width 1) (layer "B.Cu") (net 6))
   (segment (start 85.344 77.978) (end 91.694 77.978) (width 1) (layer "B.Cu") (net 6))
@@
   (segment (start 108.204 92.456) (end 112.522 96.774) (width 1) (layer "B.Cu") (net 6))
   (segment (start 113.806 96.774) (end 112.522 96.774) (width 1) (layer "B.Cu") (net 6))
-  (segment (start 121.426 104.394) (end 120.41 103.378) (width 1) (layer "B.Cu") (net 6))
+  (segment (start 128.778 104.394) (end 121.426 104.394) (width 1) (layer "B.Cu") (net 6))
   (segment (start 108.712 100.076) (end 105.41 103.378) (width 1) (layer "B.Cu") (net 7))
   (segment (start 108.712 99.314) (end 108.712 100.076) (width 1) (layer "B.Cu") (net 7))
@@
   (segment (start 138.938 78.232) (end 138.938 73.406) (width 1) (layer "B.Cu") (net 10))
   (segment (start 108.712 84.074) (end 133.096 84.074) (width 1) (layer "B.Cu") (net 10))
-  (segment (start 120.142 82.042) (end 121.92 80.264) (width 1) (layer "F.Cu") (net 11))
-  (segment (start 120.142 94.234) (end 120.142 82.042) (width 1) (layer "F.Cu") (net 11))
-  (via (at 121.92 80.264) (size 1) (drill 0.5) (layers "F.Cu" "B.Cu") (net 11))
-  (segment (start 121.92 80.264) (end 127.254 74.93) (width 1) (layer "B.Cu") (net 11))
-  (segment (start 127.254 74.93) (end 127.254 73.914) (width 1) (layer "B.Cu") (net 11))
+  (segment (start 120.142 82.55) (end 121.666 81.026) (width 1) (layer "F.Cu") (net 11))
+  (segment (start 120.142 94.234) (end 120.142 82.55) (width 1) (layer "F.Cu") (net 11))
+  (via (at 121.666 81.026) (size 1) (drill 0.5) (layers "F.Cu" "B.Cu") (net 11))
+  (segment (start 121.666 81.026) (end 128.778 73.914) (width 1) (layer "B.Cu") (net 11))
   (segment (start 116.332 68.56) (end 118.384 70.612) (width 0.5) (layer "F.Cu") (net 12))
   (segment (start 116.332 59.69) (end 116.332 68.56) (width 0.5) (layer "F.Cu") (net 12))
