File: amp-mosfet-80W/kicad-inrush-relais/v2/inrush-current-limiter-relais.kicad_sch (KiCad schematic)
At the start: 30 parts, among them J1 Conn_01x02, J2 Screw_Terminal_01x02, J3 Conn_01x02, J4 Conn_01x02, J5 Conn_01x02, J6 Screw_Terminal_01x02, K1 Omrom G5Q-1 DC24, Q1 BC559, Q2 2N7000

Commit message: Add some comment
Other:
- note added: "Input Switch: Both AC Lines must be switched!"
Changed lines of the file:
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@@
+    (effects (font (size 1.27 1.27)) (justify left bottom))
+  )
+  (text "Input Switch:\nBoth AC Lines must be switched!" (at 19.685 85.09 0)
     (effects (font (size 1.27 1.27)) (justify left bottom))
   )
