File: amp-mosfet-80W/kicad/V3a/amp-mosfet-80w.kicad_pcb (KiCad board)
At the start: 2 copper layers, 100.3 x 55.2 mm, 66 parts, among them J1 Conn_01x01, J2 Conn_01x01, J3 +50V, J4 -50V, J5 LS+, J6 LS-, J7 GND, Q1 BC856BS, Q11 ECX10P20, Q12 ECX10N20, Q2 BC856BS, Q3 BC856BS, Q4 BC846BDW1, Q5 DZT5401, Q6 DZT5551, Q7 BC856B, Q8 BC846

Commit message: WIP
Parts:
- added JP1: Jump, Connector_PinHeader_2.54mm:PinHeader_1x02_P2.54mm_Vertical, F.Cu at (197.9, 69.7)
- added JP2: Jump, Connector_PinHeader_2.54mm:PinHeader_1x02_P2.54mm_Vertical, F.Cu at (120.9, 69.7)
- C3, C8: value 47p -> 18p
- J3, J4, J5, J6, J7: footprint Connector_Wire:SolderWire-1.5sqmm_1x01_D1.7mm_OD3.9mm -> kicad-snk:TE-726386-2_Pitch5.08mm_Drill1.3mm
- Q1, Q2: value BC856BS -> BCM856BS,115
- Q3: value BC856BS -> BCM846BS,115
- Q4: value BC846BDW1 -> BCM846BS,115
- Q8: value BC846 -> BC846B
- R13, R4, R7, R8: value 1k -> 1k2
- R20, R25: value 33R -> 39R
- R23, R24: value 2.2k -> 1k
- RV1: value 200R -> 500R
- moved J5 5.08 mm to (159.4, 62.0), turned to 90 degrees
- moved J7 3.26 mm to (156.7, 97.8)
- moved J3 2.54 mm to (205.0, 72.3), turned to 90 degrees
- moved J4 2.41 mm to (113.7, 72.1), turned to 90 degrees
- moved C14 1.59 mm to (205.0, 75.7)
- moved C18 1.59 mm to (113.7, 80.7)
- turned J6 to -90 degrees
Connections:
- C18 pad 2: Net-(D6-Pad1) -> Net-(C18-Pad2)
- D5 pad 2: Net-(C14-Pad1) -> Net-(D5-Pad2)
- J4 pad 1: Net-(D6-Pad1) -> Net-(C18-Pad2)
- Q11 pad 3: Net-(D6-Pad1) -> Net-(C18-Pad2)
Routing:
- net Net-(C18-Pad2): track 0.00 -> 35.9 mm
- net Net-(D6-Pad1): track 39.2 -> 3.53 mm
- net GND: track 307.3 -> 300.6 mm
- net Net-(D5-Pad2): track 0.00 -> 3.43 mm
- net Net-(C14-Pad1): track 27.7 -> 24.5 mm

Commit message: Finalize Layout
Other:
- board text added: "Lateral MOSFET Power Amplifier 80W V3a 2022.04.03"
- board text removed: "Lateral MOSFET Power Amplifier 80W V3 2022.01.01"
Changed lines of the file:
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@@
     (property "Sheetname" "")
     (attr smd)
-    (fp_text reference "D2" (at 0 -2) (layer "F.SilkS")
+    (fp_text reference "D2" (at -1.524 -2) (layer "F.SilkS")
       (effects (font (size 1 1) (thickness 0.15)))
     )
@@
     (property "Sheetname" "")
     (attr smd)
-    (fp_text reference "D3" (at 0 2.032) (layer "F.SilkS")
+    (fp_text reference "D3" (at -1.524 1.905) (layer "F.SilkS")
       (effects (font (size 1 1) (thickness 0.15)))
     )
@@
     (property "Sheetname" "")
     (attr through_hole)
-    (fp_text reference "J3" (at 2.8 2.3 90) (layer "F.SilkS")
+    (fp_text reference "J3" (at 6.35 -2.667 90) (layer "F.SilkS")
       (effects (font (size 1 1) (thickness 0.15)))
     )
@@
     (property "Sheetname" "")
     (attr through_hole)
-    (fp_text reference "J5" (at 2.8 2.3 90) (layer "F.SilkS")
+    (fp_text reference "J5" (at 2.54 -2.54 90) (layer "F.SilkS")
       (effects (font (size 1 1) (thickness 0.15)))
     )
@@
     (property "Sheetname" "")
     (attr through_hole)
-    (fp_text reference "J6" (at 2.8 2.3 90) (layer "F.SilkS")
+    (fp_text reference "J6" (at 2.413 2.8575 90) (layer "F.SilkS")
       (effects (font (size 1 1) (thickness 0.15)))
     )
@@
     (property "Sheetname" "")
     (attr through_hole)
-    (fp_text reference "J7" (at 2.8 2.3) (layer "F.SilkS")
+    (fp_text reference "J7" (at 7.747 0) (layer "F.SilkS")
       (effects (font (size 1 1) (thickness 0.15)))
     )
@@
     (property "Sheetname" "")
     (attr through_hole)
-    (fp_text reference "J4" (at 2.8 2.3 90) (layer "F.SilkS")
+    (fp_text reference "J4" (at 6.223 2.794 90) (layer "F.SilkS")
       (effects (font (size 1 1) (thickness 0.15)))
     )
@@
     (property "Sheetname" "")
     (attr through_hole)
-    (fp_text reference "JP2" (at 0 -2.33 90) (layer "F.SilkS")
+    (fp_text reference "JP2" (at 0 -2.794 90) (layer "F.SilkS")
       (effects (font (size 1 1) (thickness 0.15)))
     )
@@
     (property "Sheetname" "")
     (attr through_hole)
-    (fp_text reference "JP1" (at 0 -2.33 90) (layer "F.SilkS")
+    (fp_text reference "JP1" (at 0.127 -2.667 90) (layer "F.SilkS")
       (effects (font (size 1 1) (thickness 0.15)))
     )
@@
   (gr_line (start 209.55 44.577) (end 209.55 99.822) (layer "Edge.Cuts") (width 0.05))
   (gr_line (start 109.22 44.577) (end 209.55 44.577) (layer "Edge.Cuts") (width 0.05))
-  (gr_text "GND" (at 164.0205 96.266) (layer "F.SilkS")
+  (gr_text "GND" (at 159.258 95.25) (layer "F.SilkS")
     (effects (font (size 1 1) (thickness 0.15)))
   )
@@
     (effects (font (size 1 1) (thickness 0.15)))
   )
-  (gr_text "°" (at 164.7 54.3) (layer "F.SilkS")
+  (gr_text "°" (at 164.592 54.61) (layer "F.SilkS")
     (effects (font (size 1 1) (thickness 0.15)))
   )
@@
     (effects (font (size 1 1) (thickness 0.15)))
   )
-  (gr_text "LS+" (at 160.782 60.198) (layer "F.SilkS")
+  (gr_text "LS+" (at 162.687 59.436) (layer "F.SilkS")
     (effects (font (size 1 1) (thickness 0.15)))
   )
@@
     (effects (font (size 1 1) (thickness 0.15)))
   )
-  (gr_text "Lateral MOSFET Power Amplifier 80W\nV3\n2022.01.01" (at 172.8 93.6) (layer "F.SilkS")
+  (gr_text "Lateral MOSFET Power Amplifier 80W\nV3a\n2022.04.03" (at 180.721 96.647) (layer "F.SilkS")
     (effects (font (size 1 1) (thickness 0.15)))
   )
@@
     (effects (font (size 1 1) (thickness 0.15)))
   )
-  (gr_text "LS-" (at 164.0205 86.106) (layer "F.SilkS")
+  (gr_text "LS-" (at 162.941 88.265) (layer "F.SilkS")
     (effects (font (size 1 1) (thickness 0.15)))
   )
