File: ECC88-test-setup/kicad/v1/ecc88-test-setup.kicad_pcb (KiCad board)
At the start: 2 copper layers, 118.7 x 92.1 mm, 27 parts, among them J1 Conn_01x01, J10 Conn_01x01, J11 Conn_01x01, J12 Conn_01x01, J13 Screw_Terminal_01x02, J14 Conn_01x01, J2 Conn_01x01, J3 Conn_01x01, J4 Conn_01x01, J5 Conn_01x01, J6 Conn_01x01, J7 Conn_01x01, J8 Screw_Terminal_01x02, J9 Conn_01x01, U1 ECC88

Commit message: Create gerber
Parts:
- moved C1 57.4 mm to (100.3, 100.9), turned to 0 degrees
- moved C2 53.4 mm to (84.7, 93.6), turned to 0 degrees
- moved J11 52.9 mm to (102.0, 121.4)
- moved H3 47.4 mm to (111.2, 134.6)
- moved J10 46.7 mm to (103.6, 85.9)
- moved J7 46.7 mm to (102.0, 116.4)
- moved C4 45.3 mm to (100.3, 106.9), turned to 0 degrees
- moved H4 42.3 mm to (111.2, 85.7)
- moved J5 40.8 mm to (79.1, 85.9)
- moved C11 35.6 mm to (87.0, 99.7), turned to 0 degrees
- moved J9 32.3 mm to (96.2, 85.9)
- moved H2 28.4 mm to (59.7, 134.6)
- moved J6 24.5 mm to (86.7, 85.9)
- moved J1 23.3 mm to (60.0, 110.2)
- moved J2 20.9 mm to (60.0, 116.1)
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Routing:
- net VDDA: track 0.00 -> 46.1 mm
- net Net-(J3-Pad1): track 0.00 -> 39.1 mm
- net FVCC: track 0.00 -> 21.3 mm
- net Net-(J1-Pad1): track 0.00 -> 17.5 mm, vias 0 -> 1
- net Net-(C3-Pad1): track 0.00 -> 13.4 mm
- net Net-(C1-Pad1): track 0.00 -> 13.1 mm
- net FGND: track 1.85 -> 0.00 mm
Other:
- board size 118.7 x 92.1 mm -> 60.3 x 57.8 mm
- board text added: "+100VDC"
- board text added: "1"
- board text added: "ECC88/E88CC Tester V1 Michael Schenk 2022.10.05"
- board text added: "IA"
- board text removed: "+"
- board text removed: "+200VDC"
- board text removed: "FGND"
- board text removed: "K"
- board text removed: "OUT"
- board text removed: "SRPP+ Tube Pre-Amp ECC88 V3 Michael Schenk 2022.09.17"
