File: ECC88-test-setup/kicad/v1/ecc88-test-setup.kicad_sch (KiCad schematic)
At the start: 27 parts, among them J1 Conn_01x01, J10 Conn_01x01, J11 Conn_01x01, J12 Conn_01x01, J13 Screw_Terminal_01x02, J14 Conn_01x01, J2 Conn_01x01, J3 Conn_01x01, J4 Conn_01x01, J5 Conn_01x01, J6 Conn_01x01, J7 Conn_01x01, J8 Screw_Terminal_01x02, J9 Conn_01x01, U1 ECC88

Commit message: Update ecc88-test-setup.kicad_sch
Other:
- note added: "+100VDC"
- note added: "Anode current (Ia) is tested with the official Telefunken/Philips/Mullard test setup: Va = 100V Vg= +9 680 Ohm cathode resistor Measurement after 10 minutes stabilization. Factory specification NEW E88CC: Ia = 15 ± 0,8mA."
- note removed: "+200VDC"
Changed lines of the file:
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@@
     (effects (font (size 1.27 1.27)) (justify left bottom))
   )
-  (text "+200VDC" (at 303.53 27.305 0)
+  (text "Anode current (Ia) is tested with the official\nTelefunken/Philips/Mullard test setup: \nVa = 100V\nVg= +9\n680 Ohm cathode resistor\nMeasurement after 10 minutes stabilization. \nFactory specification NEW E88CC: Ia = 15 ± 0,8mA.\n\n"
+    (at 160.02 172.72 0)
     (effects (font (size 1.27 1.27)) (justify left bottom))
   )
+  (text "+100VDC" (at 303.53 27.305 0)
+    (effects (font (size 1.27 1.27)) (justify left bottom))
+  )
