File: lv-lownoise-psu/kicad/v3d-4.0-msop.tantal/lv-lownoise-psu.kicad_sch (KiCad schematic)
At the start: 61 parts, among them J1 AC, J10 GND, J11 GND, J12 -5V, J2 GND, J3 AC, J4 +15V, J5 GND, J6 -15V, J7 LED, J8 GND, J9 +5V, Q1 BD139, Q2 BD140, U1 LM7805_TO220, U2 LM7905_TO220, U3 LT3045xMSE, U4 LT3094xMSE

Commit message: WIP
Parts:
- added HS1, HS2: Heatsink, Heatsink:Heatsink_Fischer_SK104-STC-STIC_35x13mm_2xDrill2.5mm, symbol Mechanical:Heatsink
Changed lines of the file:
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@@
   (title_block
     (title "Ultra Low Noise PSU")
-    (date "2021-10-17")
-    (rev "v3d-3.0-MSOP-Tantal")
+    (date "2022-10-12")
+    (rev "v3d-4.0-MSOP-Tantal")
   )
   (junction (at 257.81 123.19) (diameter 0) (color 0 0 0 0)
@@
     (pin "9")
   )
+  (symbol (lib_id "Mechanical:Heatsink") (at 292.1 45.72 0) (unit 1)
+    (in_bom yes) (on_board yes)
+    (property "Reference" "HS1" (id 0) (at 295.7068 42.6466 0)
+      (effects (font (size 1.27 1.27)) (justify left))
+    )
+    (property "Value" "Heatsink" (id 1) (at 295.7068 44.958 0)
+      (effects (font (size 1.27 1.27)) (justify left))
+    )
+    (property "Footprint" "Heatsink:Heatsink_Fischer_SK104-STC-STIC_35x13mm_2xDrill2.5mm" (id 2) (at 292.4048 45.72 0)
+      (effects (font (size 1.27 1.27)) hide)
+    )
+    (property "Datasheet" "~" (id 3) (at 292.4048 45.72 0)
+      (effects (font (size 1.27 1.27)) hide)
+    )
+  )
+  (symbol (lib_id "Mechanical:Heatsink") (at 294.005 203.2 180) (unit 1)
+    (in_bom yes) (on_board yes)
+    (property "Reference" "HS2" (id 0) (at 290.3982 206.2734 0)
+      (effects (font (size 1.27 1.27)) (justify left))
+    )
+    (property "Value" "Heatsink" (id 1) (at 290.3982 203.962 0)
+      (effects (font (size 1.27 1.27)) (justify left))
+    )
+    (property "Footprint" "Heatsink:Heatsink_Fischer_SK104-STC-STIC_35x13mm_2xDrill2.5mm" (id 2) (at 293.7002 203.2 0)
+      (effects (font (size 1.27 1.27)) hide)
+    )
+    (property "Datasheet" "~" (id 3) (at 293.7002 203.2 0)
+      (effects (font (size 1.27 1.27)) hide)
+    )
+  )
   (sheet_instances
     (path "/" (page "1"))
@@
       (reference "H4") (unit 1) (value "MountingHole") (footprint "MountingHole:MountingHole_3.2mm_M3")
     )
+    (path "/42c84127-4873-4d06-8a36-4c83792c8f84"
+      (reference "HS1") (unit 1) (value "Heatsink") (footprint "Heatsink:Heatsink_Fischer_SK104-STC-STIC_35x13mm_2xDrill2.5mm")
+    )
+    (path "/81a69b59-de7b-465d-af2b-2d638af31dd2"
+      (reference "HS2") (unit 1) (value "Heatsink") (footprint "Heatsink:Heatsink_Fischer_SK104-STC-STIC_35x13mm_2xDrill2.5mm")
+    )
     (path "/00000000-0000-0000-0000-00005f95f176"

Commit message: WIP
Parts:
- added C23: 10nF, Capacitor_THT:C_Rect_L7.2mm_W2.5mm_P5.00mm_FKS2_FKP2_MKS2_MKP2, symbol Device:C
- added J?: EARTH, Connector_Pin:Pin_D1.3mm_L11.0mm, symbol Connector_Generic:Conn_01x01
- added R1: 100R/0.6W, Resistor_THT:R_Axial_DIN0207_L6.3mm_D2.5mm_P10.16mm_Horizontal, symbol Device:R
Connections:
- net GND: now also C23.2, R1.1
- new net: C23.1, J?.1 (Pin_1), R1.2
Changed lines of the file:
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@@
   (junction (at 186.69 166.37) (diameter 0) (color 0 0 0 0)
+  )
+  (junction (at 38.1 191.135) (diameter 0) (color 0 0 0 0)
   )
   (junction (at 278.13 129.54) (diameter 0) (color 0 0 0 0)
@@
     (stroke (width 0) (type default) (color 0 0 0 0))
   )
+  (wire (pts (xy 54.61 205.105) (xy 54.61 213.36))
+    (stroke (width 0) (type default) (color 0 0 0 0))
+  )
   (wire (pts (xy 318.77 66.04) (xy 306.07 66.04))
     (stroke (width 0) (type default) (color 0 0 0 0))
@@
     (stroke (width 0) (type default) (color 0 0 0 0))
   )
+  (wire (pts (xy 38.1 197.485) (xy 38.1 191.135))
+    (stroke (width 0) (type default) (color 0 0 0 0))
+  )
   (wire (pts (xy 278.13 66.04) (xy 278.13 64.77))
     (stroke (width 0) (type default) (color 0 0 0 0))
@@
     (stroke (width 0) (type default) (color 0 0 0 0))
   )
+  (wire (pts (xy 38.1 205.105) (xy 38.1 213.36))
+    (stroke (width 0) (type default) (color 0 0 0 0))
+  )
   (wire (pts (xy 306.07 55.88) (xy 306.07 43.18))
     (stroke (width 0) (type default) (color 0 0 0 0))
@@
     (stroke (width 0) (type default) (color 0 0 0 0))
   )
+  (wire (pts (xy 38.1 191.135) (xy 27.94 191.135))
+    (stroke (width 0) (type default) (color 0 0 0 0))
+  )
   (wire (pts (xy 31.75 106.68) (xy 27.94 106.68))
     (stroke (width 0) (type default) (color 0 0 0 0))
@@
     (stroke (width 0) (type default) (color 0 0 0 0))
   )
+  (wire (pts (xy 54.61 197.485) (xy 54.61 191.135))
+    (stroke (width 0) (type default) (color 0 0 0 0))
+  )
   (wire (pts (xy 208.28 102.87) (xy 208.28 123.19))
     (stroke (width 0) (type default) (color 0 0 0 0))
@@
   )
   (wire (pts (xy 278.13 129.54) (xy 278.13 123.19))
+    (stroke (width 0) (type default) (color 0 0 0 0))
+  )
+  (wire (pts (xy 54.61 191.135) (xy 38.1 191.135))
     (stroke (width 0) (type default) (color 0 0 0 0))
   )
@@
     (pin "9")
   )
+  (symbol (lib_id "Connector_Generic:Conn_01x01") (at 22.86 191.135 180) (unit 1)
+    (in_bom yes) (on_board yes)
+    (property "Reference" "J?" (id 0) (at 24.9428 185.42 0))
+    (property "Value" "EARTH" (id 1) (at 24.9428 187.7314 0))
+    (property "Footprint" "Connector_Pin:Pin_D1.3mm_L11.0mm" (id 2) (at 22.86 191.135 0)
+      (effects (font (size 1.27 1.27)) hide)
+    )
+    (property "Datasheet" "~" (id 3) (at 22.86 191.135 0)
+      (effects (font (size 1.27 1.27)) hide)
+    )
+    (pin "1")
+  )
   (symbol (lib_id "Mechanical:Heatsink") (at 292.1 45.72 0) (unit 1)
     (in_bom yes) (on_board yes)
@@
     )
   )
+  (symbol (lib_id "Device:R") (at 38.1 201.295 180) (unit 1)
+    (in_bom yes) (on_board yes)
+    (property "Reference" "R1" (id 0) (at 39.878 200.1266 0)
+      (effects (font (size 1.27 1.27)) (justify right))
+    )
+    (property "Value" "100R/0.6W" (id 1) (at 39.878 202.438 0)
+      (effects (font (size 1.27 1.27)) (justify right))
+    )
+    (property "Footprint" "Resistor_THT:R_Axial_DIN0207_L6.3mm_D2.5mm_P10.16mm_Horizontal" (id 2) (at 39.878 201.295 90)
+      (effects (font (size 1.27 1.27)) hide)
+    )
+    (property "Datasheet" "~" (id 3) (at 38.1 201.295 0)
+      (effects (font (size 1.27 1.27)) hide)
+    )
+    (pin "1")
+    (pin "2")
+  )
+  (symbol (lib_id "power:GND") (at 38.1 213.36 0) (unit 1)
+    (in_bom yes) (on_board yes)
+    (property "Reference" "#PWR?" (id 0) (at 38.1 219.71 0)
+      (effects (font (size 1.27 1.27)) hide)
+    )
+    (property "Value" "GND" (id 1) (at 38.227 217.7542 0))
+    (property "Footprint" "" (id 2) (at 38.1 213.36 0)
+      (effects (font (size 1.27 1.27)) hide)
+    )
+    (property "Datasheet" "" (id 3) (at 38.1 213.36 0)
+      (effects (font (size 1.27 1.27)) hide)
+    )
+    (pin "1")
+  )
   (symbol (lib_id "Mechanical:Heatsink") (at 294.005 203.2 180) (unit 1)
     (in_bom yes) (on_board yes)
@@
       (effects (font (size 1.27 1.27)) hide)
     )
+  )
+  (symbol (lib_id "Device:C") (at 54.61 201.295 0) (unit 1)
+    (in_bom yes) (on_board yes)
+    (property "Reference" "C23" (id 0) (at 57.531 200.1266 0)
+      (effects (font (size 1.27 1.27)) (justify left))
+    )
+    (property "Value" "10nF" (id 1) (at 57.531 202.438 0)
+      (effects (font (size 1.27 1.27)) (justify left))
+    )
+    (property "Footprint" "Capacitor_THT:C_Rect_L7.2mm_W2.5mm_P5.00mm_FKS2_FKP2_MKS2_MKP2" (id 2) (at 55.5752 205.105 0)
+      (effects (font (size 1.27 1.27)) hide)
+    )
+    (property "Datasheet" "~" (id 3) (at 54.61 201.295 0)
+      (effects (font (size 1.27 1.27)) hide)
+    )
+    (pin "1")
+    (pin "2")
+  )
+  (symbol (lib_id "power:GND") (at 54.61 213.36 0) (unit 1)
+    (in_bom yes) (on_board yes)
+    (property "Reference" "#PWR?" (id 0) (at 54.61 219.71 0)
+      (effects (font (size 1.27 1.27)) hide)
+    )
+    (property "Value" "GND" (id 1) (at 54.737 217.7542 0))
+    (property "Footprint" "" (id 2) (at 54.61 213.36 0)
+      (effects (font (size 1.27 1.27)) hide)
+    )
+    (property "Datasheet" "" (id 3) (at 54.61 213.36 0)
+      (effects (font (size 1.27 1.27)) hide)
+    )
+    (pin "1")
   )
   (sheet_instances
@@
       (reference "#PWR05") (unit 1) (value "GND") (footprint "")
     )
+    (path "/6ef8b8a9-3b6c-4035-b63c-a849275e4543"
+      (reference "#PWR?") (unit 1) (value "GND") (footprint "")
+    )
+    (path "/ea06e694-403f-4d63-bd1a-eac49c45ba0c"
+      (reference "#PWR?") (unit 1) (value "GND") (footprint "")
+    )
     (path "/00000000-0000-0000-0000-00005f961063"
       (reference "C1") (unit 1) (value "2200uF") (footprint "Capacitor_THT:CP_Radial_D16.0mm_P7.50mm")
@@
       (reference "C22") (unit 1) (value "4.7uF/50V") (footprint "Capacitor_SMD:C_1206_3216Metric_Pad1.33x1.80mm_HandSolder")
     )
+    (path "/aa24abdc-9e35-4e9b-a00f-de3614e96dab"
+      (reference "C23") (unit 1) (value "10nF") (footprint "Capacitor_THT:C_Rect_L7.2mm_W2.5mm_P5.00mm_FKS2_FKP2_MKS2_MKP2")
+    )
     (path "/00000000-0000-0000-0000-00005fedaddc"
       (reference "D1") (unit 1) (value "BYG20D") (footprint "Diode_SMD:D_SMA_Handsoldering")
@@
       (reference "J12") (unit 1) (value "-5V") (footprint "Connector_Pin:Pin_D1.0mm_L10.0mm")
     )
+    (path "/11936b0a-663c-49b1-825c-3278bd212564"
+      (reference "J?") (unit 1) (value "EARTH") (footprint "Connector_Pin:Pin_D1.3mm_L11.0mm")
+    )
     (path "/00000000-0000-0000-0000-0000613b0ed5"
       (reference "Q1") (unit 1) (value "BD139") (footprint "Package_TO_SOT_THT:TO-126-3_Vertical")
@@
       (reference "Q2") (unit 1) (value "BD140") (footprint "Package_TO_SOT_THT:TO-126-3_Vertical")
     )
+    (path "/638e12ac-287d-4bc3-a891-66952336b2be"
+      (reference "R1") (unit 1) (value "100R/0.6W") (footprint "Resistor_THT:R_Axial_DIN0207_L6.3mm_D2.5mm_P10.16mm_Horizontal")
+    )
     (path "/00000000-0000-0000-0000-00005fabe010"

Commit message: WIP
Parts:
- gave numbers to parts that had none: 1
Other:
- note added: "13,4°/W"
Changed lines of the file:
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@@
     (stroke (width 0) (type default) (color 0 0 0 0))
+  )
+  (text "13,4°/W" (at 282.575 209.55 0)
+    (effects (font (size 1.27 1.27)) (justify left bottom))
   )
   (text "Snubber" (at 27.94 101.6 0)
@@
   )
   (text "Cs=100nF/50\nRs=25.8R/0.125W" (at 27.94 154.94 0)
+    (effects (font (size 1.27 1.27)) (justify left bottom))
+  )
+  (text "13,4°/W" (at 295.91 48.26 0)
     (effects (font (size 1.27 1.27)) (justify left bottom))
   )
@@
   (symbol (lib_id "Connector_Generic:Conn_01x01") (at 22.86 191.135 180) (unit 1)
     (in_bom yes) (on_board yes)
-    (property "Reference" "J?" (id 0) (at 24.9428 185.42 0))
+    (property "Reference" "J13" (id 0) (at 24.9428 185.42 0))
     (property "Value" "EARTH" (id 1) (at 24.9428 187.7314 0))
     (property "Footprint" "Connector_Pin:Pin_D1.3mm_L11.0mm" (id 2) (at 22.86 191.135 0)
@@
   (symbol (lib_id "power:GND") (at 38.1 213.36 0) (unit 1)
     (in_bom yes) (on_board yes)
-    (property "Reference" "#PWR?" (id 0) (at 38.1 219.71 0)
+    (property "Reference" "#PWR0101" (id 0) (at 38.1 219.71 0)
       (effects (font (size 1.27 1.27)) hide)
     )
@@
   (symbol (lib_id "power:GND") (at 54.61 213.36 0) (unit 1)
     (in_bom yes) (on_board yes)
-    (property "Reference" "#PWR?" (id 0) (at 54.61 219.71 0)
+    (property "Reference" "#PWR0102" (id 0) (at 54.61 219.71 0)
       (effects (font (size 1.27 1.27)) hide)
     )
@@
     )
     (path "/6ef8b8a9-3b6c-4035-b63c-a849275e4543"
-      (reference "#PWR?") (unit 1) (value "GND") (footprint "")
+      (reference "#PWR0101") (unit 1) (value "GND") (footprint "")
     )
     (path "/ea06e694-403f-4d63-bd1a-eac49c45ba0c"
-      (reference "#PWR?") (unit 1) (value "GND") (footprint "")
+      (reference "#PWR0102") (unit 1) (value "GND") (footprint "")
     )
     (path "/00000000-0000-0000-0000-00005f961063"
@@
     )
     (path "/11936b0a-663c-49b1-825c-3278bd212564"
-      (reference "J?") (unit 1) (value "EARTH") (footprint "Connector_Pin:Pin_D1.3mm_L11.0mm")
+      (reference "J13") (unit 1) (value "EARTH") (footprint "Connector_Pin:Pin_D1.3mm_L11.0mm")
     )
     (path "/00000000-0000-0000-0000-0000613b0ed5"
