File: pre-amp-discret-elektor/kicad/v2e-servo/pre-amp-discret.kicad_sch (KiCad schematic)
At the start: 77 parts, among them J1 Conn_01x01, J2 Conn_01x01, J3 Conn_01x01, J4 Conn_01x01, J5 Conn_01x01, J6 Conn_01x01, J7 Conn_01x01, J8 Conn_01x01, J9 Conn_01x01, Q1 BCM857DS,115, Q11 BCM847DS,115, Q13 BCM847DS,115, Q2 BC850C, Q3 BCM857DS,115, Q4 BC550C, Q5 BC560C, Q6 BC337-40, Q7 BC860C, Q8 BC327-40, U1 OPA188xxDBV

Commit message: create gerber for v2e
Parts:
- removed R10, R12: 10k, Resistor_SMD:R_0805_2012Metric_Pad1.20x1.40mm_HandSolder, symbol Device:R
- C7, C8: value 150p -> 22pF
Connections:
- net GND: no longer C7.1, C8.2
- net at Q1.6 (C1), Q2.1 (B), R3.1: now also C8.2
- net at Q13.6 (C1), Q7.1 (B), R20.2: now also C7.2
- net at C9.2, Q4.1 (C), Q6.2 (B)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: now also C7.1
- net at C9.1, Q2.3 (C), Q5.1 (C)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: now also C8.1
Other:
- note added: "C7: not equipped"
