File: pre-amp-discret-symetric/kicad/v4a-servo/pre-amp-discret.kicad_sch (KiCad schematic)
At the start: 78 parts, among them J1 Conn_01x01, J2 Conn_01x01, J3 Conn_01x01, J4 Conn_01x01, J5 Conn_01x01, J6 Conn_01x01, J7 Conn_01x01, J8 Conn_01x01, J9 Conn_01x01, Q10 BC860C, Q11 BCM847DS,115, Q14 BCM857DS,115, Q18 BC860C, Q19 BC860C, Q2 BCM847DS,115, Q20 BC850C, Q3 BCM857DS,115, Q4 THAT340, Q6 BC850C, Q7 BC860C, Q8 BC850C, Q9 BCM857DS,115, U1 OPA188xxDBV

Commit message: wip
Parts:
- removed Q10: BC860C, Package_TO_SOT_SMD:SOT-23, symbol Transistor_BJT:BC860
- removed Q9: BCM857DS,115, Package_SO:SC-74-6_1.5x2.9mm_P0.95mm, symbol kicad-snk:BCM857DS,115
- added Q1: BC860C, Package_TO_SOT_SMD:SOT-23, symbol Transistor_BJT:BC860
- added Q5, Q9: DZT5401, Package_TO_SOT_SMD:SOT-223-3_TabPin2, symbol kicad-snk:DZT5401
- R12: value 100R -> 40.2R
- R14, R16: value 100k -> 160k
- R18: value 10k -> 47k
- R19: value 470R -> 0R
- R8: value 10k -> 4.7k
Connections:
- net +15V: now also Q1.2 (E)
- net -15V: now also Q9.2 (C)
- net at C12.1, R13.2, R9.1: now also Q5.2 (C), Q9.3 (E)
- net at C17.1, C7.1, Q7.3 (C)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: now also Q9.1 (B)
- net at R12.2: now also Q1.1 (B), Q5.3 (E)
- net at R28.1: now also Q1.3 (C), Q5.1 (B)
Other:
- note added: "C1: not equipped"
- note added: "Notes R19/C11: Not used as volume resistore influence the fg"
- note added: "R8//R18 = 4.27k"
- note added: "Servo Inject Ratio: 1:10 (4.7k : 47k) Example: Offset = 30mV, DCSERVO_OUT = 300mV"
- note added: "V = 1 + (R9 / (R8//R18) = 3.34"
- note added: "fg = 1Hz (160k, 1uF)"
