File: amp-mosfet-80W/kicad/v5f/amp-mosfet-80w.kicad_pcb (KiCad board)
At the start: 2 copper layers, 100.3 x 55.2 mm, 67 parts, among them J1 Conn_01x01, J2 Conn_01x01, J3 +50V, J4 -50V, J5 LS+, J6 LS-, J7 GND, Q1 BCM856BS,115, Q11 ECX10P20, Q12 ECX10N20, Q2 BCM856BS,115, Q3 BCM846BS,115, Q4 BCM846BS,115, Q5 BC856B, Q6 DZT5551, Q7 DZT5401, Q8 BC846B

Commit message: v5f ready for production
Parts:
- added C2: 150pF/100V/COG, Capacitor_SMD:C_0805_2012Metric_Pad1.18x1.45mm_HandSolder, F.Cu at (140.0, 63.2)
- added R29: 1k/0.3W, Resistor_SMD:R_0805_2012Metric_Pad1.20x1.40mm_HandSolder, F.Cu at (154.4, 63.2)
- C8: value 100pF/50V/Film -> 47pF/100V/COG
- R8: value 22k/0.25W -> 22k/0.3W
- moved C8 2.11 mm to (137.8, 63.2)
Connections:
- C8 pad 1: Net-(D4-A) -> Net-(C2-Pad2)
Routing:
- net Net-(C2-Pad2): track 0.00 -> 17.5 mm, vias 0 -> 2
- net Net-(D2-A): track 108.9 -> 114.5 mm
Other:
- board text added: "Lateral MOSFET Power Amplifier 80W V5f 2023.09.03"
- board text removed: "Lateral MOSFET Power Amplifier 80W V5e 2023.08.20"
