File: rpi-hat-uart/kicad/V1/rpi-hat-spdif/rpi-hat-uart.kicad_sch (KiCad schematic)
At the start: 37 parts, among them IC1 WM8804GEDS_V, J1 GPIO, J2 TTL-232R-3V3, U1 TSOP32538, U2 PLT237/T10WH, U3 KC3225Z24.5760C1KX00, U4 KC3225Z22.5792C15XXK, U5 TPS7A2033PDBVR, U6 TPS7A2033PDBVR, U7 APX809S-31SA-7

Commit message: Ready to order
Parts:
- removed C1, C2, C4: 100nF/50V, Capacitor_SMD:C_0603_1608Metric_Pad1.08x0.95mm_HandSolder, symbol Device:C
- removed C11, C12, C8: 1uF/25V, Capacitor_SMD:C_0603_1608Metric_Pad1.08x0.95mm_HandSolder, symbol Device:C
- removed C13, C14: 10uF/25V, Capacitor_SMD:C_1206_3216Metric_Pad1.33x1.80mm_HandSolder, symbol Device:C
- removed C3, C5, C6: 100nF/50V, Capacitor_SMD:C_0603_1608Metric, symbol Device:C
- removed C7, C9: 47uF/6.3V, Capacitor_SMD:C_1206_3216Metric_Pad1.33x1.80mm_HandSolder, symbol Device:C_Polarized
- removed FB1: 1k@100MHz, Resistor_SMD:R_0603_1608Metric_Pad0.98x0.95mm_HandSolder, symbol dac-rescue:Ferrite_Bead_Small-Device
- removed IC1: WM8804GEDS_V, Package_SO:SSOP-20_5.3x7.2mm_P0.65mm, symbol kicad-snk:WM8804GEDS_V
- removed J1: GPIO, Connector_PinSocket_2.54mm:PinSocket_2x20_P2.54mm_Vertical, symbol Connector_Generic:Conn_02x20_Odd_Even
- removed R1, R10, R2, R9: 0R, Resistor_SMD:R_0603_1608Metric_Pad0.98x0.95mm_HandSolder, symbol Device:R
- removed R11, R5, R6, R8: 10k, Resistor_SMD:R_0603_1608Metric_Pad0.98x0.95mm_HandSolder, symbol Device:R
- removed R12, R13, R14, R3, R7: 33R, Resistor_SMD:R_0603_1608Metric_Pad0.98x0.95mm_HandSolder, symbol Device:R
- removed U1: TSOP32538, OptoDevice:Vishay_MOLD-3Pin, symbol Interface_Optical:TSOP325xx
- removed U2: PLT237/T10WH, kicad-snk:PLR135-T10_PLT133-T10W, symbol kicad-snk:PLT237/T10WH
- removed U3: KC3225Z24.5760C1KX00, Crystal:Crystal_SMD_3225-4Pin_3.2x2.5mm_HandSoldering, symbol Oscillator:KC2520Z
- removed U4: KC3225Z22.5792C15XXK, Crystal:Crystal_SMD_3225-4Pin_3.2x2.5mm_HandSoldering, symbol Oscillator:KC2520Z
- removed U5, U6: TPS7A2033PDBVR, Package_TO_SOT_SMD:SOT-23-5, symbol Regulator_Linear:TPS7A0533PDBV
- removed U7: APX809S-31SA-7, Package_TO_SOT_SMD:SOT-23, symbol Power_Supervisor:LM809
- added J1: GPIO, Connector_PinHeader_2.54mm:PinHeader_2x05_P2.54mm_Vertical, symbol Connector_Generic:Conn_02x05_Odd_Even
Connections:
- net +3.3VP: now also J1.1 (Pin_1)
- net +5V: now also J1.2 (Pin_2), J1.4 (Pin_4)
- net GND: now also J1.6 (Pin_6), J1.9 (Pin_9)
- net GPIO14/TXD0: now also J1.8 (Pin_8)
- net GPIO15/RXD0: now also J1.10 (Pin_10)
- net GPIO2/SDA1: now also J1.3 (Pin_3)
- net GPIO3/SCL1: now also J1.5 (Pin_5)
- net GPIO4/GPCLK0: now also J1.7 (Pin_7)
- no-connect marks 8 -> 3
Other:
- note added: "https://www.raspberrypi.com/documentation/computers/raspberry-pi.html"
- note removed: "*)Default"
- note removed: "22.5792MHZ 44.1kHz"
- note removed: "24.5760MHZ 48kHz"
- note removed: "WM8804 (3.3V) Voh >= 2.97V Vol <= 0.33V PLT237 (+5V) Vih >= 2V Vil <= 0.8V"
- note removed: "https://www.raspberrypi.com/documentation/computers/raspberry-pi.html Device Tree dtoverlay=gpio-ir,gpio_pin=22 dtoverlay=hifiberry-digi-pro"
- title: RPI HAT S/PDIF and IR -> RPI HAT UART
- moved on the sheet: J2
