File: tube-testers/ecc88/kicad/v3/ecc88-test-setup.kicad_pcb (KiCad board)
At the start: 2 copper layers, 60.3 x 57.8 mm, 27 parts, among them J1 Conn_01x01, J10 Conn_01x01, J11 Conn_01x01, J12 Conn_01x01, J13 Screw_Terminal_01x02, J14 Conn_01x01, J2 Conn_01x01, J3 Conn_01x01, J4 Conn_01x01, J5 Conn_01x01, J6 Conn_01x01, J7 Conn_01x01, J8 Screw_Terminal_01x02, J9 Conn_01x01, U1 ECC88

Commit message: WIP
Parts:
- added JP1: Jumper_2_Open, Connector_PinHeader_2.54mm:PinHeader_1x02_P2.54mm_Vertical, F.Cu at (121.5, 90.4)
- added JP2: Jumper_2_Open, Connector_PinHeader_2.54mm:PinHeader_1x02_P2.54mm_Vertical, F.Cu at (126.1, 90.4)
- added JP3: Jumper_2_Open, Connector_PinHeader_2.54mm:PinHeader_1x02_P2.54mm_Vertical, F.Cu at (130.8, 90.4)
- added JP4: Jumper_3_Open, Connector_PinHeader_2.54mm:PinHeader_1x03_P2.54mm_Vertical, F.Cu at (130.3, 114.5)
- added JP5: Jumper_3_Open, Connector_PinHeader_2.54mm:PinHeader_1x03_P2.54mm_Vertical, F.Cu at (135.0, 114.5)
- added R3: 1Meg/0.6W, Resistor_THT:R_Axial_DIN0207_L6.3mm_D2.5mm_P10.16mm_Horizontal, F.Cu at (129.6, 106.1)
- added R4: 1Meg/0.6W, Resistor_THT:R_Axial_DIN0207_L6.3mm_D2.5mm_P10.16mm_Horizontal, F.Cu at (129.6, 110.2)
Connections:
- C1 pad 1: Net-(C1-Pad1) -> Net-(JP4-B)
- C3 pad 1: Net-(C3-Pad1) -> Net-(JP5-B)
- C4 pad 1: Net-(C1-Pad1) -> Net-(JP4-B)
- C5 pad 1: Net-(C3-Pad1) -> Net-(JP5-B)
- R1 pad 2: Net-(C1-Pad1) -> Net-(JP4-B)
- R2 pad 2: Net-(C3-Pad1) -> Net-(JP5-B)
- U1 pad 3: Net-(C1-Pad1) -> Net-(JP4-C)
- U1 pad 8: Net-(C3-Pad1) -> Net-(JP5-C)
Routing:
- net (no net): track 0.00 -> 26.5 mm
- net Net-(C3-Pad1): track 13.4 -> 0.00 mm
- net Net-(C1-Pad1): track 13.1 -> 0.00 mm
Other:
- board text added: "ECC88/E88CC Tester V3 Michael Schenk 2024.08.02"
- board text removed: "ECC88/E88CC Tester V2 Michael Schenk 2022.10.12"

Commit message: Finalize V3
Parts:
- added C6: 100nF, Capacitor_THT:C_Rect_L16.5mm_W5.0mm_P15.00mm_MKT, F.Cu at (102.0, 114.9)
- H1, H2, H3, H4: footprint MountingHole:MountingHole_3.2mm_M3 -> MountingHole:MountingHole_3.2mm_M3_Pad_Via
- moved JP3 66.6 mm to (66.5, 108.1), turned to 90 degrees
- moved JP1 66.2 mm to (59.9, 114.8)
- moved JP5 65.1 mm to (69.8, 113.9)
- moved JP2 56.1 mm to (89.5, 132.9), turned to 180 degrees
- moved R4 53.2 mm to (76.7, 104.6), turned to 180 degrees
- moved R3 37.9 mm to (102.8, 132.9), turned to 180 degrees
- moved C3 28.9 mm to (71.1, 136.1)
- moved JP4 28.0 mm to (102.9, 109.2), turned to 180 degrees
- moved C5 17.1 mm to (71.1, 130.2), turned to 0 degrees
- moved C2 11.6 mm to (74.6, 87.9), turned to 180 degrees
- moved R2 10.7 mm to (61.0, 126.9)
- moved C1 9.80 mm to (102.9, 91.4)
- moved R1 9.80 mm to (113.0, 100.8)
- moved C4 9.80 mm to (102.9, 97.5)
- moved H1 7.65 mm to (54.0, 80.6)
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Routing:
- net VDDA: track 58.3 -> 86.7 mm
- net (no net): track 26.5 -> 0.00 mm
- net Net-(J3-Pin_1): track 39.1 -> 64.5 mm
- net Net-(JP5-B): track 0.00 -> 17.7 mm
- net Net-(J1-Pin_1): track 17.5 -> 30.5 mm, vias 1 -> 0
- net Net-(JP4-B): track 0.00 -> 12.7 mm
- net Net-(JP4-C): track 0.00 -> 7.77 mm
- net Net-(JP5-C): track 0.00 -> 7.73 mm
- net FVCC: track 21.3 -> 27.1 mm
- net Net-(J13-Pin_2): track 11.5 -> 15.2 mm
- net Net-(JP3-A): track 0.00 -> 3.48 mm
- net Net-(JP2-A): track 0.00 -> 3.10 mm
- net Net-(J11-Pin_1): track 14.9 -> 17.5 mm
Other:
- board size 60.3 x 57.8 mm -> 70.6 x 67.6 mm
- board text added: "ECC88/E88CC Tester V3 Michael Schenk 2024.08.04"
- board text added: "Ia System 1"
- board text added: "Ia System 2"
- board text added: "System 1:K=8,G=7,A=6 System 2:K=3,G=2,A=1"
- board text added: "Ua"
- board text added: "Ug"
- board text added: "Ug System 1"
- board text added: "Ug System 2"
- board text added: "Uh"
- board text added: "Va=100V, Vg= +9 with 680 Ohm cathode resistor After 10 minutes stabilization Ia = 15 ± 0.8mA"
- board text removed: "ECC88/E88CC Tester V3 Michael Schenk 2024.08.02"
- board text removed: "IA"
- board text removed: "IN"
