File: tube-testers/6sn7/kicad/v1/6sn7-test-setup.kicad_pcb (KiCad board)
At the start: 2 copper layers, 70.6 x 67.6 mm, 27 parts, among them J1 Conn_01x01, J10 Conn_01x01, J11 Conn_01x01, J12 Conn_01x01, J13 Screw_Terminal_01x02, J14 Conn_01x01, J2 Conn_01x01, J3 Conn_01x01, J4 Conn_01x01, J5 Conn_01x01, J6 Conn_01x01, J7 Conn_01x01, J8 Screw_Terminal_01x02, J9 Conn_01x01, U1 6SN7

Commit message: Ordered
Other:
- board text added: "2"
- board text added: "3"
- board text added: "4"
- board text added: "5"
- board text added: "6"
- board text added: "7"
- board text added: "8"
Changed lines of the file:
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@@
 		(at 87.0712 113.3348 180)
 		(property "Reference" "U1"
-			(at 0 -18.795 360)
+			(at 0 -18.795 0)
 			(layer "F.SilkS")
 			(effects
@@
 		)
 		(property "Value" "6SN7"
-			(at 0 18.795 360)
+			(at 0 18.795 0)
 			(layer "F.Fab")
 			(effects
@@
 		)
 		(property "Footprint" "kicad-snk:TubeOctal"
-			(at 0 0 360)
+			(at 0 0 0)
 			(layer "F.Fab")
 			(hide yes)
@@
 		)
 		(property "Datasheet" "https://frank.pocnet.net/sheets/049/6/6SN7GTA.pdf"
-			(at 0 0 360)
+			(at 0 0 0)
 			(layer "F.Fab")
 			(hide yes)
@@
 		)
 		(property "Description" "double triode"
-			(at 0 0 360)
+			(at 0 0 0)
 			(layer "F.Fab")
 			(hide yes)
@@
 		(tags "Resistor Axial_DIN0207 series Axial Horizontal pin pitch 10.16mm 0.25W = 1/4W length 6.3mm diameter 2.5mm")
 		(property "Reference" "R3"
-			(at 5.1816 2.2098 360)
+			(at 5.1816 2.2098 0)
 			(layer "F.SilkS")
 			(effects
@@
 		)
 		(property "Value" "1Meg/0.6W"
-			(at 5.08 2.37 360)
+			(at 5.08 2.37 0)
 			(layer "F.Fab")
 			(effects
@@
 		)
 		(fp_text user "${REFERENCE}"
-			(at 5.08 0 360)
+			(at 5.08 0 0)
 			(layer "F.Fab")
 			(effects
@@
 		(tags "Resistor Axial_DIN0207 series Axial Horizontal pin pitch 10.16mm 0.25W = 1/4W length 6.3mm diameter 2.5mm")
 		(property "Reference" "R4"
-			(at 4.191 -2.37 360)
+			(at 4.191 -2.37 0)
 			(layer "F.SilkS")
 			(effects
@@
 		)
 		(property "Value" "1Meg/0.6W"
-			(at 5.08 2.37 360)
+			(at 5.08 2.37 0)
 			(layer "F.Fab")
 			(effects
@@
 		)
 		(fp_text user "${REFERENCE}"
-			(at 5.08 0 360)
+			(at 5.08 0 0)
 			(layer "F.Fab")
 			(effects
@@
 		(tags "Through hole pin header THT 1x02 2.54mm single row")
 		(property "Reference" "JP3"
-			(at 0 5.842 360)
+			(at 0 5.842 0)
 			(layer "F.SilkS")
 			(effects
@@
 		)
 		(fp_text user "${REFERENCE}"
-			(at 0 1.27 360)
+			(at 0 1.27 0)
 			(layer "F.Fab")
 			(effects
@@
 		)
 	)
+	(gr_text "4"
+		(at 79.9084 131.5212 0)
+		(layer "F.SilkS")
+		(effects
+			(font
+				(size 1 1)
+				(thickness 0.15)
+			)
+		)
+	)
+	(gr_text "3"
+		(at 68.9356 120.4976 0)
+		(layer "F.SilkS")
+		(effects
+			(font
+				(size 1 1)
+				(thickness 0.15)
+			)
+		)
+	)
 	(gr_text "Datasheet: Ua=+250V,Ug=-8V,Ia>=9mA\nFunke: Ua=+150V,Ug=-2V,Ia>=11mA\n"
 		(at 100.5332 139.8016 180)
@@
 		)
 	)
+	(gr_text "2"
+		(at 69.342 106.426 0)
+		(layer "F.SilkS")
+		(effects
+			(font
+				(size 1 1)
+				(thickness 0.15)
+			)
+		)
+	)
+	(gr_text "8"
+		(at 94.3864 95.6056 0)
+		(layer "F.SilkS")
+		(effects
+			(font
+				(size 1 1)
+				(thickness 0.15)
+			)
+		)
+	)
+	(gr_text "5"
+		(at 94.1832 131.7244 0)
+		(layer "F.SilkS")
+		(effects
+			(font
+				(size 1 1)
+				(thickness 0.15)
+			)
+		)
+	)
 	(gr_text "Ua"
 		(at 78.994 77.216 180)
@@
 		)
 	)
+	(gr_text "7"
+		(at 105.1052 105.5624 0)
+		(layer "F.SilkS")
+		(effects
+			(font
+				(size 1 1)
+				(thickness 0.15)
+			)
+		)
+	)
 	(gr_text "Ug"
 		(at 50.978786 110.236 270)
@@
 	)
 	(gr_text "1"
-		(at 93.98 124.079 0)
+		(at 79.4004 95.4532 0)
 		(layer "F.SilkS")
 		(effects
+			(font
+				(size 1 1)
+				(thickness 0.15)
+			)
+		)
+	)
+	(gr_text "6"
+		(at 105.2068 119.4816 0)
+		(layer "F.SilkS")
+		(effects
