File: tube-testers/ecc808/kicad/gm-v1/ecc808-gm-test-setup.kicad_pcb (KiCad board)
At the start: 2 copper layers, 99.6 x 99.6 mm, 32 parts, among them J10 Conn_01x01, J15 1Vrms@1kHz, J16 Conn_01x01, J17 Conn_01x01, J5 Conn_01x01, J6 Conn_01x01, J9 Conn_01x01, SW1 DPDT_SW_ANT21SECQE, U2 ECC88

Commit message: Finalize
Parts:
- removed C11: 100nF, Capacitor_THT:C_Rect_L7.2mm_W2.5mm_P5.00mm_FKS2_FKP2_MKS2_MKP2
- removed C4: 220uF, Capacitor_THT:CP_Radial_D8.0mm_P3.50mm
- removed JP1, JP2: Jumper_2_Open, Connector_PinHeader_2.54mm:PinHeader_1x02_P2.54mm_Vertical
- removed R1, R2: 680R/0.6W, Resistor_THT:R_Axial_DIN0207_L6.3mm_D2.5mm_P10.16mm_Horizontal
- removed TP2, TP3: TestPoint, TestPoint:TestPoint_Pad_D2.0mm
- C3: value 220uF -> 100nF; footprint Capacitor_THT:CP_Radial_D8.0mm_P3.50mm -> Capacitor_THT:C_Rect_L7.2mm_W2.5mm_P5.00mm_FKS2_FKP2_MKS2_MKP2
- R7: value 10R/0.4W/0.1% -> 100R/0.6W/0.1%
- U2: value ECC88 -> ECC808
- moved C3 15.0 mm to (82.4, 92.5)
Connections:
- C3 pad 1: Net-(JP1-B) -> FVCC
- SW1 pad 1: Net-(U2A-G) -> Net-(U2B-G)
- SW1 pad 3: Net-(U2B-G) -> Net-(U2A-G)
- SW1 pad 4: Net-(U2A-A) -> Net-(U2B-A)
- SW1 pad 6: Net-(U2B-A) -> Net-(U2A-A)
- U2 pad 1: Net-(U2A-A) -> Net-(U2B-G)
- U2 pad 2: Net-(U2A-G) -> FGND
- U2 pad 3: Net-(JP1-B) -> Net-(U2B-A)
- U2 pad 6: Net-(U2B-A) -> FGND
- U2 pad 7: Net-(U2B-G) -> Net-(U2A-A)
- U2 pad 8: Net-(JP2-B) -> FGND
- U2 pad 9: FGND -> Net-(U2A-G)
Routing:
- net Net-(JP2-B): track 21.1 -> 0.00 mm
- net Net-(JP1-B): track 21.0 -> 0.00 mm
- net Net-(U2B-G): track 31.1 -> 39.6 mm, vias 3 -> 2
- net Net-(U2A-A): track 38.7 -> 31.3 mm
- net Net-(U2A-G): track 41.1 -> 37.2 mm
- net Net-(U2B-A): track 37.0 -> 40.9 mm
- net FVCC: track 51.1 -> 50.4 mm
Other:
- board text added: "+250VDC"
- board text added: "-1.9VDC"
- board text added: "100mV/1mA"
- board text added: "ECC808 GM Tester V1 Michael Schenk 2024.09.15"
- board text added: "System 1:K=8,G=9,A=7 System 2:K=2,G=1,A=3"
- board text added: "Ua=250V, Ug=-1.9V, Ia=1.2mA, gm=1600uS (1.6mA/V) If=340mA"
- board text removed: "+100VDC"
- board text removed: "+9VDC"
- board text removed: "10mV/1mA"
- board text removed: "ECC88/E88CC GM Tester V4 Michael Schenk 2024.09.04"
- board text removed: "System 1:K=8,G=7,A=6 System 2:K=3,G=2,A=1"
- board text removed: "Ua=100V, Ug=+9V, Ia=15mA (Tol: +- 0.8mA), gm=12500uS (12.5mA/V Tol: +2.5mA/V, -2mA/V) Ia is VDC over R7 150mV gm is VAC over R7 of 125mVrms (Ug=+9VDC + 1Vrms@1kHz) End of life: Ia <= 13mA, gm <= mA/V"
