File: dac-pcm1702-v1/kicad-asrc-v10/src4392.kicad_sch (KiCad schematic)
At the start: 82 parts, among them J16 +5VIN, J17 GND, J2 TE MicroMatch, J5 COAXIN, J6 ISP, J7 Conn_01x15, J8 COAXGND, T1 Murata_DA103, U1 PLR237/T10BK, U10 TLV1117-33, U11 TLV1117-18, U13 24.576MHz, U14 FIN1047, U15 74LVC1G17, U16 74LVC1G17, U17 74LVC1G17, U18 PIC16F18056-I/SS, U2 PLR237/T10BK, U3 SRC4382/SRC4392, U6 PL133-37TI-R, U9 PLR237/T10BK

Commit message: Finalize V10
Parts:
- J7: footprint Connector_FFC-FPC:Molex_502231-1500_1x15-1SH_P0.5mm_Vertical -> Connector_TE-Connectivity:TE_Micro-MaTch_1-215079-4_2x07_P1.27mm_Vertical; symbol Connector_Generic:Conn_01x15 -> Connector_Generic:Conn_01x14
Connections:
- net GND: no longer J7.12 (Pin_12)
- net RESET: now also J7.12 (Pin_12); no longer J7.13 (Pin_13)
- net SCL: now also J7.13 (Pin_13); no longer J7.14 (Pin_14)
- net SDA: now also J7.14 (Pin_14); no longer J7.15 (Pin_15)
Other:
- note added: "History ------- V8 : 2024.04.13 Replace J15 with correct TE micro match V9 : 2025.04.20 LVDS V10 : 2025.04.26 J7 14pin micro match"
- note removed: "History ------- V8 2024.04.13 Replace J15 with correct TE micro match V9 2025.04.20 LVDS"
Changed lines of the file:
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@@
 	(title_block
 		(title "Async sample rate converter")
-		(date "2025-04-23")
-		(rev "V9")
+		(date "2025-04-26")
+		(rev "V10")
 	)
 	(text "ENC1_CHAN_B"
@@
 		)
 	)
-	(text "History\n-------\nV8 2024.04.13 Replace J15 with correct TE micro match\nV9 2025.04.20 LVDS"
+	(text "History\n-------\nV8  : 2024.04.13 Replace J15 with correct TE micro match\nV9  : 2025.04.20 LVDS\nV10 : 2025.04.26 J7 14pin micro match"
 		(exclude_from_sim no)
 		(at 297.688 149.098 0)
@@
 	(text "RESET\nSCL\nSCA"
 		(exclude_from_sim no)
-		(at 386.334 117.348 0)
+		(at 386.334 114.554 0)
 		(effects
 			(font
@@
 	(wire
 		(pts
-			(xy 363.22 114.3) (xy 379.73 114.3)
+			(xy 363.22 111.76) (xy 379.73 111.76)
 		)
 		(stroke
@@
 	(wire
 		(pts
-			(xy 364.49 116.84) (xy 379.73 116.84)
+			(xy 364.49 114.3) (xy 379.73 114.3)
 		)
 		(stroke
@@
 	(wire
 		(pts
-			(xy 359.41 129.54) (xy 364.49 129.54)
+			(xy 359.41 127) (xy 364.49 127)
 		)
 		(stroke
@@
 	(wire
 		(pts
-			(xy 359.41 132.08) (xy 365.76 132.08)
+			(xy 359.41 129.54) (xy 365.76 129.54)
 		)
 		(stroke
@@
 	(wire
 		(pts
-			(xy 365.76 119.38) (xy 379.73 119.38)
+			(xy 365.76 116.84) (xy 379.73 116.84)
 		)
 		(stroke
@@
 	(wire
 		(pts
-			(xy 363.22 127) (xy 359.41 127)
+			(xy 363.22 124.46) (xy 359.41 124.46)
 		)
 		(stroke
@@
 	(wire
 		(pts
-			(xy 364.49 129.54) (xy 364.49 116.84)
+			(xy 364.49 127) (xy 364.49 114.3)
 		)
 		(stroke
@@
 	(wire
 		(pts
-			(xy 363.22 114.3) (xy 363.22 127)
+			(xy 363.22 111.76) (xy 363.22 124.46)
 		)
 		(stroke
@@
 	(wire
 		(pts
-			(xy 365.76 132.08) (xy 365.76 119.38)
+			(xy 365.76 129.54) (xy 365.76 116.84)
 		)
 		(stroke
@@
 	)
 	(label "LRCLK-"
-		(at 359.41 109.22 0)
+		(at 360.68 109.22 0)
 		(effects
 			(font
@@
 	)
 	(label "DATAIN+"
-		(at 359.41 101.6 0)
+		(at 360.68 101.6 0)
 		(effects
 			(font
@@
 	)
 	(label "BCLK+"
-		(at 359.41 91.44 0)
+		(at 360.68 91.44 0)
 		(effects
 			(font
@@
 	)
 	(label "BCLK-"
-		(at 359.41 93.98 0)
+		(at 360.68 93.98 0)
 		(effects
 			(font
@@
 	)
 	(label "LRCLK+"
-		(at 359.41 106.68 0)
+		(at 360.68 106.68 0)
 		(effects
 			(font
@@
 	)
 	(label "DATAIN-"
-		(at 359.41 99.06 0)
+		(at 360.68 99.06 0)
 		(effects
 			(font
@@
 	(global_label "SCL"
 		(shape input)
-		(at 359.41 129.54 180)
+		(at 359.41 127 180)
 		(fields_autoplaced yes)
 		(effects
@@
 		)
 		(property "Intersheetrefs" "${INTERSHEET_REFS}"
-			(at 353.5714 129.54 0)
+			(at 353.5714 127 0)
 			(effects
 				(font
@@
 	(global_label "SDA"
 		(shape bidirectional)
-		(at 359.41 132.08 180)
+		(at 359.41 129.54 180)
 		(fields_autoplaced yes)
 		(effects
@@
 		)
 		(property "Intersheetrefs" "${INTERSHEET_REFS}"
-			(at 352.5584 132.08 0)
+			(at 352.5584 129.54 0)
 			(effects
 				(font
@@
 	(global_label "RESET"
 		(shape input)
-		(at 359.41 127 180)
+		(at 359.41 124.46 180)
 		(fields_autoplaced yes)
 		(effects
@@
 		)
 		(property "Intersheetrefs" "${INTERSHEET_REFS}"
-			(at 351.3339 127 0)
+			(at 351.3339 124.46 0)
 			(effects
 				(font
@@
 	)
 	(symbol
-		(lib_name "GND_60")
-		(lib_id "power:GND")
-		(at 379.73 111.76 270)
-		(unit 1)
-		(exclude_from_sim no)
-		(in_bom yes)
-		(on_board yes)
-		(dnp no)
-		(property "Reference" "#PWR0153"
-			(at 373.38 111.76 0)
-			(effects
-				(font
-					(size 1.27 1.27)
-				)
-				(hide yes)
-			)
-		)
-		(property "Value" "GND"
-			(at 375.3358 111.887 0)
-			(effects
-				(font
-					(size 1.27 1.27)
-				)
-			)
-		)
-		(property "Footprint" ""
-			(at 379.73 111.76 0)
-			(effects
-				(font
-					(size 1.27 1.27)
-				)
-				(hide yes)
-			)
-		)
-		(property "Datasheet" ""
-			(at 379.73 111.76 0)
-			(effects
-				(font
-					(size 1.27 1.27)
-				)
-				(hide yes)
-			)
-		)
-		(property "Description" ""
-			(at 379.73 111.76 0)
-			(effects
-				(font
-					(size 1.27 1.27)
-				)
-			)
-		)
-		(pin "1"
-		)
-		(instances
-			(project "src4392"
-				(path "/cf9dbafa-c7de-45de-ba16-6cea74dacd41"
-					(reference "#PWR0153")
-					(unit 1)
-				)
-			)
-		)
-	)
-	(symbol
 		(lib_name "+3.3V_2")
 		(lib_id "power:+3.3V")
@@
 	)
 	(symbol
-		(lib_id "Connector_Generic:Conn_01x15")
-		(at 384.81 101.6 0)
+		(lib_id "Connector_Generic:Conn_01x14")
+		(at 384.81 99.06 0)
 		(unit 1)
 		(exclude_from_sim no)
@@
 		(dnp no)
 		(property "Reference" "J7"
-			(at 384.048 122.174 0)
+			(at 384.048 119.634 0)
 			(effects
 				(font
@@
 		)
 		(property "Value" "Conn_01x15"
-			(at 380.746 123.952 0)
+			(at 380.746 121.412 0)
 			(effects
 				(font
@@
 			)
 		)
-		(property "Footprint" "Connector_FFC-FPC:Molex_502231-1500_1x15-1SH_P0.5mm_Vertical"
-			(at 384.81 101.6 0)
+		(property "Footprint" "Connector_TE-Connectivity:TE_Micro-MaTch_1-215079-4_2x07_P1.27mm_Vertical"
+			(at 384.81 99.06 0)
 			(effects
 				(font
@@
 		)
 		(property "Datasheet" "~"
-			(at 384.81 101.6 0)
+			(at 384.81 99.06 0)
 			(effects
 				(font
@@
 			)
 		)
-		(property "Description" "Generic connector, single row, 01x15, script generated (kicad-library-utils/schlib/autogen/connector/)"
-			(at 384.81 101.6 0)
+		(property "Description" "Generic connector, single row, 01x14, script generated (kicad-library-utils/schlib/autogen/connector/)"
+			(at 384.81 99.06 0)
 			(effects
 				(font
@@
 		(pin "4"
 		)
-		(pin "15"
-		)
 		(instances

Commit message: Update src4392.kicad_sch
Other:
- note added: "Current on 5V input Not prog: 21mA Prog: 61mA IWork: 125mA"
Changed lines of the file:
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@@
+		)
+	)
+	(text "Current on 5V input\nNot prog: 21mA\nProg: 61mA\nIWork: 125mA"
+		(exclude_from_sim no)
+		(at 337.058 20.828 0)
+		(effects
+			(font
+				(size 1.27 1.27)
+			)
+			(justify left)
 		)
 	)
