File: dac-pcm1702-v1/kicad-i2s-nos-v6/dac-i2s-nos.kicad_sch (KiCad schematic)
At the start: 81 parts, among them IC1 PCM1702P, IC2 PCM1702P, J10 GND, J11 +15VAIN, J12 GND, J13 -15VAIN, J15 A, J16 +5VIN, J17 GND, J18 GND, J2 Conn_02x07_Odd_Even, J3 +5VAIN, J6 OUT, J7 -5VAIN, J8 GND, J9 OUT, U1 OPA1612, U2 TC1185-1.8VCT713, U3 TC1185-3.3VCT713, U4 XC2C64A-xVQ44, U5 CM1293A−04SO, U6 OPA1612

Commit message: work in progress
Parts:
- removed C2: 10uF/6.3V, Capacitor_SMD:C_0805_2012Metric_Pad1.18x1.45mm_HandSolder, symbol dac-i2s-nos-rescue:CP-Device
- removed C3, C4: 10uF/6.3V, Capacitor_SMD:C_0805_2012Metric_Pad1.18x1.45mm_HandSolder, symbol dac-i2s-nos-rescue:CP-Device
- removed J15: A, kicad-snk:TE_CONN_RCPT_10POS_0.1_TIN_PCB, symbol kicad-snk:TE_CONN_RCPT_10POS_0.1_TIN_PCB
- removed R24, R25, R26, R27: 33R, Resistor_SMD:R_0603_1608Metric_Pad0.98x0.95mm_HandSolder, symbol Device:R
- added C2: 22uF/25V, Capacitor_SMD:C_1210_3225Metric_Pad1.33x2.70mm_HandSolder, symbol Device:C
- added C3, C4: 10uF/50V, Capacitor_SMD:C_1206_3216Metric_Pad1.33x1.80mm_HandSolder, symbol Device:C
- added C44: 1uF, Capacitor_SMD:C_0603_1608Metric_Pad1.08x0.95mm_HandSolder, symbol Device:C
- added J1: Conn_01x15, Connector_TE-Connectivity:TE_Micro-MaTch_1-215079-4_2x07_P1.27mm_Vertical, symbol Connector_Generic:Conn_01x14
- added R13, R14, R15, R16: 100R, Resistor_SMD:R_0402_1005Metric_Pad0.72x0.64mm_HandSolder, symbol Device:R
- added U7: FIN1048MTCX, Package_SO:TSSOP-16_4.4x5mm_P0.65mm, symbol kicad-snk:FIN1048
- C1, C41: value 220pF -> 47p
- C13, C14, C15, C22, C23, C24, C26, C33, C34, C39, C40, C5, C6, C7, C8, C9: value 100nF -> 1uF
- C31, C42: value 2n2 -> 1n
- C32, C43: value 560p -> 270p
Connections:
- net +1V8: now also C3.1
- net +3V3: now also C4.1, C44.2, U7.13 (VCC), U7.16 (EN)
- net BCK: now also U7.14 (ROUT2)
- net DATAIN: now also U7.11 (ROUT3)
- net GND: now also C2.2, C3.2, C4.2, C44.1, J1.3 (Pin_3), J1.6 (Pin_6), J1.9 (Pin_9), U7.12 (GND)
- net LRCK: now also U7.10 (ROUT4)
- net at J16.1 (Pin_1), U2.1 (VIN), U2.3 (~{SHDN})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: now also C2.1
- new net BCLK+: J1.4 (Pin_4), R13.2, U7.3 (RIN2+)
- new net BCLK-: J1.5 (Pin_5), R13.1, U7.4 (RIN2-)
- new net DATAIN+: J1.8 (Pin_8), R14.1, U7.6 (RIN3+)
- new net DATAIN-: J1.7 (Pin_7), R14.2, U7.5 (RIN3-)
- new net LRCLK+: J1.10 (Pin_10), R15.2, U7.7 (RIN4+)
- new net LRCLK-: J1.11 (Pin_11), R15.1, U7.8 (RIN4-)
- new net MCLK+: J1.2 (Pin_2), R16.1
- new net MCLK-: J1.1 (Pin_1), R16.2
- new net RESET: J1.12 (Pin_12)
- new net SCL: J1.13 (Pin_13)
- new net SDA: J1.14 (Pin_14)
- no-connect marks 7 -> 6
Other:
- note added: "App Note -------- C42=2.2n, C43=560p => fc(-3db)=46.7kHz Optimized for 192kHz -------------------- C42=1nF, C43=270pF => fc(-3db)=99.9kHz"
- note added: "MCLK 1/2"
- note added: "R4,R5,R6,R7: 0.1% C41,C42,C43: C0G 1%"
- note added: "R8,R9,R10,R11: 0.1% C1,C31,C32: C0G 1%"
- note removed: "R4,R5,R6,R7: 0.1% C41,C42,C43: film 2%"
- note removed: "R8,R9,R10,R11: 0.1% C1,C31,C32: film 2%"
- moved on the sheet: C5, C6, C7, C8, J11, J13, J18, J3, J7, J8, U4

Commit message: wip
Parts:
- C16, C17, C18, C25, C27, C28, C29, C30: footprint Capacitor_Tantalum_SMD:CP_EIA-3216-18_Kemet-A_Pad1.58x1.35mm_HandSolder -> Capacitor_SMD:C_1206_3216Metric_Pad1.33x1.80mm_HandSolder
- C35, C36, C37, C38: footprint Capacitor_Tantalum_SMD:CP_EIA-3528-21_Kemet-B_Pad1.50x2.35mm_HandSolder -> Capacitor_SMD:C_1206_3216Metric_Pad1.33x1.80mm_HandSolder
Connections:
- net MCLK: no longer names the net of U4.44 (IO1/GCK1)
Other:
- note added: "All CP are tantal polymer Ceramic capacitor 25V/0603"
- note added: "Input from ASRC is 192kHz PCM1702 support x16 oversampling (44.1kHz) CLKOUTR/CLKOUTL are 12.288MHz 2 channels x 32 bits x 192kHz => 12288000 Input from ASRC is 384kHz PCM1702 support x16 oversampling at 44.1kHz => 705.6kHz CLKOUTR/CLKOUTL are 24.576MHz 2 channels x 32 bits x 384kHz => 24.576MHz"
- note added: "v6 : LVDS, J1 14pin micro match, Footprint"
- note removed: "All CP are tantal polymer Ceramic capacitor 50V/0603"
- note removed: "Input from ASRC is 192kHz PCM1702 support x16 oversampling (44.1kHz) CLKOUTR/CLKOUTL are 12.288MHz 2 channels x 32 bits x 192kHz => 12288000"
Changed lines of the file:
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@@
 	(title_block
 		(title "DAC I2S NOS")
-		(date "2022-06-16")
-		(rev "V5")
+		(date "2025-05-09")
+		(rev "V6")
 	)
-	(text "All CP are tantal polymer\nCeramic capacitor 50V/0603"
+	(text "v6 : LVDS, J1 14pin micro match, Footprint"
+		(exclude_from_sim no)
+		(at 216.916 213.36 0)
+		(effects
+			(font
+				(size 1.27 1.27)
+			)
+			(justify left bottom)
+		)
+	)
+	(text "All CP are tantal polymer\nCeramic capacitor 25V/0603"
 		(exclude_from_sim no)
 		(at 248.92 246.38 0)
@@
 		)
 	)
-	(text "Input from ASRC is 192kHz\nPCM1702 support x16 oversampling (44.1kHz)\nCLKOUTR/CLKOUTL are 12.288MHz\n2 channels x 32 bits x 192kHz => 12288000"
+	(text "Input from ASRC is 192kHz\nPCM1702 support x16 oversampling (44.1kHz)\nCLKOUTR/CLKOUTL are 12.288MHz\n2 channels x 32 bits x 192kHz => 12288000\n\nInput from ASRC is 384kHz\nPCM1702 support x16 oversampling at 44.1kHz => 705.6kHz\nCLKOUTR/CLKOUTL are 24.576MHz\n2 channels x 32 bits x 384kHz => 24.576MHz"
 		(exclude_from_sim no)
-		(at 137.795 27.305 0)
+		(at 136.652 36.322 0)
 		(effects
 			(font
@@
 	(wire
 		(pts
-			(xy 30.48 173.99) (xy 44.45 173.99)
-		)
-		(stroke
-			(width 0)
-			(type default)
-		)
-	)
-	(wire
-		(pts
 			(xy 170.18 82.55) (xy 170.18 81.28)
 		)
@@
 		)
 	)
-	(global_label "MCLK"
-		(shape input)
-		(at 30.48 173.99 180)
-		(fields_autoplaced yes)
-		(effects
-			(font
-				(size 1.27 1.27)
-			)
-			(justify right)
-		)
-		(property "Intersheetrefs" "${INTERSHEET_REFS}"
-			(at 23.1295 173.99 0)
-			(effects
-				(font
-					(size 1.27 1.27)
-				)
-				(justify right)
-				(hide yes)
-			)
-		)
-	)
 	(global_label "CLKOUTL"
 		(shape output)
@@
 			)
 		)
-		(property "Footprint" "Capacitor_Tantalum_SMD:CP_EIA-3528-21_Kemet-B_Pad1.50x2.35mm_HandSolder"
+		(property "Footprint" "Capacitor_SMD:C_1206_3216Metric_Pad1.33x1.80mm_HandSolder"
 			(at 274.0152 172.72 0)
 			(effects
@@
 			)
 		)
-		(property "Footprint" "Capacitor_Tantalum_SMD:CP_EIA-3528-21_Kemet-B_Pad1.50x2.35mm_HandSolder"
+		(property "Footprint" "Capacitor_SMD:C_1206_3216Metric_Pad1.33x1.80mm_HandSolder"
 			(at 272.0848 181.61 0)
 			(effects
@@
 			)
 		)
-		(property "Footprint" "Capacitor_Tantalum_SMD:CP_EIA-3216-18_Kemet-A_Pad1.58x1.35mm_HandSolder"
+		(property "Footprint" "Capacitor_SMD:C_1206_3216Metric_Pad1.33x1.80mm_HandSolder"
 			(at 239.7252 154.94 0)
 			(effects
@@
 			)
 		)
-		(property "Footprint" "Capacitor_Tantalum_SMD:CP_EIA-3216-18_Kemet-A_Pad1.58x1.35mm_HandSolder"
+		(property "Footprint" "Capacitor_SMD:C_1206_3216Metric_Pad1.33x1.80mm_HandSolder"
 			(at 240.9952 113.03 0)
 			(effects
@@
 			)
 		)
-		(property "Footprint" "Capacitor_Tantalum_SMD:CP_EIA-3216-18_Kemet-A_Pad1.58x1.35mm_HandSolder"
+		(property "Footprint" "Capacitor_SMD:C_1206_3216Metric_Pad1.33x1.80mm_HandSolder"
 			(at 240.9952 124.46 0)
 			(effects
@@
 			)
 		)
-		(property "Footprint" "Capacitor_Tantalum_SMD:CP_EIA-3216-18_Kemet-A_Pad1.58x1.35mm_HandSolder"
+		(property "Footprint" "Capacitor_SMD:C_1206_3216Metric_Pad1.33x1.80mm_HandSolder"
 			(at 239.7252 166.37 0)
 			(effects
@@
 			)
 		)
-		(property "Footprint" "Capacitor_Tantalum_SMD:CP_EIA-3216-18_Kemet-A_Pad1.58x1.35mm_HandSolder"
+		(property "Footprint" "Capacitor_SMD:C_1206_3216Metric_Pad1.33x1.80mm_HandSolder"
 			(at 239.7252 25.4 0)
 			(effects
@@
 			)
 		)
-		(property "Footprint" "Capacitor_Tantalum_SMD:CP_EIA-3216-18_Kemet-A_Pad1.58x1.35mm_HandSolder"
+		(property "Footprint" "Capacitor_SMD:C_1206_3216Metric_Pad1.33x1.80mm_HandSolder"
 			(at 239.7252 36.83 0)
 			(effects
@@
 			)
 		)
-		(property "Footprint" "Capacitor_Tantalum_SMD:CP_EIA-3216-18_Kemet-A_Pad1.58x1.35mm_HandSolder"
+		(property "Footprint" "Capacitor_SMD:C_1206_3216Metric_Pad1.33x1.80mm_HandSolder"
 			(at 239.7252 67.31 0)
 			(effects
@@
 			)
 		)
-		(property "Footprint" "Capacitor_Tantalum_SMD:CP_EIA-3216-18_Kemet-A_Pad1.58x1.35mm_HandSolder"
+		(property "Footprint" "Capacitor_SMD:C_1206_3216Metric_Pad1.33x1.80mm_HandSolder"
 			(at 239.7252 78.74 0)
 			(effects
@@
 			)
 		)
-		(property "Footprint" "Capacitor_Tantalum_SMD:CP_EIA-3528-21_Kemet-B_Pad1.50x2.35mm_HandSolder"
+		(property "Footprint" "Capacitor_SMD:C_1206_3216Metric_Pad1.33x1.80mm_HandSolder"
 			(at 274.0152 85.09 0)
 			(effects
@@
 			)
 		)
-		(property "Footprint" "Capacitor_Tantalum_SMD:CP_EIA-3528-21_Kemet-B_Pad1.50x2.35mm_HandSolder"
+		(property "Footprint" "Capacitor_SMD:C_1206_3216Metric_Pad1.33x1.80mm_HandSolder"
 			(at 272.0848 93.98 0)
 			(effects

Commit message: Near finish
Parts:
- U5: footprint Package_SO:SC-74-6_1.5x2.9mm_P0.95mm -> Package_TO_SOT_SMD:SC-74-6_1.55x2.9mm_P0.95mm
Changed lines of the file:
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@@
 			)
 		)
-		(property "Footprint" "Package_SO:SC-74-6_1.5x2.9mm_P0.95mm"
+		(property "Footprint" "Package_TO_SOT_SMD:SC-74-6_1.55x2.9mm_P0.95mm"
 			(at 337.82 246.38 0)
 			(effects
