File: spdif-recv-cs8416-ak4137/kicad/v6/spdif_recv_cs8416_ak4137.kicad_pcb (KiCad board)
At the start: 4 copper layers, 76.9 x 56.5 mm, 84 parts, among them J16 +5VIN, J17 GND, J2 TE MicroMatch, J4 ISP, J5 COAXIN, J7 Conn_01x15, J8 COAXGND, T1 Murata_DA103, U1 PLR237/T10BK, U10 TLV1117-33, U12 74LVC1G17, U13 PIC16F18056-I/SS, U14 FIN1047, U2 PLR237/T10BK, U3 CS8416-xZZ, U4 74LVC1G17, U5 AK4137, U7 74LVC1G17, U8 24.576/49.152MHz, U9 PLR237/T10BK

Commit message: Update spdif_recv_cs8416_ak4137.kicad_pcb
Parts:
- C10, C5: moved to B.Cu
- moved C10 0.31 mm to (158.4, 85.3)
- moved C5 0.18 mm to (156.8, 85.2)
Routing:
- net GND: track 82.6 -> 86.4 mm, vias 2 -> 4
- net SRCEN: track 29.3 -> 31.0 mm
- net CM3: track 20.5 -> 19.4 mm
- net LRCKA: track 18.3 -> 17.2 mm
- net +3.3V: track 250.3 -> 249.5 mm

Commit message: Ready to order
Parts:
- moved G*** 41.9 mm to (171.9, 105.3)
- moved C5 0.25 mm to (157.0, 85.2)
- moved C10 0.25 mm to (158.7, 85.3)
Routing:
- net +3.3V: vias 19 -> 18
- net SRCEN: vias 3 -> 2
Other:
- board text added: "CS8416/AK4137 V6 2025.05.24"
- board text removed: "CS8416/AK4137 V5 2025.05.18"
