File: dac-pcm1702-v1/kicad-psu-v5/dac-psu.kicad_sch (KiCad schematic)
At the start: 81 parts, among them J1 AC, J10 LED, J11 GND, J12 +5V, J13 GND, J14 EARTH, J15 +17V, J16 -17V, J2 GND, J3 AC, J4 +15V, J5 GND, J6 -15V, J7 +5V, J8 GND, J9 -5V, U1 LM317_TO-220, U2 LT3045xMSE, U3 LT3094xMSE, U4 LT3045xMSE, U5 LT3094xMSE, U6 LM317_TO-220, U7 LM337_TO220

Commit message: Finalize V5 PSU
Parts:
- added D11: LED, LED_SMD:LED_0805_2012Metric_Pad1.15x1.40mm_HandSolder, symbol Device:LED
- added R15: 330R, Resistor_SMD:R_0603_1608Metric_Pad0.98x0.95mm_HandSolder, symbol Device:R
- C15, C16, C22, C23, C24, C25, C26, C27, C7, C8, C9: footprint Capacitor_Tantalum_SMD:CP_EIA-3528-21_Kemet-B_Pad1.50x2.35mm_HandSolder -> Capacitor_Tantalum_SMD:CP_EIA-3528-21_Kemet-B_HandSolder
- C17, C18, C19, C20: footprint Capacitor_Tantalum_SMD:CP_EIA-7343-31_Kemet-D_Pad2.25x2.55mm_HandSolder -> Capacitor_Tantalum_SMD:CP_EIA-7343-31_Kemet-D_HandSolder
- C5: manf# LGY1E223MELB45 -> 25MXG22000MEFCSN30X35
- C6: manf# LGY1E223MELB45 -> 1189-3893-ND
- U2, U3, U4, U5: footprint Package_SO:MSOP-12-1EP_3x4mm_P0.65mm_EP1.65x2.85mm -> Package_SO:MSOP-12-1EP_3x4.039mm_P0.65mm_EP1.651x2.845mm
Connections:
- net GND: now also D11.1 (K)
- net at C21.1, C9.1, D5.2 (A)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: now also R15.1
- new net: D11.2 (A), R15.2
Other:
- note added: "History ------- V5: Rounded PCB edge"
- note added: "Material -------- Trafo: PWR XFMR TOROIDAL 15VA 2x12V D:57.5mm H:24mm (Amgis LLC, XF-10232) Digikey:419-XF-10232-ND PWR XFMR TOROIDAL 15VA 2x12V D:57.5mm H:24mm (Talema Group LLC, 62052) Digikey:1295-1064-ND Line Filter: 250VAC 0.5A Schaffner 45mm x 28mm (FN402B-0.5-02) Digikey:817-2355-ND"
- moved on the sheet: C15, C16, C21, C9, D5, D6, HS1, J10, J11, J12, J13, R1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

Commit message: Update
Parts:
- H1, H2, H3, H4: footprint MountingHole:MountingHole_3.2mm_M3 -> MountingHole:MountingHole_3.2mm_M3_Pad_Via
Changed lines of the file:
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@@
 			)
 		)
-		(property "Footprint" "MountingHole:MountingHole_3.2mm_M3"
+		(property "Footprint" "MountingHole:MountingHole_3.2mm_M3_Pad_Via"
 			(at 254 262.89 0)
 			(effects
@@
 			)
 		)
-		(property "Footprint" "MountingHole:MountingHole_3.2mm_M3"
+		(property "Footprint" "MountingHole:MountingHole_3.2mm_M3_Pad_Via"
 			(at 276.86 262.89 0)
 			(effects
@@
 			)
 		)
-		(property "Footprint" "MountingHole:MountingHole_3.2mm_M3"
+		(property "Footprint" "MountingHole:MountingHole_3.2mm_M3_Pad_Via"
 			(at 254 273.05 0)
 			(effects
@@
 			)
 		)
-		(property "Footprint" "MountingHole:MountingHole_3.2mm_M3"
+		(property "Footprint" "MountingHole:MountingHole_3.2mm_M3_Pad_Via"
 			(at 276.86 273.05 0)
 			(effects
