File: dac-pcm1702-v1/kicad-psu-v5/dac-psu.kicad_pcb (KiCad board)
At the start: 2 copper layers, 123.2 x 81.3 mm, 81 parts, among them J1 AC, J10 LED, J11 GND, J12 +5V, J13 GND, J14 EARTH, J15 +17V, J16 -17V, J2 GND, J3 AC, J4 +15V, J5 GND, J6 -15V, J7 +5V, J8 GND, J9 -5V, U1 LM317_TO-220, U2 LT3045xMSE, U3 LT3094xMSE, U4 LT3045xMSE, U5 LT3094xMSE, U6 LM317_TO-220, U7 LM337_TO220

Commit message: Finalize V5 PSU
Parts:
- added D11: LED, LED_SMD:LED_0805_2012Metric_Pad1.15x1.40mm_HandSolder, F.Cu at (206.2, 61.9)
- added G***: LOGO, LOGO, F.Cu at (102.5, 112.0)
- added R15: 330R, Resistor_SMD:R_0603_1608Metric_Pad0.98x0.95mm_HandSolder, F.Cu at (209.9, 61.8)
- C15, C16, C22, C23, C24, C25, C26, C27, C7, C8, C9: footprint Capacitor_Tantalum_SMD:CP_EIA-3528-21_Kemet-B_Pad1.50x2.35mm_HandSolder -> Capacitor_Tantalum_SMD:CP_EIA-3528-21_Kemet-B_HandSolder
- C17, C18, C19, C20: value 47uF -> 47uF/25V; footprint Capacitor_Tantalum_SMD:CP_EIA-7343-31_Kemet-D_Pad2.25x2.55mm_HandSolder -> Capacitor_Tantalum_SMD:CP_EIA-7343-31_Kemet-D_HandSolder
- U2, U3, U4, U5: footprint Package_SO:MSOP-12-1EP_3x4mm_P0.65mm_EP1.65x2.85mm -> Package_SO:MSOP-12-1EP_3x4.039mm_P0.65mm_EP1.651x2.845mm
Routing:
- net GND: track 18.3 -> 28.0 mm
- net +17V: track 191.4 -> 186.7 mm
- net Net-(D5-A): track 66.5 -> 68.8 mm
- net Net-(D11-A): track 0.00 -> 1.70 mm
- net -17V: track 122.8 -> 123.5 mm
Other:
- board size 123.2 x 81.3 mm -> 123 x 81 mm
- board text added: "+"
- board text added: "Low noise +5V/+-5V/+-15V Power Supply V5 Michael Schenk, 2025.08.03"
- board text removed: "Low noise +5V/+-5V/+-15V Power Supplay V3 Michael Schenk, 2022.04.20"
- board text removed: "https://github.com/schenkmi/electronic-projects michaelschenk72@gmail.com"
- board text removed: "°"

Commit message: Update
Parts:
- H1, H2, H3, H4: footprint MountingHole:MountingHole_3.2mm_M3 -> MountingHole:MountingHole_3.2mm_M3_Pad_Via

Commit message: Some re-layout
Parts:
- D10, D5, D6, D7, D8, D9: moved to B.Cu
- moved R12 20.6 mm to (111.1, 54.6), turned to -90 degrees
- moved C10 20.1 mm to (105.7, 54.9), turned to -90 degrees
- moved C26 13.3 mm to (171.4, 76.3), turned to 90 degrees
- moved C9 13.3 mm to (171.4, 56.2), turned to 90 degrees
- moved D10 11.5 mm to (172.1, 109.8), turned to 0 degrees
- moved C27 11.2 mm to (176.7, 108.9), turned to 90 degrees
- moved R11 6.83 mm to (164.9, 107.9), turned to 90 degrees
- moved D8 6.34 mm to (172.9, 104.9), turned to 180 degrees
- moved D9 5.14 mm to (173.9, 83.2)
- moved D6 5.10 mm to (173.8, 63.1)
- moved D7 5.10 mm to (169.0, 83.2)
- moved D5 5.04 mm to (169.0, 63.1)
- moved C15 4.44 mm to (166.1, 58.8)
- moved C22 4.43 mm to (166.0, 79.1)
- moved R9 3.79 mm to (164.9, 111.9)
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Routing:
- net -17V: track 123.5 -> 149.4 mm, vias 4 -> 3
- net +17V: track 186.7 -> 211.8 mm
- net Net-(D7-A): track 53.5 -> 43.7 mm
- net Net-(D5-A): track 68.8 -> 59.2 mm, vias 1 -> 2
- net Net-(D9-A): track 17.4 -> 11.2 mm, vias 1 -> 0
- net Net-(J14-Pin_1): track 19.2 -> 13.3 mm
- net Net-(D6-A): track 17.5 -> 12.0 mm, vias 1 -> 0
- net Net-(D10-A): track 49.8 -> 54.2 mm
- net GND: track 28.0 -> 31.8 mm
- net Net-(D10-K): track 14.3 -> 12.2 mm, vias 1 -> 0
- net Net-(J9-Pin_1): track 16.4 -> 14.5 mm, vias 1 -> 0
- net Net-(J7-Pin_1): track 16.4 -> 14.5 mm, vias 1 -> 0
- net Net-(J6-Pin_1): track 15.8 -> 13.9 mm, vias 1 -> 0
- net Net-(J4-Pin_1): track 15.9 -> 14.1 mm, vias 1 -> 0
- net Net-(U3-SET): track 4.83 -> 4.19 mm
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Other:
- board text added: "Low noise +5V/+-5V/+-15V Power Supply V5 Michael Schenk, 2025.08.10"
- board text removed: "Low noise +5V/+-5V/+-15V Power Supply V5 Michael Schenk, 2025.08.03"
