File: lv-lownoise-psu/kicad/v5/lv-lownoise-psu.kicad_pcb (KiCad board)
At the start: 2 copper layers, 67.8 x 63 mm, 69 parts, among them J1 AC, J10 GND, J11 GND, J12 -5V, J13 EARTH, J2 GND, J3 AC, J4 +15V, J5 GND, J6 -15V, J7 LED, J8 GND, J9 +5V, Q1 BD139, Q2 BD140, U1 LM7805_TO220, U2 LM7905_TO220, U3 LT3045xMSE, U4 LT3094xMSE

Commit message: Minor change
Routing:
- net GND: track 13.3 -> 18.6 mm
Changed lines of the file:
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@@
+	)
+	(segment
+		(start 125.67312 51.8864)
+		(end 126.72032 52.9336)
+		(width 0.4)
+		(layer "F.Cu")
+		(net 1)
 	)
 	(segment
@@
 	)
 	(segment
+		(start 123.7782 51.8864)
+		(end 125.67312 51.8864)
+		(width 0.4)
+		(layer "F.Cu")
+		(net 1)
+	)
+	(segment
 		(start 117.3143 71.2204)
 		(end 117.2361 71.2986)
@@
 		(start 123.7782 51.8864)
 		(end 121.9532 51.8864)
+		(width 0.4)
+		(layer "F.Cu")
+		(net 1)
+	)
+	(segment
+		(start 126.72032 52.9336)
+		(end 128.6256 52.9336)
 		(width 0.4)
 		(layer "F.Cu")
@@
 	)
 	(segment
+		(start 117.1828 50)
+		(end 117.1956 49.9872)
+		(width 1)
+		(layer "F.Cu")
+		(net 12)
+	)
+	(segment
 		(start 119.4782 51.8864)
 		(end 119.4782 51.2364)
@@
 	)
 	(segment
+		(start 113.5 50)
+		(end 117.1828 50)
+		(width 1)
+		(layer "F.Cu")
+		(net 12)
+	)
+	(segment
 		(start 119.4782 50.5864)
 		(end 117.7948 50.5864)
@@
 	)
 	(segment
-		(start 117.1828 50)
-		(end 117.1956 49.9872)
-		(width 0.5)
-		(layer "F.Cu")
-		(net 12)
-	)
-	(segment
 		(start 118.4448 51.2364)
 		(end 117.1956 49.9872)
@@
 		(net 12)
 	)
-	(segment
-		(start 113.5 50)
-		(end 117.1828 50)
-		(width 0.5)
-		(layer "F.Cu")
-		(net 12)
-	)
 	(via
 		(at 122.4092 53.6244)
@@
 	)
 	(segment
-		(start 127.4318 50.6222)
-		(end 127.508 50.546)
-		(width 0.4)
-		(layer "F.Cu")
-		(net 14)
-	)
-	(segment
 		(start 126.5682 49.9364)
 		(end 127.254 50.6222)
@@
 	)
 	(segment
-		(start 127.508 50.546)
-		(end 138.9634 50.546)
-		(width 0.4)
-		(layer "F.Cu")
-		(net 14)
-	)
-	(segment
 		(start 127.2182 50.5864)
 		(end 127.254 50.6222)
@@
 	)
 	(segment
+		(start 138.8872 50.6222)
+		(end 138.9634 50.546)
+		(width 1)
+		(layer "F.Cu")
+		(net 14)
+	)
+	(segment
 		(start 123.7782 51.2364)
 		(end 126.6398 51.2364)
@@
 	(segment
 		(start 127.254 50.6222)
-		(end 127.4318 50.6222)
-		(width 0.4)
+		(end 138.8872 50.6222)
+		(width 1)
 		(layer "F.Cu")
 		(net 14)
@@
 	)
 	(segment
+		(start 127.3556 68.6308)
+		(end 138.9126 68.6308)
+		(width 1)
+		(layer "F.Cu")
+		(net 15)
+	)
+	(segment
 		(start 127.3452 68.6204)
 		(end 127.3556 68.6308)
@@
 	)
 	(segment
-		(start 127.3556 68.6308)
-		(end 138.9126 68.6308)
-		(width 0.4)
-		(layer "F.Cu")
-		(net 15)
-	)
-	(segment
 		(start 123.8832 69.2704)
 		(end 126.716 69.2704)
@@
 	)
 	(segment
+		(start 119.5832 68.6204)
+		(end 117.6829 68.6204)
+		(width 0.4)
+		(layer "F.Cu")
+		(net 18)
+	)
+	(segment
+		(start 119.5832 70.5704)
+		(end 118.796908 70.5704)
+		(width 0.4)
+		(layer "F.Cu")
+		(net 18)
+	)
+	(segment
+		(start 119.5832 68.6204)
+		(end 120.7582 68.6204)
+		(width 0.4)
+		(layer "F.Cu")
+		(net 18)
+	)
+	(segment
+		(start 119.5832 69.2704)
+		(end 119.5832 68.6204)
+		(width 0.4)
+		(layer "F.Cu")
+		(net 18)
+	)
+	(segment
+		(start 117.6829 68.6204)
+		(end 117.2361 68.1736)
+		(width 0.4)
+		(layer "F.Cu")
+		(net 18)
+	)
+	(segment
 		(start 113.08 68)
 		(end 117.0625 68)
-		(width 0.5)
-		(layer "F.Cu")
-		(net 18)
-	)
-	(segment
-		(start 119.5832 68.6204)
-		(end 117.6829 68.6204)
+		(width 1)
+		(layer "F.Cu")
+		(net 18)
+	)
+	(segment
+		(start 119.5832 67.9704)
+		(end 117.4393 67.9704)
+		(width 0.4)
+		(layer "F.Cu")
+		(net 18)
+	)
+	(segment
+		(start 117.2188 68)
+		(end 117.2361 67.9827)
+		(width 0.5)
+		(layer "F.Cu")
+		(net 18)
+	)
+	(segment
+		(start 121.5136 67.9704)
+		(end 121.7332 68.19)
+		(width 0.4)
+		(layer "F.Cu")
+		(net 18)
+	)
+	(segment
+		(start 118.796908 70.5704)
+		(end 117.2361 69.009592)
+		(width 0.4)
+		(layer "F.Cu")
+		(net 18)
+	)
+	(segment
+		(start 117.4393 67.9704)
+		(end 117.2361 68.1736)
+		(width 0.4)
+		(layer "F.Cu")
+		(net 18)
+	)
+	(segment
+		(start 121.7332 68.19)
+		(end 121.7332 69.5954)
 		(width 0.4)
 		(layer "F.Cu")
@@
 		(start 117.0625 68)
 		(end 117.2361 68.1736)
-		(width 0.5)
-		(layer "F.Cu")
-		(net 18)
-	)
-	(segment
-		(start 119.5832 70.5704)
-		(end 118.796908 70.5704)
-		(width 0.4)
-		(layer "F.Cu")
-		(net 18)
-	)
-	(segment
-		(start 119.5832 68.6204)
-		(end 120.7582 68.6204)
-		(width 0.4)
-		(layer "F.Cu")
-		(net 18)
-	)
-	(segment
-		(start 119.5832 69.2704)
-		(end 119.5832 68.6204)
-		(width 0.4)
-		(layer "F.Cu")
-		(net 18)
-	)
-	(segment
-		(start 117.6829 68.6204)
-		(end 117.2361 68.1736)
-		(width 0.4)
-		(layer "F.Cu")
-		(net 18)
-	)
-	(segment
-		(start 119.5832 67.9704)
-		(end 117.4393 67.9704)
-		(width 0.4)
-		(layer "F.Cu")
-		(net 18)
-	)
-	(segment
-		(start 117.2188 68)
-		(end 117.2361 67.9827)
-		(width 0.5)
-		(layer "F.Cu")
-		(net 18)
-	)
-	(segment
-		(start 121.5136 67.9704)
-		(end 121.7332 68.19)
-		(width 0.4)
-		(layer "F.Cu")
-		(net 18)
-	)
-	(segment
-		(start 118.796908 70.5704)
-		(end 117.2361 69.009592)
-		(width 0.4)
-		(layer "F.Cu")
-		(net 18)
-	)
-	(segment
-		(start 117.4393 67.9704)
-		(end 117.2361 68.1736)
-		(width 0.4)
-		(layer "F.Cu")
-		(net 18)
-	)
-	(segment
-		(start 121.7332 68.19)
-		(end 121.7332 69.5954)
-		(width 0.4)
-		(layer "F.Cu")
-		(net 18)
+		(width 1)
+		(layer "F.Cu")
+		(net 18)
