File: lt1115-phono-mm-mc/kicad/v6/lt1115-phono-mm-mc.kicad_pcb (KiCad board)
At the start: 2 copper layers, 96.5 x 54.6 mm, 49 parts, among them J1 IN, J2 IN_GND, J3 +15V, J4 GND, J5 -15V, J6 OUT, J7 OUT_GND, SW1 SW_SPST, U1 LT1115, U2 LM334M, U3 LT1010, U4 OPA188xxDBV

Commit message: WIP
Parts:
- removed SW1: SW_SPST, Button_Switch_SMD:SW_DIP_SPSTx01_Slide_Omron_A6S-110x_W8.9mm_P2.54mm
- added C2: 10pF, Capacitor_SMD:C_0805_2012Metric_Pad1.18x1.45mm_HandSolder, F.Cu at (128.8, 156.9)
- added C20: 100pF, Capacitor_SMD:C_0805_2012Metric_Pad1.18x1.45mm_HandSolder, F.Cu at (128.8, 162.9)
- added C21: 220p, Capacitor_SMD:C_0805_2012Metric_Pad1.18x1.45mm_HandSolder, F.Cu at (128.8, 165.9)
- added C22: 220uF/25V, Capacitor_THT:CP_Radial_D8.0mm_P3.50mm, F.Cu at (149.2, 162.8)
- added C3: 47pF, Capacitor_SMD:C_0805_2012Metric_Pad1.18x1.45mm_HandSolder, F.Cu at (128.8, 159.9)
- added R17: 100R, Resistor_SMD:R_0805_2012Metric_Pad1.20x1.40mm_HandSolder, F.Cu at (133.6, 156.9)
- added R18: 10R, Resistor_SMD:R_0805_2012Metric_Pad1.20x1.40mm_HandSolder, F.Cu at (133.6, 159.8)
- added R19: 330R, Resistor_SMD:R_0805_2012Metric_Pad1.20x1.40mm_HandSolder, F.Cu at (133.6, 162.8)
- added SW2: SW_DIP_x03, Button_Switch_SMD:SW_DIP_SPSTx03_Slide_6.7x9.18mm_W8.61mm_P2.54mm_LowProfile, F.Cu at (120.1, 152.5)
- added SW3: SW_DIP_x02, Button_Switch_SMD:SW_DIP_SPSTx02_Slide_6.7x6.64mm_W8.61mm_P2.54mm_LowProfile, F.Cu at (132.7, 151.2)
- added SW4: SW_DIP_x03, Button_Switch_SMD:SW_DIP_SPSTx03_Slide_6.7x9.18mm_W8.61mm_P2.54mm_LowProfile, F.Cu at (120.1, 163.4)
- C1: value C -> 220uF/25V; footprint Capacitor_SMD:C_0805_2012Metric_Pad1.18x1.45mm_HandSolder -> Capacitor_THT:CP_Radial_D8.0mm_P3.50mm
- C4, C7: value 220uF/25V -> 10uF/25V; footprint Capacitor_THT:CP_Radial_D8.0mm_P3.50mm -> Capacitor_Tantalum_SMD:CP_EIA-3528-12_Kemet-T_HandSolder
- R1: value 100R -> 47k
- moved C1 64.6 mm to (149.2, 153.3), turned to 0 degrees
Connections:
- C1 pad 1: Net-(C1-Pad1) -> unconnected-(C1-Pad1)
- C1 pad 2: GND -> unconnected-(C1-Pad2)
- J1 pad 1: Net-(C1-Pad1) -> Net-(J1-Pin_1)
- R1 pad 1: Net-(C1-Pad1) -> Net-(J1-Pin_1)
- U1 pad 3: Net-(C1-Pad1) -> Net-(J1-Pin_1)
Routing:
- net Net-(J1-Pin_1): track 0.00 -> 16.8 mm, vias 0 -> 2
- net Net-(C1-Pad1): track 16.8 -> 0.00 mm, vias 2 -> 0

Commit message: wip
Parts:
- added J8: IN_GND, Connector_Pin:Pin_D1.0mm_L10.0mm, F.Cu at (84.7, 105.9)
- added J9: OUT_GND, Connector_Pin:Pin_D1.0mm_L10.0mm, F.Cu at (163.7, 106.3)
- C10: renamed from C6; footprint Capacitor_SMD:C_1210_3225Metric_Pad1.33x2.70mm_HandSolder -> Capacitor_SMD:C_0805_2012Metric_Pad1.18x1.45mm_HandSolder
- C17: renamed from C11; value 220uF/25V -> 10uF/25V; footprint Capacitor_THT:CP_Radial_D8.0mm_P3.50mm -> Capacitor_Tantalum_SMD:CP_EIA-3528-12_Kemet-T_HandSolder
- C18: renamed from C12; footprint Capacitor_SMD:C_1210_3225Metric_Pad1.33x2.70mm_HandSolder -> Capacitor_SMD:C_0805_2012Metric_Pad1.18x1.45mm_HandSolder
- C19: renamed from C13; footprint Capacitor_SMD:C_1210_3225Metric_Pad1.33x2.70mm_HandSolder -> Capacitor_SMD:C_0805_2012Metric_Pad1.18x1.45mm_HandSolder
- C20: renamed from C14; value 220uF/25V -> 10uF/25V; footprint Capacitor_THT:CP_Radial_D8.0mm_P3.50mm -> Capacitor_Tantalum_SMD:CP_EIA-3528-12_Kemet-T_HandSolder
- C6: renamed from C17; value 100nF -> 1uF
- C7: renamed from C18; value 100nF -> 1uF
- C9: renamed from C5; footprint Capacitor_SMD:C_1210_3225Metric_Pad1.33x2.70mm_HandSolder -> Capacitor_SMD:C_0805_2012Metric_Pad1.18x1.45mm_HandSolder
- H1, H2, H3, H4: footprint MountingHole:MountingHole_3.2mm_M3 -> MountingHole:MountingHole_3.2mm_M3_Pad_Via
- U1: renamed from U4; value OPA188xxDBV -> OPA182IDBVR
- U2: renamed from U1; footprint Package_DIP:DIP-8_W7.62mm -> Package_DIP:DIP-8_W7.62mm_Socket
- U4: renamed from U3; footprint Package_DIP:DIP-8_W7.62mm -> Package_DIP:DIP-8_W7.62mm_Socket
- moved C4 72.7 mm to (93.3, 102.5), turned to 90 degrees
- moved C21 70.2 mm to (182.4, 101.0)
- moved C3 68.9 mm to (95.9, 102.5), turned to 90 degrees
- moved C2 65.0 mm to (98.4, 102.5), turned to 90 degrees
- moved SW2 58.4 mm to (95.9, 110.2), turned to 90 degrees
- moved C1 55.7 mm to (89.8, 117.2), turned to -90 degrees
- moved R2 50.4 mm to (93.3, 129.6), turned to -90 degrees
- moved R4 48.4 mm to (98.4, 129.6), turned to -90 degrees
- moved R3 46.6 mm to (95.9, 129.6), turned to -90 degrees
- moved SW1 39.1 mm to (95.9, 121.9), turned to -90 degrees
- moved C16 38.8 mm to (185.6, 140.1)
- moved C17 23.8 mm to (158.8, 123.7)
- moved C19 15.0 mm to (147.1, 114.8)
- moved C20 9.92 mm to (145.4, 124.7), turned to 0 degrees
- moved C22 9.78 mm to (160.8, 114.3)
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- renumbered C2 to C1, C7 to C11, C19 to C12, C8 to C13, C9 to C14, C10 to C15, C1 to C16, C3 to C2, C22 to C21, C15 to C22, C20 to C3, C21 to C4, C16 to C5, C4 to C8, R16 to R10, R6 to R11, R7 to R12, R9 to R13, R10 to R14, R11 to R15, R12 to R16, R8 to R17, R13 to R18, R14 to R19, R18 to R2, R17 to R3, R19 to R4, R4 to R5, R2 to R6, R3 to R7, R15 to R8, R5 to R9, SW2 to SW1, SW4 to SW2, U2 to U3
Connections:
- C16 pad 1: unconnected-(C1-Pad1) -> GND
- C16 pad 2: unconnected-(C1-Pad2) -> -15V
- C21 pad 1: unconnected-(C22-Pad1) -> +15V
- C21 pad 2: unconnected-(C22-Pad2) -> GND
Routing:
- net -15V: track 139.3 -> 101.7 mm
- net +15V: track 110.2 -> 81.2 mm
- net Net-(J1-Pin_1): track 16.8 -> 33.4 mm, vias 2 -> 1
- net Net-(C4-Pad1): track 0.00 -> 2.41 mm
- net Net-(C3-Pad1): track 0.00 -> 2.41 mm
- net Net-(C2-Pad1): track 0.00 -> 2.41 mm
- net Net-(R4-Pad1): track 0.00 -> 2.41 mm
- net Net-(R3-Pad1): track 0.00 -> 2.41 mm
- net Net-(R2-Pad1): track 0.00 -> 2.41 mm
Other:
- board text added: "LT1115 MC/MM Phono PreAmp V6 Michael Schenk 2025.08.23"
- board text removed: "LT1115 MC/MM Phono PreAmp V5 Michael Schenk 2023.02.01"

Commit message: wip
Parts:
- added G***: LOGO, LOGO, F.Cu at (121.9, 157.2)
- C1, C13, C2, C3, C4: footprint Capacitor_SMD:C_0805_2012Metric_Pad1.18x1.45mm_HandSolder -> Capacitor_SMD:C_0603_1608Metric_Pad1.08x0.95mm_HandSolder
- C14, C22: footprint Capacitor_SMD:C_1206_3216Metric_Pad1.33x1.80mm_HandSolder -> Capacitor_SMD:C_0603_1608Metric_Pad1.08x0.95mm_HandSolder
- C15: footprint Capacitor_SMD:C_1210_3225Metric_Pad1.33x2.70mm_HandSolder -> Capacitor_SMD:C_0603_1608Metric_Pad1.08x0.95mm_HandSolder
- moved SW3 40.0 mm to (104.2, 123.1), turned to -90 degrees
- moved C16 29.2 mm to (156.9, 134.8), turned to 90 degrees
- moved C21 25.5 mm to (156.9, 101.1), turned to 90 degrees
- moved C20 15.0 mm to (136.9, 112.4), turned to 90 degrees
- moved R14 11.2 mm to (112.3, 107.7), turned to 180 degrees
- moved R17 11.2 mm to (113.2, 103.3), turned to 90 degrees
- moved C8 10.5 mm to (121.9, 110.8), turned to 0 degrees
- moved C11 9.83 mm to (111.7, 124.1), turned to 180 degrees
- moved C14 9.78 mm to (108.5, 105.9)
- moved C13 9.44 mm to (108.5, 104.4)
- moved R12 8.39 mm to (108.5, 107.7)
- moved C15 8.29 mm to (112.3, 106.0), turned to 180 degrees
- moved C19 8.01 mm to (139.6, 111.8), turned to 90 degrees
- moved R11 7.18 mm to (104.2, 111.0), turned to 0 degrees
- moved R13 6.88 mm to (127.7, 122.2)
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Routing:
- net Net-(R15-Pad2): track 22.9 -> 1.86 mm, vias 2 -> 1
- net -15V: track 101.7 -> 84.5 mm, vias 4 -> 3
- net SERVO_INR: track 60.4 -> 44.3 mm, vias 4 -> 3
- net +15V: track 81.2 -> 93.7 mm, vias 1 -> 3
- net Net-(C5-Pad1): track 13.8 -> 2.96 mm, vias 2 -> 0
- net Net-(C13-Pad2): track 13.1 -> 5.28 mm, vias 2 -> 0
- net SERVO_OUT: track 2.79 -> 7.65 mm, vias 0 -> 1
- net Net-(U1--): track 9.06 -> 13.3 mm, vias 1 -> 2
- net GND: track 3.72 -> 0.00 mm
- net Net-(R13-Pad1): track 3.63 -> 0.00 mm
- net Net-(C13-Pad1): track 10.4 -> 6.97 mm
- net Net-(C4-Pad1): track 2.41 -> 0.00 mm
- net Net-(C3-Pad1): track 2.41 -> 0.00 mm
- net Net-(C2-Pad1): track 2.41 -> 0.00 mm
- net Net-(R4-Pad1): track 2.41 -> 0.00 mm
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Other:
- board text removed: "michaelschenk72@gmail.com"

Commit message: Update lt1115-phono-mm-mc.kicad_pcb
Parts:
- moved G*** 32.5 mm to (137.7, 128.8)
- moved J2 7.14 mm to (84.8, 122.3)
- moved J9 4.53 mm to (161.3, 110.1)
- moved J8 4.24 mm to (84.8, 110.2)
- moved R13 3.15 mm to (125.8, 119.6)
- moved U3 3.15 mm to (122.1, 121.1)
- moved J6 2.47 mm to (161.3, 116.2)
- moved J7 2.44 mm to (161.3, 122.3)
- moved R18 0.34 mm to (153.6, 111.1)
- moved C22 0.33 mm to (158.2, 110.3)
- moved R19 0.33 mm to (156.5, 110.1)
Routing:
- net -15V: track 84.5 -> 143.3 mm, vias 3 -> 6
- net Net-(R15-Pad2): track 1.86 -> 21.1 mm, vias 1 -> 4
- net Net-(C5-Pad1): track 2.96 -> 9.53 mm, vias 0 -> 1
- net +15V: track 93.7 -> 98.0 mm
- net Net-(R6-Pad2): track 4.53 -> 7.84 mm
- net Net-(J6-Pin_1): track 7.13 -> 10.0 mm, vias 0 -> 1
- net Net-(R4-Pad1): track 0.00 -> 2.41 mm
- net Net-(R3-Pad1): track 0.00 -> 2.41 mm
- net Net-(R2-Pad1): track 0.00 -> 2.41 mm
- net Net-(C4-Pad1): track 0.00 -> 2.37 mm
- net Net-(C3-Pad1): track 0.00 -> 2.37 mm
- net Net-(C2-Pad1): track 0.00 -> 2.37 mm
- net Net-(R13-Pad1): track 0.00 -> 1.83 mm
- net SERVO_INR: track 44.3 -> 45.8 mm, vias 3 -> 2
Other:
- board size 96.5 x 54.6 mm -> 96.6 x 54.6 mm
- board text added: "+"
- board text added: "LT1115 MC/MM Phono PreAmp V6 Michael Schenk 2025.08.25"
- board text removed: "LT1115 MC/MM Phono PreAmp V6 Michael Schenk 2025.08.23"

Commit message: Finalize
Other:
- board text added: "SW1 1:CLOSE => R2 10R 2:CLOSE => R3 100R 3:CLOSE => R4 330R"
- board text added: "SW2 1:CLOSE => C2 47pF 2:CLOSE => C3 100pF 3:CLOSE => C4 220pF"
- board text added: "SW3 1:CLOSE => MC / OPEN => MM 2:CLOSE => MC / OPEN => MM MM:40dB, MC:60dB"
