File: spdif-recv-ak4118-ak4137/kicad/v2/spdif_recv_ak4118_ak4137.kicad_pcb (KiCad board)
At the start: 4 copper layers, 76.9 x 56.5 mm, 86 parts, among them J1 COAXIN, J2 COAXGND, J3 ISP, J4 TTL-232R-3V3, J5 Conn_01x04_Pin, J6 TE MicroMatch, J7 +5VIN, J8 GND, J9 Conn_01x15, T1 Murata_DA103, U1 PLR237/T10BK, U10 NCP163ASN330T1G, U11 NCP163ASN330T1G, U12 NCP163ASN330T1G, U13 24.576/49.152MHz, U14 FIN1047, U2 PLR237/T10BK, U3 PLR237/T10BK, U4 PIC16F18056-I/SS, U5 74LVC1G17, U6 74LVC1G17, U7 74LVC1G17, U8 AK4118AEQ, U9 AK4137

Commit message: V2 finalize
Parts:
- moved J4 19.3 mm to (161.9, 68.6), turned to 90 degrees
Routing:
- net GND: track 128.5 -> 103.3 mm
- net ICSPDAT: track 19.3 -> 30.2 mm
- net ICSPCLK: track 23.3 -> 30.3 mm
- net Net-(U8A-RX0): track 10.4 -> 11.3 mm
Other:
- board text added: "AK4118/AK4137 V2 2026.05.10"
- board text removed: "AK4118/AK4137 V1 2026.04.24"
