File: dac-pcm1702-v1/kicad-asrc-v14/src4392.kicad_pcb (KiCad board)
At the start: 4 copper layers, 76.8 x 56.5 mm, 84 parts, among them J10 TE MicroMatch, J18 +5VIN, J19 GND, J2 TE MicroMatch, J4 TTL-232R-3V3, J5 COAXIN, J6 ISP, J7 Conn_01x15, J8 COAXGND, J9 Conn_01x04_Pin, T1 Murata_DA103, U1 PLR237/T10BK, U12 NCP163ASN180T1G, U13 24.576MHz, U14 FIN1047, U15 74LVC1G17, U16 74LVC1G17, U17 74LVC1G17, U18 PIC16F18056-I/SS, U19 NCP163ASN330T1G, U2 PLR237/T10BK, U20 NCP163ASN330T1G, U3 SRC4382/SRC4392, U6 PL133-37TI-R, U9 PLR237/T10BK

Commit message: Finalize V14
Parts:
- added J11: LED, Connector_Pin:Pin_D1.0mm_L10.0mm, F.Cu at (145.7, 110.4)
- added J12: GND, Connector_Pin:Pin_D1.0mm_L10.0mm, F.Cu at (151.3, 110.5)
- added R18: 330R, Resistor_SMD:R_0603_1608Metric_Pad0.98x0.95mm_HandSolder, F.Cu at (148.0, 109.5)
- moved J19 0.58 mm to (136.4, 110.4)
Connections:
- U18 pad 15: unconnected-(U18-RC4-Pad15) -> RC4/LED
Routing:
- net RC4/LED: track 0.00 -> 34.7 mm, vias 0 -> 2
- net Net-(J11-Pin_1): track 0.00 -> 2.23 mm
Other:
- board text added: "ASRC V14 2026.06.05"
- board text added: "LED"
- board text removed: "ASRC V14 2026.06.04"
