File: pre-amp-ECC86/kicad/psu-v3/power-supply-30V-6.3V-5V.kicad_sch (KiCad schematic)
At the start: 67 parts, among them J1 AC-LV, J10 GND, J11 IN, J12 GND, J13 EARTH, J14 GND, J2 AC-LV, J3 HV, J5 LV, J6 GND, J7 LED, J8 GND, J9 +5V, K1 G6S-2 DC5, Q3 MMBTRC116SS, U2 AP64202QSP-13, U3 AP64202QSP-13, U4 TLC555xD, U5 LT3080xST

Commit message: Update power-supply-30V-6.3V-5V.kicad_sch
Other:
- note added: "With real PSUv1 100k (1MHz) Out: 6.3V@660mA, Vrippel 4.31mVeff(BW=20MHz) => 4.158W, n=85%, TU3=46°C In: 35V@140mA => 4.9W With real PSUv3 100k (1MHz) Out: 6.3V@660mA, Vrippel 4.6mVeff(BW=20MHz) TU3=44°C In: 37V"
- note removed: "With real PSUv1 100k (1MHz) Out: 6.3V@660mA, Vrippel 4.31mVeff(BW=20MHz) => 4.158W, n=85%, TU3=46°C In: 35V@140mA => 4.9W"
Changed lines of the file:
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@@
 		)
 	)
-	(text "With real PSUv1\n100k (1MHz)\nOut: 6.3V@660mA, Vrippel 4.31mVeff(BW=20MHz) => 4.158W, n=85%, TU3=46°C\nIn: 35V@140mA => 4.9W"
+	(text "With real PSUv1\n100k (1MHz)\nOut: 6.3V@660mA, Vrippel 4.31mVeff(BW=20MHz) => 4.158W, n=85%, TU3=46°C\nIn: 35V@140mA => 4.9W\n\nWith real PSUv3\n100k (1MHz)\nOut: 6.3V@660mA, Vrippel 4.6mVeff(BW=20MHz) TU3=44°C\nIn: 37V"
 		(exclude_from_sim no)
-		(at 19.812 108.712 0)
+		(at 19.812 114.046 0)
 		(effects
 			(font

Commit message: Using 10nF
Parts:
- C28: value 100nF/50V -> 10nF/50V
Changed lines of the file:
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@@
 			)
 		)
-		(property "Value" "100nF/50V"
+		(property "Value" "10nF/50V"
 			(at 207.01 167.6399 0)
 			(show_name no)
